Commit message: added xacro property

File: src/picknik_ur_base_config/description/picknik_ur5e.xacro (robot description, xacro)
@@ -28,6 +28,8 @@
   <!-- Import environment macros -->
   <xacro:include filename="$(find picknik_accessories)/descriptions/geometry/collision_and_visual/cube_collision_and_visual.urdf.xacro" />
-  <!-- initial positions for simulations (Mock Hardware and Gazebo) -->
+  <!-- Initial positions for simulations (Mock Hardware and Gazebo) -->
   <xacro:arg name="initial_positions_file" default="$(find picknik_ur5e_base_config)/config/initial_positions.yaml"/>
+  <!-- Convert args to properties for substitution in macros -->
+  <xacro:property name="initial_positions_file" default="$(arg initial_positions_file)"/>
   <link name="world" />
   <!-- arm -->

Commit message: Update base descriptions

File: src/picknik_ur_base_config/description/picknik_ur5e.xacro (robot description, xacro)
@@ -2,7 +2,8 @@
 <robot xmlns:xacro="http://wiki.ros.org/xacro" name="$(arg name)">
   <!-- parameters -->
-  <xacro:arg name="use_fake_hardware" default="true" />
+  <xacro:arg name="use_fake_hardware" default="false" />
   <xacro:arg name="external_camera" default="false" />
   <xacro:arg name="has_tool_changer" default="true" />
+  <xacro:arg name="use_pinch_link" default="true" />
   <xacro:arg name="name" default="" />
   <xacro:arg name="joint_limits_parameters_file" default="" />
@@ -26,10 +27,10 @@
   <xacro:include filename="$(find picknik_accessories)/descriptions/sensors/realsense_d415.urdf.xacro" />
   <xacro:include filename="$(find picknik_accessories)/descriptions/sensors/realsense_d435.urdf.xacro" />
+  <xacro:include filename="$(find picknik_ur_base_config)/description/pinch_link.xacro" />
+  <!-- Initial positions for simulations (Mock Hardware and Gazebo) -->
+  <xacro:arg name="initial_positions_file" default="$(find picknik_ur_base_config)/config/initial_positions.yaml"/>
+  <xacro:property name="initial_positions_file" default="$(arg initial_positions_file)"/>
   <!-- Import environment macros -->
   <xacro:include filename="$(find picknik_accessories)/descriptions/geometry/collision_and_visual/cube_collision_and_visual.urdf.xacro" />
-  <!-- Initial positions for simulations (Mock Hardware and Gazebo) -->
-  <xacro:arg name="initial_positions_file" default="$(find picknik_ur_base_config)/config/initial_positions.yaml"/>
-  <!-- Convert args to properties for substitution in macros -->
-  <xacro:property name="initial_positions_file" default="$(arg initial_positions_file)"/>
   <link name="world" />
   <!-- arm -->
@@ -39,7 +40,7 @@
     parent="world"
     joint_limits_parameters_file="$(arg joint_limits_parameters_file)"
-    kinematics_parameters_file="$(arg kinematics_parameters_file)/$(arg name)/default_kinematics.yaml"
-    physical_parameters_file="$(arg physical_parameters_file)/$(arg name)/physical_parameters.yaml"
-    visual_parameters_file="$(arg visual_parameters_file)/$(arg name)/visual_parameters.yaml"
+    kinematics_parameters_file="$(arg kinematics_parameters_file)"
+    physical_parameters_file="$(arg physical_parameters_file)"
+    visual_parameters_file="$(arg visual_parameters_file)"
     use_fake_hardware="$(arg use_fake_hardware)"
     initial_positions="${xacro.load_yaml(initial_positions_file)}"
@@ -54,4 +55,8 @@
     <!-- tool changer-->
     <xacro:mtc_ur_tool_changer prefix="" connected_to="tool0" rotation="0" />
+  </xacro:if>
+  <!-- pinch geometry for moveit motion planning. see https://github.com/UniversalRobots/Universal_Robots_ROS2_Driver/issues/611 -->
+  <xacro:if value="$(arg use_pinch_link)">
+    <xacro:pinch_link prefix="" />
   </xacro:if>
   <!-- wrist camera adapter and camera-->
@@ -91,5 +96,5 @@
     <origin rpy="0 0 0" xyz="0 0 0" />
   </joint>
-  <!-- External Camera -->
+  <!-- Camera External -->
   <link name="external_camera_link" />
   <joint name="external_camera_joint" type="fixed">

Commit message: Add Objectives and Configuration for PickNik UR Robots (#18)
* add objectives from base config

* Update looping_pick_and_place_object.xml

* remove parenthesis

* Update objectives from main

* Add additional foundational controllers

* Update defaults and launch files

* Update base moveit configuration for UR5e robots

* Update base descriptions

* Update GZ objectives

* Add realsense high accuracy config file

* Fix path typos for UR description

* Adjust objective definition locations

* Add mock hardware flag

* Fix servo config

* Additional objective parameterization

* Update default compose file

* Remove overriding push button objective

* Remove tree nodes models

* Add additional waypoints for all base objectives

* Slow down default servo speed

* Fix more copyrights

* Add more waypoints for GZ config

* Screen output for gz config

* Update gz launch and site config

* Remove sensor data qos

* Fix paths

* Spawn scene vs spawn cabinet

* One more QoS

* Update gz waypoints

* Apply suggestions from code review

Co-authored-by: Sebastian Castro <4603398+sea-bass@users.noreply.github.com>

* Revert all non-critical changes to gz config

* Update src/picknik_ur_base_config/objectives/looping_pick_and_place_object.xml

Co-authored-by: Michael Wrock <mike.wrock@gmail.com>

* External <-> Camera

* Move Pick waypoint back

* Adjust stall params for GAC in GZ sim

* Fix whitespace

* Remove unused config yaml

* Remove unused servo param

* Sequences -> control ids

* Sequences -> control ids

---------

Co-authored-by: Erik Holum <erik.holum@picknik.ai>
Co-authored-by: Sebastian Castro <4603398+sea-bass@users.noreply.github.com>
Co-authored-by: Michael Wrock <mike.wrock@gmail.com>
Co-authored-by: Sebastian Castro <sebas.a.castro@gmail.com>

File: src/picknik_ur_base_config/description/picknik_ur5e.xacro (robot description, xacro)
@@ -2,7 +2,8 @@
 <robot xmlns:xacro="http://wiki.ros.org/xacro" name="$(arg name)">
   <!-- parameters -->
-  <xacro:arg name="use_fake_hardware" default="true" />
+  <xacro:arg name="use_fake_hardware" default="false" />
   <xacro:arg name="external_camera" default="false" />
   <xacro:arg name="has_tool_changer" default="true" />
+  <xacro:arg name="use_pinch_link" default="true" />
   <xacro:arg name="name" default="" />
   <xacro:arg name="joint_limits_parameters_file" default="" />
@@ -26,10 +27,10 @@
   <xacro:include filename="$(find picknik_accessories)/descriptions/sensors/realsense_d415.urdf.xacro" />
   <xacro:include filename="$(find picknik_accessories)/descriptions/sensors/realsense_d435.urdf.xacro" />
+  <xacro:include filename="$(find picknik_ur_base_config)/description/pinch_link.xacro" />
+  <!-- Initial positions for simulations (Mock Hardware and Gazebo) -->
+  <xacro:arg name="initial_positions_file" default="$(find picknik_ur_base_config)/config/initial_positions.yaml"/>
+  <xacro:property name="initial_positions_file" default="$(arg initial_positions_file)"/>
   <!-- Import environment macros -->
   <xacro:include filename="$(find picknik_accessories)/descriptions/geometry/collision_and_visual/cube_collision_and_visual.urdf.xacro" />
-  <!-- Initial positions for simulations (Mock Hardware and Gazebo) -->
-  <xacro:arg name="initial_positions_file" default="$(find picknik_ur_base_config)/config/initial_positions.yaml"/>
-  <!-- Convert args to properties for substitution in macros -->
-  <xacro:property name="initial_positions_file" default="$(arg initial_positions_file)"/>
   <link name="world" />
   <!-- arm -->
@@ -39,7 +40,7 @@
     parent="world"
     joint_limits_parameters_file="$(arg joint_limits_parameters_file)"
-    kinematics_parameters_file="$(arg kinematics_parameters_file)/$(arg name)/default_kinematics.yaml"
-    physical_parameters_file="$(arg physical_parameters_file)/$(arg name)/physical_parameters.yaml"
-    visual_parameters_file="$(arg visual_parameters_file)/$(arg name)/visual_parameters.yaml"
+    kinematics_parameters_file="$(arg kinematics_parameters_file)"
+    physical_parameters_file="$(arg physical_parameters_file)"
+    visual_parameters_file="$(arg visual_parameters_file)"
     use_fake_hardware="$(arg use_fake_hardware)"
     initial_positions="${xacro.load_yaml(initial_positions_file)}"
@@ -54,4 +55,8 @@
     <!-- tool changer-->
     <xacro:mtc_ur_tool_changer prefix="" connected_to="tool0" rotation="0" />
+  </xacro:if>
+  <!-- pinch geometry for moveit motion planning. see https://github.com/UniversalRobots/Universal_Robots_ROS2_Driver/issues/611 -->
+  <xacro:if value="$(arg use_pinch_link)">
+    <xacro:pinch_link prefix="" />
   </xacro:if>
   <!-- wrist camera adapter and camera-->

Commit message: Replace blue block with wood block

File: src/picknik_ur_base_config/description/picknik_ur5e.xacro (robot description, xacro)
@@ -33,4 +33,5 @@
   <!-- Import environment macros -->
   <xacro:include filename="$(find picknik_accessories)/descriptions/geometry/collision_and_visual/cube_collision_and_visual.urdf.xacro" />
+  <xacro:include filename="$(find picknik_accessories)/descriptions/geometry/collision_and_visual/cube_visual.urdf.xacro" />
   <link name="world" />
   <!-- arm -->
@@ -86,13 +87,21 @@
   <!-- Environment -->
   <link name="environment">
-    <!-- Table -->
-    <xacro:cube_collision_and_visual length="2.0" width="2.0" height="0.25" alpha="0.3">
-      <origin xyz="0 0 ${-0.25/2}" rpy="0 0 0" />
-    </xacro:cube_collision_and_visual>
+    <visual>
+      <origin xyz="0 0 0" rpy="0 0 0" />
+      <geometry>
+        <mesh filename="package://picknik_accessories/descriptions/furniture/generic_table/wood_block.dae" scale="0.5 0.5 0.1"/>
+      </geometry>
+    </visual>
+    <collision>
+      <origin rpy="0 0 0" xyz="0 0 0"/>
+      <geometry>
+        <mesh filename="package://picknik_accessories/descriptions/furniture/generic_table/wood_block.dae" scale="0.5 0.5 0.1"/>
+      </geometry>
+    </collision>
   </link>
-  <joint name="base_to_environment" type="fixed">
+  <joint name="table_joint" type="fixed">
     <parent link="base" />
     <child link="environment" />
-    <origin rpy="0 0 0" xyz="0 0 0" />
+    <origin rpy="0 0 0" xyz="0 0 -0.05" />
   </joint>
   <!-- External Camera -->

Commit message: Add cubes and waypoints

File: src/picknik_ur_base_config/description/picknik_ur5e.xacro (robot description, xacro)
@@ -105,4 +105,59 @@
     <origin rpy="0 0 0" xyz="0 0 -0.05" />
   </joint>
+  <link name="box_1">
+    <xacro:cube_visual length="0.05" width="0.05" height="0.05">
+      <origin xyz="0 0 0" rpy="0 0 0" />
+      <color rgba="0.1 0.1 0.1 0.9" />
+    </xacro:cube_visual>
+  </link>
+  <joint name="box1_on_table" type="fixed">
+    <parent link="environment" />
+    <child link="box_1" />
+    <origin rpy="0 0 0" xyz="0.65 -0.35 0.1" />
+  </joint>
+  <link name="box_2">
+    <xacro:cube_visual length="0.05" width="0.05" height="0.05">
+      <origin xyz="0 0 0" rpy="0 0 0" />
+      <color rgba="0.5 0.5 0.5 0.9" />
+    </xacro:cube_visual>
+  </link>
+  <joint name="box2_on_table" type="fixed">
+    <parent link="environment" />
+    <child link="box_2" />
+    <origin rpy="0 0 0" xyz="0.65 0.35 0.1" />
+  </joint>
+  <link name="box_3">
+    <xacro:cube_visual length="0.05" width="0.05" height="0.05">
+      <origin xyz="0 0 0" rpy="0 0 0" />
+      <color rgba="0.8 0.3 0.1 0.9" />
+    </xacro:cube_visual>
+  </link>
+  <joint name="box3_on_table" type="fixed">
+    <parent link="environment" />
+    <child link="box_3" />
+    <origin rpy="0 0 0" xyz="0.65 0 0.1" />
+  </joint>
+  <link name="box_4">
+    <xacro:cube_visual length="0.05" width="0.05" height="0.05">
+      <origin xyz="0 0 0" rpy="0 0 0" />
+      <color rgba="0.8 0.3 0.1 0.9" />
+    </xacro:cube_visual>
+  </link>
+  <joint name="box4_on_table" type="fixed">
+    <parent link="environment" />
+    <child link="box_4" />
+    <origin rpy="0 0 0" xyz="-0.65 0.25 0.1" />
+  </joint>
+  <link name="box_5">
+    <xacro:cube_visual length="0.05" width="0.05" height="0.05">
+      <origin xyz="0 0 0" rpy="0 0 0" />
+      <color rgba="0.1 0.3 0.8 0.9" />
+    </xacro:cube_visual>
+  </link>
+  <joint name="box5_on_table" type="fixed">
+    <parent link="environment" />
+    <child link="box_5" />
+    <origin rpy="0 0 0" xyz="-0.65 -0.25 0.1" />
+  </joint>
   <!-- External Camera -->
   <link name="external_camera_link" />

Commit message: Add wood texture and blocks to mock sim (#24)
* Replace blue block with wood block

* Fix link and gazebo xacro

* Add cubes and waypoints

File: src/picknik_ur_base_config/description/picknik_ur5e.xacro (robot description, xacro)
@@ -33,4 +33,5 @@
   <!-- Import environment macros -->
   <xacro:include filename="$(find picknik_accessories)/descriptions/geometry/collision_and_visual/cube_collision_and_visual.urdf.xacro" />
+  <xacro:include filename="$(find picknik_accessories)/descriptions/geometry/visual/cube_visual.urdf.xacro" />
   <link name="world" />
   <!-- arm -->
@@ -86,13 +87,76 @@
   <!-- Environment -->
   <link name="environment">
-    <!-- Table -->
-    <xacro:cube_collision_and_visual length="2.0" width="2.0" height="0.25" alpha="0.3">
-      <origin xyz="0 0 ${-0.25/2}" rpy="0 0 0" />
-    </xacro:cube_collision_and_visual>
+    <visual>
+      <origin xyz="0 0 0" rpy="0 0 0" />
+      <geometry>
+        <mesh filename="package://picknik_accessories/descriptions/furniture/generic_table/wood_block.dae" scale="0.5 0.5 0.1"/>
+      </geometry>
+    </visual>
+    <collision>
+      <origin rpy="0 0 0" xyz="0 0 0"/>
+      <geometry>
+        <mesh filename="package://picknik_accessories/descriptions/furniture/generic_table/wood_block.dae" scale="0.5 0.5 0.1"/>
+      </geometry>
+    </collision>
   </link>
-  <joint name="base_to_environment" type="fixed">
+  <joint name="table_joint" type="fixed">
     <parent link="base" />
     <child link="environment" />
-    <origin rpy="0 0 0" xyz="0 0 0" />
+    <origin rpy="0 0 0" xyz="0 0 -0.05" />
+  </joint>
+  <link name="box_1">
+    <xacro:cube_visual length="0.05" width="0.05" height="0.05">
+      <origin xyz="0 0 0" rpy="0 0 0" />
+      <color rgba="0.1 0.1 0.1 0.9" />
+    </xacro:cube_visual>
+  </link>
+  <joint name="box1_on_table" type="fixed">
+    <parent link="environment" />
+    <child link="box_1" />
+    <origin rpy="0 0 0" xyz="0.65 -0.35 0.1" />
+  </joint>
+  <link name="box_2">
+    <xacro:cube_visual length="0.05" width="0.05" height="0.05">
+      <origin xyz="0 0 0" rpy="0 0 0" />
+      <color rgba="0.5 0.5 0.5 0.9" />
+    </xacro:cube_visual>
+  </link>
+  <joint name="box2_on_table" type="fixed">
+    <parent link="environment" />
+    <child link="box_2" />
+    <origin rpy="0 0 0" xyz="0.65 0.35 0.1" />
+  </joint>
+  <link name="box_3">
+    <xacro:cube_visual length="0.05" width="0.05" height="0.05">
+      <origin xyz="0 0 0" rpy="0 0 0" />
+      <color rgba="0.8 0.3 0.1 0.9" />
+    </xacro:cube_visual>
+  </link>
+  <joint name="box3_on_table" type="fixed">
+    <parent link="environment" />
+    <child link="box_3" />
+    <origin rpy="0 0 0" xyz="0.65 0 0.1" />
+  </joint>
+  <link name="box_4">
+    <xacro:cube_visual length="0.05" width="0.05" height="0.05">
+      <origin xyz="0 0 0" rpy="0 0 0" />
+      <color rgba="0.8 0.3 0.1 0.9" />
+    </xacro:cube_visual>
+  </link>
+  <joint name="box4_on_table" type="fixed">
+    <parent link="environment" />
+    <child link="box_4" />
+    <origin rpy="0 0 0" xyz="-0.65 0.25 0.1" />
+  </joint>
+  <link name="box_5">
+    <xacro:cube_visual length="0.05" width="0.05" height="0.05">
+      <origin xyz="0 0 0" rpy="0 0 0" />
+      <color rgba="0.1 0.3 0.8 0.9" />
+    </xacro:cube_visual>
+  </link>
+  <joint name="box5_on_table" type="fixed">
+    <parent link="environment" />
+    <child link="box_5" />
+    <origin rpy="0 0 0" xyz="-0.65 -0.25 0.1" />
   </joint>
   <!-- External Camera -->

Commit message: Reduce table block size in mock sim

File: src/picknik_ur_base_config/description/picknik_ur5e.xacro (robot description, xacro)
@@ -90,5 +90,5 @@
       <origin xyz="0 0 0" rpy="0 0 0" />
       <geometry>
-        <mesh filename="package://picknik_accessories/descriptions/furniture/generic_table/wood_block.dae" scale="0.5 0.5 0.1"/>
+        <mesh filename="package://picknik_accessories/descriptions/furniture/generic_table/wood_block.dae" scale="0.25 0.25 0.1"/>
       </geometry>
     </visual>
@@ -96,5 +96,5 @@
       <origin rpy="0 0 0" xyz="0 0 0"/>
       <geometry>
-        <mesh filename="package://picknik_accessories/descriptions/furniture/generic_table/wood_block.dae" scale="0.5 0.5 0.1"/>
+        <mesh filename="package://picknik_accessories/descriptions/furniture/generic_table/wood_block.dae" scale="0.25 0.25 0.1"/>
       </geometry>
     </collision>
