Commit message: Lengthened pinch link and added tool_changer_link to its excluded collisions

File: src/picknik_ur_base_config/description/pinch_link.xacro (robot description, xacro)
@@ -2,5 +2,5 @@
 <robot xmlns:xacro="http://ros.org/wiki/xacro">
   <!-- radius of wrist_2_link/forearm_link is ~0.045m. Actual offset of this is (radius - attached_link's radius) -->
-  <xacro:macro name="pinch_link" params="prefix:='' connected_to:='forearm_link' length:=0.25 radius:=0.055">
+  <xacro:macro name="pinch_link" params="prefix:='' connected_to:='forearm_link' length:=0.30 radius:=0.055">
     <xacro:property name="prefix_" value='${prefix + "_" if prefix else ""}' />
     <link name="pinch_link">
@@ -24,5 +24,5 @@
       <parent link="${connected_to}"/>
       <child link="pinch_link"/>
-      <origin xyz="${-0.09 - length/2} 0 0.0049" rpy="0 ${pi/2} 0" />
+      <origin xyz="${-0.08 - length/2} 0 0.0049" rpy="0 ${pi/2} 0" />
     </joint>
   </xacro:macro>

Commit message: Made pinch link wider

File: src/picknik_ur_base_config/description/pinch_link.xacro (robot description, xacro)
@@ -2,5 +2,5 @@
 <robot xmlns:xacro="http://ros.org/wiki/xacro">
   <!-- radius of wrist_2_link/forearm_link is ~0.045m. Actual offset of this is (radius - attached_link's radius) -->
-  <xacro:macro name="pinch_link" params="prefix:='' connected_to:='forearm_link' length:=0.30 radius:=0.055">
+  <xacro:macro name="pinch_link" params="prefix:='' connected_to:='forearm_link' length:=0.30 radius:=0.065">
     <xacro:property name="prefix_" value='${prefix + "_" if prefix else ""}' />
     <link name="pinch_link">

Commit message: Widen pinch link

File: src/picknik_ur_base_config/description/pinch_link.xacro (robot description, xacro)
@@ -2,5 +2,5 @@
 <robot xmlns:xacro="http://ros.org/wiki/xacro">
   <!-- radius of wrist_2_link/forearm_link is ~0.045m. Actual offset of this is (radius - attached_link's radius) -->
-  <xacro:macro name="pinch_link" params="prefix:='' connected_to:='forearm_link' length:=0.30 radius:=0.065">
+  <xacro:macro name="pinch_link" params="prefix:='' connected_to:='forearm_link' length:=0.30 radius:=0.07">
     <xacro:property name="prefix_" value='${prefix + "_" if prefix else ""}' />
     <link name="pinch_link">

Commit message: Make pinch link slightly narrower and slightly less long

File: src/picknik_ur_base_config/description/pinch_link.xacro (robot description, xacro)
@@ -2,5 +2,5 @@
 <robot xmlns:xacro="http://ros.org/wiki/xacro">
   <!-- radius of wrist_2_link/forearm_link is ~0.045m. Actual offset of this is (radius - attached_link's radius) -->
-  <xacro:macro name="pinch_link" params="prefix:='' connected_to:='forearm_link' length:=0.30 radius:=0.07">
+  <xacro:macro name="pinch_link" params="prefix:='' connected_to:='forearm_link' length:=0.28 radius:=0.0675">
     <xacro:property name="prefix_" value='${prefix + "_" if prefix else ""}' />
     <link name="pinch_link">
