Commit message: Update wrist_3 pinch link

File: src/picknik_ur_base_config/description/pinch_links.xacro (robot description, xacro)
@@ -29,5 +29,5 @@
     </joint>
   </xacro:macro>
-  <xacro:macro name="wrist_3_pinch_link" params="prefix:='' length:=0.11 offset:=0.015">
+  <xacro:macro name="wrist_3_pinch_link" params="prefix:='' length:=0.15 offset:=0.015">
     <xacro:property name="prefix_" value='${prefix + "_" if prefix else ""}' />
     <xacro:property name="radius" value='${0.0375 + offset}' />
@@ -52,5 +52,5 @@
       <parent link="wrist_3_link"/>
       <child link="${prefix_}wrist_3_pinch_link"/>
-      <origin xyz="0.01 0 0" rpy="0 0 0" />
+      <origin xyz="0 0 0.015" rpy="0 0 0" />
     </joint>
   </xacro:macro>

Commit message: Fixed placement of wrist_3 pinch link

File: src/picknik_ur_base_config/description/pinch_links.xacro (robot description, xacro)
@@ -29,5 +29,5 @@
     </joint>
   </xacro:macro>
-  <xacro:macro name="wrist_3_pinch_link" params="prefix:='' length:=0.15 offset:=0.015">
+  <xacro:macro name="wrist_3_pinch_link" params="prefix:='' length:=0.11 offset:=0.015">
     <xacro:property name="prefix_" value='${prefix + "_" if prefix else ""}' />
     <xacro:property name="radius" value='${0.0375 + offset}' />
@@ -52,5 +52,5 @@
       <parent link="wrist_3_link"/>
       <child link="${prefix_}wrist_3_pinch_link"/>
-      <origin xyz="0 0 0.015" rpy="0 0 0" />
+      <origin xyz="0 0 0" rpy="0 0 0" />
     </joint>
   </xacro:macro>

Commit message: Added missing prefix

File: src/picknik_ur_base_config/description/pinch_links.xacro (robot description, xacro)
@@ -24,5 +24,5 @@
     </link>
     <joint name="${prefix_}forearm_pinch_joint" type="fixed">
-      <parent link="forearm_link"/>
+      <parent link="${prefix_}forearm_link"/>
       <child link="${prefix_}forearm_pinch_link"/>
       <origin xyz="${-0.08 - length/2} 0 0.0049" rpy="0 ${pi/2} 0" />
@@ -50,5 +50,5 @@
     </link>
     <joint name="${prefix_}wrist_3_pinch_joint" type="fixed">
-      <parent link="wrist_3_link"/>
+      <parent link="${prefix_}wrist_3_link"/>
       <child link="${prefix_}wrist_3_pinch_link"/>
       <origin xyz="0 0 0" rpy="0 0 0" />

Commit message: Reduce diameter of pinch links just barely and perturb yaw of links so the cylinder approximations don't have jutting edges towards each other

File: src/picknik_ur_base_config/description/pinch_links.xacro (robot description, xacro)
@@ -3,10 +3,10 @@
   <!-- wrist_3_link/forearm_link have a radius 0f 0.0375m. Actual offset from surface is (radius - attached_link's radius). -->
   <!-- UR Drivers check for a 2.5cm  distance between tool_flange/wrist_3 and forearm links. -->
-  <xacro:macro name="forearm_pinch_link" params="prefix:='' length:=0.28 offset:=0.015">
+  <xacro:macro name="forearm_pinch_link" params="prefix:='' length:=0.28 offset:=0.0125">
     <xacro:property name="prefix_" value='${prefix + "_" if prefix else ""}' />
     <xacro:property name="radius" value='${0.0375 + offset}' />
     <link name="${prefix_}forearm_pinch_link">
       <visual>
-        <origin xyz="0 0 0" rpy="0 0 0"/>
+        <origin xyz="0 0 0" rpy="0 0 ${pi/16}"/>
         <geometry>
           <cylinder length="${length}" radius="${radius}"/>
@@ -17,5 +17,5 @@
       </visual>
       <collision>
-        <origin xyz="0 0 0" rpy="0 0 0"/>
+        <origin xyz="0 0 0" rpy="0 0 ${pi/16"/>
         <geometry>
             <cylinder length="${length}" radius="${radius}"/>
@@ -29,5 +29,5 @@
     </joint>
   </xacro:macro>
-  <xacro:macro name="wrist_3_pinch_link" params="prefix:='' length:=0.11 offset:=0.015">
+  <xacro:macro name="wrist_3_pinch_link" params="prefix:='' length:=0.11 offset:=0.0125">
     <xacro:property name="prefix_" value='${prefix + "_" if prefix else ""}' />
     <xacro:property name="radius" value='${0.0375 + offset}' />
@@ -52,5 +52,5 @@
       <parent link="${prefix_}wrist_3_link"/>
       <child link="${prefix_}wrist_3_pinch_link"/>
-      <origin xyz="0 0 0" rpy="0 0 0" />
+      <origin xyz="0 0 0" rpy="0 0 ${pi/16}" />
     </joint>
   </xacro:macro>

Commit message: Closing bracket.

File: src/picknik_ur_base_config/description/pinch_links.xacro (robot description, xacro)
@@ -17,5 +17,5 @@
       </visual>
       <collision>
-        <origin xyz="0 0 0" rpy="0 0 ${pi/16"/>
+        <origin xyz="0 0 0" rpy="0 0 ${pi/16}"/>
         <geometry>
             <cylinder length="${length}" radius="${radius}"/>

Commit message: Use different sizes for each pinch link to hopefully help with planning

File: src/picknik_ur_base_config/description/pinch_links.xacro (robot description, xacro)
@@ -3,5 +3,5 @@
   <!-- wrist_3_link/forearm_link have a radius 0f 0.0375m. Actual offset from surface is (radius - attached_link's radius). -->
   <!-- UR Drivers check for a 2.5cm  distance between tool_flange/wrist_3 and forearm links. -->
-  <xacro:macro name="forearm_pinch_link" params="prefix:='' length:=0.28 offset:=0.0125">
+  <xacro:macro name="forearm_pinch_link" params="prefix:='' length:=0.28 offset:=0.0175">
     <xacro:property name="prefix_" value='${prefix + "_" if prefix else ""}' />
     <xacro:property name="radius" value='${0.0375 + offset}' />
@@ -29,5 +29,5 @@
     </joint>
   </xacro:macro>
-  <xacro:macro name="wrist_3_pinch_link" params="prefix:='' length:=0.11 offset:=0.0125">
+  <xacro:macro name="wrist_3_pinch_link" params="prefix:='' length:=0.11 offset:=0.075">
     <xacro:property name="prefix_" value='${prefix + "_" if prefix else ""}' />
     <xacro:property name="radius" value='${0.0375 + offset}' />

Commit message: Add missing 0 throwing off radius

File: src/picknik_ur_base_config/description/pinch_links.xacro (robot description, xacro)
@@ -29,5 +29,5 @@
     </joint>
   </xacro:macro>
-  <xacro:macro name="wrist_3_pinch_link" params="prefix:='' length:=0.11 offset:=0.075">
+  <xacro:macro name="wrist_3_pinch_link" params="prefix:='' length:=0.11 offset:=0.0075">
     <xacro:property name="prefix_" value='${prefix + "_" if prefix else ""}' />
     <xacro:property name="radius" value='${0.0375 + offset}' />

Commit message: Update to make wrist pinch link slightly bigger and forearm slightly smaller

File: src/picknik_ur_base_config/description/pinch_links.xacro (robot description, xacro)
@@ -3,5 +3,5 @@
   <!-- wrist_3_link/forearm_link have a radius 0f 0.0375m. Actual offset from surface is (radius - attached_link's radius). -->
   <!-- UR Drivers check for a 2.5cm  distance between tool_flange/wrist_3 and forearm links. -->
-  <xacro:macro name="forearm_pinch_link" params="prefix:='' length:=0.28 offset:=0.0175">
+  <xacro:macro name="forearm_pinch_link" params="prefix:='' length:=0.28 offset:=0.015">
     <xacro:property name="prefix_" value='${prefix + "_" if prefix else ""}' />
     <xacro:property name="radius" value='${0.0375 + offset}' />
@@ -29,5 +29,5 @@
     </joint>
   </xacro:macro>
-  <xacro:macro name="wrist_3_pinch_link" params="prefix:='' length:=0.11 offset:=0.0075">
+  <xacro:macro name="wrist_3_pinch_link" params="prefix:='' length:=0.11 offset:=0.01">
     <xacro:property name="prefix_" value='${prefix + "_" if prefix else ""}' />
     <xacro:property name="radius" value='${0.0375 + offset}' />

Commit message: Alphabetize srdf more. Update pinch links size to correctly pass tests.

File: src/picknik_ur_base_config/description/pinch_links.xacro (robot description, xacro)
@@ -29,5 +29,5 @@
     </joint>
   </xacro:macro>
-  <xacro:macro name="wrist_3_pinch_link" params="prefix:='' length:=0.11 offset:=0.01">
+  <xacro:macro name="wrist_3_pinch_link" params="prefix:='' length:=0.11 offset:=0.015">
     <xacro:property name="prefix_" value='${prefix + "_" if prefix else ""}' />
     <xacro:property name="radius" value='${0.0375 + offset}' />

Commit message: Make wrist pinch link slightly smaller for better planning

File: src/picknik_ur_base_config/description/pinch_links.xacro (robot description, xacro)
@@ -29,5 +29,5 @@
     </joint>
   </xacro:macro>
-  <xacro:macro name="wrist_3_pinch_link" params="prefix:='' length:=0.11 offset:=0.015">
+  <xacro:macro name="wrist_3_pinch_link" params="prefix:='' length:=0.11 offset:=0.012">
     <xacro:property name="prefix_" value='${prefix + "_" if prefix else ""}' />
     <xacro:property name="radius" value='${0.0375 + offset}' />
