Commit message: Update paths for our 2f_85 gripper URDF

File: src/picknik_ur_base_config/description/robotiq_2f_85_gripper.urdf (robot description, URDF)
Before this commit: robot ur5e_gripper_and_camera, 28 links, 27 joints
Links:
- link robotiq_85_base_link: geometry collision mesh filename=package://robotiq_description/meshes/collision/2f_85/roboti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; visual mesh filename=package://robotiq_description/meshes/visual/2f_85/robotiq_b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
- link robotiq_85_left_finger_link: geometry collision mesh filename=package://robotiq_description/meshes/collision/2f_85/left_f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; visual mesh filename=package://robotiq_description/meshes/visual/2f_85/left_fing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
- link robotiq_85_left_finger_tip_link: geometry collision mesh filename=package://robotiq_description/meshes/collision/2f_85/left_f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; visual mesh filename=package://robotiq_description/meshes/visual/2f_85/left_fing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
- link robotiq_85_left_inner_knuckle_link: geometry collision mesh filename=package://robotiq_description/meshes/collision/2f_85/left_i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; visual mesh filename=package://robotiq_description/meshes/visual/2f_85/left_inne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
- link robotiq_85_left_knuckle_link: geometry collision mesh filename=package://robotiq_description/meshes/collision/2f_85/left_k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; visual mesh filename=package://robotiq_description/meshes/visual/2f_85/left_knuc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
- link robotiq_85_right_finger_link: geometry collision mesh filename=package://robotiq_description/meshes/collision/2f_85/right_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; visual mesh filename=package://robotiq_description/meshes/visual/2f_85/right_fin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
- link robotiq_85_right_finger_tip_link: geometry collision mesh filename=package://robotiq_description/meshes/collision/2f_85/right_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; visual mesh filename=package://robotiq_description/meshes/visual/2f_85/right_fin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
- link robotiq_85_right_inner_knuckle_link: geometry collision mesh filename=package://robotiq_description/meshes/collision/2f_85/right_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; visual mesh filename=package://robotiq_description/meshes/visual/2f_85/right_inn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
- link robotiq_85_right_knuckle_link: geometry collision mesh filename=package://robotiq_description/meshes/collision/2f_85/right_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; visual mesh filename=package://robotiq_description/meshes/visual/2f_85/right_knu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
- link ur_to_robotiq_link: geometry collision mesh filename=package://robotiq_description/meshes/collision/2f_85/ur_to_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; visual mesh filename=package://robotiq_description/meshes/visual/2f_85/ur_to_rob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
