Commit message: Remove manual_grasp_link

File: src/picknik_ur_base_config/description/gripper_and_camera.xacro (robot description, xacro)
@@ -7,11 +7,11 @@
   <xacro:include filename="$(find picknik_accessories)/descriptions/sensors/realsense_d415.urdf.xacro"/>
   <!-- Create base link -->
-  <!-- Moveit Studio requires a link name called manual_grasp_link to perform built-in Objectives such as inspect surface without modification. -->
-  <link name="manual_grasp_link" />
+  <!-- We use a link name called grasp_link to perform built-in Objectives such as inspect surface without modification. -->
+  <link name="grasp_link"/>
   <link name="tool0" />
   <joint name="flange-tool0" type="fixed">
-    <parent link="manual_grasp_link" />
+    <parent link="grasp_link" />
     <child link="tool0" />
-    <origin xyz="0.0 -0.016124 -0.18430" rpy="${pi / 180.0 * 5} 0 -${pi}" />
+    <origin xyz="0 -0.016124 -0.18430" rpy="0 0 -${pi}" />
   </joint>
   <link name="tool_changer_tool0" />

File: src/picknik_ur_base_config/description/picknik_ur.xacro (robot description, xacro)
@@ -84,11 +84,4 @@
     <child link="grasp_link" />
     <origin xyz="0.0 0.0 0.134" rpy="0.0 0.0 ${pi}" />
-  </joint>
-  <!-- Moveit Studio requires a link name called manual_grasp_link to perform quick tasks such as inspect surface -->
-  <link name="manual_grasp_link" />
-  <joint name="manual_grasp_joint" type="fixed">
-    <parent link="grasp_link" />
-    <child link="manual_grasp_link" />
-    <origin xyz="0 0 0" rpy="${pi / 180.0 * 5} 0 0" />
   </joint>
   <!-- Environment -->

File: src/picknik_ur_base_config/description/robotiq_2f_85_gripper.urdf (robot description, URDF)
Before this commit: robot ur5e_gripper_and_camera, 28 links, 27 joints
Links:
- removed link manual_grasp_link
- added link grasp_link
Joints:
- joint flange-tool0: origin xyz=0.0 -0.016124 -0.18430 rpy=0.08726646259971647 0 -3.141592653589793 -> xyz=0.0 -0.016124 -0.18430 rpy=0 0 -3.141592653589793; parent manual_grasp_link -> grasp_link

File: src/picknik_ur_gazebo_config/config/moveit/picknik_ur_gazebo.srdf.xacro (robot description, xacro)
@@ -13,5 +13,5 @@
     <!--SUBGROUPS: Groups can also be formed by referencing to already defined group names-->
     <group name="manipulator">
-        <chain base_link="base_link" tip_link="manual_grasp_link"/>
+        <chain base_link="base_link" tip_link="grasp_link"/>
     </group>
     <group name="gripper">

File: src/picknik_ur_gazebo_config/description/picknik_ur_gazebo.xacro (robot description, xacro)
@@ -58,11 +58,4 @@
     <child link="grasp_link" />
     <origin xyz="0.0 0.0 0.134" rpy="0.0 0.0 ${pi}" />
-  </joint>
-  <!-- Moveit Studio requires a link name called manual_grasp_link to perform quick tasks such as inspect surface -->
-  <link name="manual_grasp_link" />
-  <joint name="manual_grasp_joint" type="fixed">
-    <parent link="grasp_link" />
-    <child link="manual_grasp_link" />
-    <origin xyz="0 0 0" rpy="${pi / 180.0 * 5} 0 0" />
   </joint>
   <!-- Environment -->

File: src/picknik_ur_mock_hw_config/description/picknik_ur_machine_tending.xacro (robot description, xacro)
@@ -74,11 +74,4 @@
     <child link="grasp_link" />
     <origin xyz="0.0 0.0 0.134" rpy="0.0 0.0 ${pi}" />
-  </joint>
-  <!-- Moveit Studio requires a link name called manual_grasp_link to perform quick tasks such as inspect surface -->
-  <link name="manual_grasp_link" />
-  <joint name="manual_grasp_joint" type="fixed">
-    <parent link="grasp_link" />
-    <child link="manual_grasp_link" />
-    <origin xyz="0 0 0" rpy="${pi / 180.0 * 5} 0 0" />
   </joint>
   <!-- CNC machine -->
