Commit message: use yaml substitution instead of xacro logic
Signed-off-by: Paul Gesel <paulgesel@gmail.com>

File: src/picknik_ur_base_config/description/picknik_ur_macro.xacro (robot description, xacro)
@@ -34,15 +34,4 @@
         <xacro:property name="simulation" default="$(arg simulation)"/>
         <xacro:property name="visual_parameters_file" default="$(arg visual_parameters_file)"/>
-        <xacro:if value="${not visual_parameters_file == ''}">
-            <xacro:property name="visual_parameters_file_full_path" default="$(arg visual_parameters_file)/$(arg name)/visual_parameters.yaml"/>
-        </xacro:if>
-        <xacro:property name="physical_parameters_file" default="$(arg physical_parameters_file)"/>
-        <xacro:if value="${not physical_parameters_file == ''}">
-            <xacro:property name="physical_parameters_file_full_path" default="$(arg physical_parameters_file)/$(arg name)/physical_parameters.yaml"/>
-        </xacro:if>
-        <xacro:property name="kinematics_parameters_file" default="$(arg kinematics_parameters_file)"/>
-        <xacro:if value="${not kinematics_parameters_file == ''}">
-            <xacro:property name="kinematics_parameters_file_full_path" default="$(arg kinematics_parameters_file)/$(arg name)/default_kinematics.yaml"/>
-        </xacro:if>
         <xacro:if value="${simulation == 'gazebo'}">
             <xacro:property name="use_fake_hardware" default="false"/>
@@ -58,7 +47,7 @@
                 parent="${parent}"
                 joint_limits_parameters_file="$(arg joint_limits_parameters_file)"
-                kinematics_parameters_file="${kinematics_parameters_file_full_path}"
-                physical_parameters_file="${physical_parameters_file_full_path}"
-                visual_parameters_file="${visual_parameters_file_full_path}"
+                kinematics_parameters_file="$(arg kinematics_parameters_file)"
+                physical_parameters_file="$(arg physical_parameters_file)"
+                visual_parameters_file="$(arg visual_parameters_file)"
                 use_fake_hardware="${use_fake_hardware}"
                 initial_positions="${xacro.load_yaml(initial_positions_file)}"

Commit message: Fix UR location for mock hw

File: src/picknik_ur_base_config/description/picknik_ur_macro.xacro (robot description, xacro)
@@ -55,5 +55,5 @@
                 output_recipe_filename="$(find ur_robot_driver)/resources/rtde_output_recipe.txt"
                 input_recipe_filename="$(find ur_robot_driver)/resources/rtde_input_recipe.txt">
-            <origin xyz="0 0 0" rpy="0 0 0"/>
+            <origin xyz="0 0 0" rpy="0 0 1.57"/>
         </xacro:ur_robot>
         <xacro:unless value="$(arg has_tool_changer)">

Commit message: Use pi/2

File: src/picknik_ur_base_config/description/picknik_ur_macro.xacro (robot description, xacro)
@@ -55,5 +55,5 @@
                 output_recipe_filename="$(find ur_robot_driver)/resources/rtde_output_recipe.txt"
                 input_recipe_filename="$(find ur_robot_driver)/resources/rtde_input_recipe.txt">
-            <origin xyz="0 0 0" rpy="0 0 1.57"/>
+            <origin xyz="0 0 0" rpy="0 0 ${pi/2}"/>
         </xacro:ur_robot>
         <xacro:unless value="$(arg has_tool_changer)">

Commit message: Make origin a macro param

File: src/picknik_ur_base_config/description/picknik_ur_macro.xacro (robot description, xacro)
@@ -1,5 +1,5 @@
 <?xml version="1.0" encoding="utf-8"?>
 <robot xmlns:xacro="http://ros.org/wiki/xacro">
-    <xacro:macro name="picknik_ur" params="parent child initial_positions_file">
+    <xacro:macro name="picknik_ur" params="parent child initial_positions_file *origin">
         <!-- parameters -->
         <xacro:arg name="use_fake_hardware" default="false"/>
@@ -55,5 +55,9 @@
                 output_recipe_filename="$(find ur_robot_driver)/resources/rtde_output_recipe.txt"
                 input_recipe_filename="$(find ur_robot_driver)/resources/rtde_input_recipe.txt">
+<<<<<<< Updated upstream
             <origin xyz="0 0 0" rpy="0 0 ${pi/2}"/>
+=======
+            <xacro:insert_block name="origin" />
+>>>>>>> Stashed changes
         </xacro:ur_robot>
         <xacro:unless value="$(arg has_tool_changer)">

File: src/picknik_ur_gazebo_config/description/picknik_ur_gazebo.xacro (robot description, xacro)
@@ -26,5 +26,7 @@
   <xacro:include filename="$(arg environment_xacro)"/>
   <!-- Robot: contains robot description from the world frame to the tool frame -->
-  <xacro:picknik_ur parent="world"  child="tool0" initial_positions_file="$(arg initial_positions_file)" />
+  <xacro:picknik_ur parent="world"  child="tool0" initial_positions_file="$(arg initial_positions_file)">
+    <origin xyz="0 0 0" rpy="0 0 0" />
+  </xacro:picknik_ur>
   <!-- Gripper and UR adapter and realsense camera -->
   <xacro:picknik_ur_attachments parent="tool0" child="grasp_link" has_tool_changer="$(arg has_tool_changer)"/>

File: src/picknik_ur_mock_hw_config/description/picknik_ur_machine_tending.xacro (robot description, xacro)
@@ -23,5 +23,7 @@
     <xacro:include filename="$(arg environment_xacro)"/>
     <!-- Robot: contains robot description from the world frame to the tool frame -->
-    <xacro:picknik_ur parent="world"  child="tool0" initial_positions_file="$(arg initial_positions_file)" />
+    <xacro:picknik_ur parent="world"  child="tool0" initial_positions_file="$(arg initial_positions_file)">
+      <origin xyz="0 0 0" rpy="0 0 ${pi/2}" />
+    </xacro:picknik_ur>
     <!-- Gripper and UR adapter and realsense camera -->
     <xacro:picknik_ur_attachments parent="tool0" child="grasp_link" has_tool_changer="$(arg has_tool_changer)"/>

Commit message: Resolve conflict

File: src/picknik_ur_base_config/description/picknik_ur_macro.xacro (robot description, xacro)
@@ -55,9 +55,5 @@
                 output_recipe_filename="$(find ur_robot_driver)/resources/rtde_output_recipe.txt"
                 input_recipe_filename="$(find ur_robot_driver)/resources/rtde_input_recipe.txt">
-<<<<<<< Updated upstream
-            <origin xyz="0 0 0" rpy="0 0 ${pi/2}"/>
-=======
             <xacro:insert_block name="origin" />
->>>>>>> Stashed changes
         </xacro:ur_robot>
         <xacro:unless value="$(arg has_tool_changer)">

Commit message: Fix UR location for Mock HW (#236)

File: src/picknik_ur_base_config/description/picknik_ur_macro.xacro (robot description, xacro)
@@ -1,5 +1,5 @@
 <?xml version="1.0" encoding="utf-8"?>
 <robot xmlns:xacro="http://ros.org/wiki/xacro">
-    <xacro:macro name="picknik_ur" params="parent child initial_positions_file">
+    <xacro:macro name="picknik_ur" params="parent child initial_positions_file *origin">
         <!-- parameters -->
         <xacro:arg name="use_fake_hardware" default="false"/>
@@ -55,5 +55,5 @@
                 output_recipe_filename="$(find ur_robot_driver)/resources/rtde_output_recipe.txt"
                 input_recipe_filename="$(find ur_robot_driver)/resources/rtde_input_recipe.txt">
-            <origin xyz="0 0 0" rpy="0 0 0"/>
+            <xacro:insert_block name="origin" />
         </xacro:ur_robot>
         <xacro:unless value="$(arg has_tool_changer)">
