Commit message: convert gazebo
Signed-off-by: Paul Gesel <paulgesel@gmail.com>

File: src/picknik_ur_base_config/description/picknik_ur_attachments_macro.xacro (robot description, xacro)
@@ -2,4 +2,6 @@
 <robot xmlns:xacro="http://ros.org/wiki/xacro">
     <xacro:macro name="picknik_ur_attachments" params="parent child has_tool_changer">
+        <!-- parameters -->
+        <xacro:arg name="simulation" default=""/>
         <xacro:include filename="$(find picknik_accessories)/descriptions/brackets/ur_realsense_camera_adapter/picknik_ur_camera_adapter.urdf.xacro"/>
         <xacro:include filename="$(find picknik_accessories)/descriptions/sensors/realsense_d415.urdf.xacro"/>
@@ -17,5 +19,6 @@
         <!-- wrist camera adapter and camera-->
         <xacro:ur_realsense_camera_adapter prefix="" parent="${ur_realsense_camera_adapter_parent}" child_tool="realsense_camera_adapter_tool0" child_camera="d415_mount_link" rotation="0"/>
-        <xacro:realsense_d415 parent="d415_mount_link" name="wrist_mounted_camera">
+        <xacro:property name="simulation" default="$(arg simulation)"/>
+        <xacro:realsense_d415 parent="d415_mount_link" name="wrist_mounted_camera" use_mesh="${simulation == 'gazebo'}">
             <origin xyz="0 0 0" rpy="0 0 0"/>
         </xacro:realsense_d415>

File: src/picknik_ur_base_config/description/picknik_ur_macro.xacro (robot description, xacro)
@@ -17,4 +17,5 @@
         <xacro:arg name="tool_voltage" default="0"/>
         <xacro:arg name="tool_device_name" default="/dev/ttyUSB0"/>
+        <xacro:arg name="simulation" default=""/>
         <xacro:if value="$(arg has_tool_changer)">
             <xacro:property name="camera_adapter_parent" value="tool_changer_tool0"/>
@@ -31,4 +32,5 @@
         <!-- Initial positions for simulations (Mock Hardware and Gazebo) -->
         <xacro:property name="initial_positions_file" default="$(arg initial_positions_file)"/>
+        <xacro:property name="simulation" default="$(arg simulation)"/>
         <link name="${parent}"/>
         <!-- arm -->
@@ -43,4 +45,5 @@
                 use_fake_hardware="$(arg use_fake_hardware)"
                 initial_positions="${xacro.load_yaml(initial_positions_file)}"
+                sim_ignition="${simulation == 'gazebo'}"
                 headless_mode="$(arg headless_mode)"
                 robot_ip="$(arg robot_ip)"

File: src/picknik_ur_gazebo_config/description/picknik_ur_gazebo.xacro (robot description, xacro)
@@ -2,170 +2,32 @@
 <robot xmlns:xacro="http://wiki.ros.org/xacro" name="$(arg name)">
   <!-- parameters -->
-  <xacro:arg name="name" default="" />
-  <xacro:arg name="joint_limits_parameters_file" default="" />
-  <xacro:arg name="kinematics_parameters_file" default="" />
-  <xacro:arg name="physical_parameters_file" default="" />
-  <xacro:arg name="visual_parameters_file" default="" />
+  <xacro:arg name="use_fake_hardware" default="false"/>
+  <xacro:arg name="external_camera" default="false"/>
+  <xacro:arg name="has_tool_changer" default="true"/>
+  <xacro:arg name="use_pinch_links" default="true"/>
+  <xacro:arg name="name" default=""/>
+  <xacro:arg name="joint_limits_parameters_file" default=""/>
+  <xacro:arg name="kinematics_parameters_file" default=""/>
+  <xacro:arg name="physical_parameters_file" default=""/>
+  <xacro:arg name="visual_parameters_file" default=""/>
+  <xacro:arg name="headless_mode" default="false"/>
+  <xacro:arg name="robot_ip" default="0.0.0.0"/>
+  <xacro:arg name="use_tool_communication" default="false"/>
+  <xacro:arg name="tool_voltage" default="0"/>
+  <xacro:arg name="tool_device_name" default="/dev/ttyUSB0"/>
+  <xacro:arg name="initial_positions_file" default="$(find picknik_ur_base_config)/config/initial_positions.yaml"/>
+  <xacro:arg name="environment_xacro" default="$(find picknik_ur_gazebo_config)/description/environment.xacro"/>
+  <xacro:arg name="simulation" default="gazebo"/>
+  <xacro:arg name="gazebo_renderer" default="ogre"/>
   <xacro:arg name="use_extra_camera" default="false"/>
-  <xacro:arg name="gazebo_renderer" default="ogre"/>
-  <!-- Import macros for main hardware components -->
-  <xacro:include filename="$(find ur_description)/urdf/ur_macro.xacro" />
-  <xacro:include filename="$(find robotiq_description)/urdf/ur_to_robotiq_adapter.urdf.xacro" />
-  <xacro:include filename="$(find robotiq_description)/urdf/robotiq_2f_85_macro.urdf.xacro" />
-  <xacro:include filename="$(find picknik_accessories)/descriptions/brackets/mtc_ur_tool_changer/mtc_ur_tool_changer.urdf.xacro" />
-  <xacro:include filename="$(find picknik_accessories)/descriptions/brackets/ur_realsense_camera_adapter/picknik_ur_camera_adapter.urdf.xacro" />
-  <xacro:include filename="$(find picknik_accessories)/descriptions/sensors/realsense_d415.urdf.xacro" />
-  <xacro:include filename="$(find picknik_accessories)/descriptions/sensors/realsense_d435.urdf.xacro" />
-  <!-- Import environment macros -->
-  <xacro:include filename="$(find picknik_accessories)/descriptions/geometry/collision_and_visual/cube_collision_and_visual.urdf.xacro" />
-  <!-- initial position for simulations (Fake Hardware and Gazebo) -->
-  <xacro:arg name="initial_positions_file" default="$(find picknik_ur_base_config)/config/initial_positions.yaml"/>
-  <!-- convert to properties to use substitution in function -->
-  <xacro:property name="initial_positions_file" default="$(arg initial_positions_file)"/>
-  <xacro:property name="gazebo_renderer" default="$(arg gazebo_renderer)"/>
-  <!-- create link fixed to the "world" -->
-  <link name="world" />
-  <!-- arm -->
-  <xacro:ur_robot
-    name="$(arg name)"
-    tf_prefix=""
-    parent="world"
-    joint_limits_parameters_file="$(arg joint_limits_parameters_file)"
-    kinematics_parameters_file="$(arg kinematics_parameters_file)/$(arg name)/default_kinematics.yaml"
-    physical_parameters_file="$(arg physical_parameters_file)/$(arg name)/physical_parameters.yaml"
-    visual_parameters_file="$(arg visual_parameters_file)/$(arg name)/visual_parameters.yaml"
-    sim_ignition="true"
-    initial_positions="${xacro.load_yaml(initial_positions_file)}">
-    <origin xyz="0 0 0" rpy="0 0 0" /> <!-- position robot in the world -->
-  </xacro:ur_robot>
-  <!-- tool changer-->
-  <xacro:mtc_ur_tool_changer prefix="" connected_to="tool0" rotation="0" />
-  <!-- wrist camera adapter and camera-->
-  <xacro:ur_realsense_camera_adapter prefix="" connected_to="tool_changer_tool0" rotation="0" />
-  <!-- TODO: With ogre renderer and use_mesh="true",
-  the camera image will be obstructed by the mesh-->
-  <xacro:realsense_d415 parent="d415_mount_link" name="wrist_mounted_camera" use_mesh="${gazebo_renderer == 'ogre2'}">
-    <origin xyz="0 0 0" rpy="0 0 0" />
-  </xacro:realsense_d415>
-  <!-- Gripper and UR adapter-->
-  <xacro:ur_to_robotiq prefix="" connected_to="realsense_camera_adapter_tool0" rotation="0" />
-  <xacro:robotiq_gripper name="RobotiqGripperHardwareInterface" prefix="" parent="gripper_mount_link" sim_ignition="true">
-    <origin xyz="0 0 0" rpy="0 0 0" />
-  </xacro:robotiq_gripper>
-  <link name="grasp_link" />
-  <joint name="grasp_link_joint" type="fixed">
-    <parent link="robotiq_85_base_link" />
-    <child link="grasp_link" />
-    <origin xyz="0.0 0.0 0.134" rpy="0.0 0.0 ${pi}" />
-  </joint>
-  <!-- Environment -->
-  <link name="environment">
-    <!-- Table -->
-    <xacro:cube_collision_and_visual length="1.5" width="1.0" height="0.25">
-      <origin rpy="0 0 0" xyz="0 0 ${-0.25/2}" />
-      <color rgba="0 0 1 0" />
-    </xacro:cube_collision_and_visual>
-  </link>
-  <joint name="base_to_environment" type="fixed">
-    <parent link="base" />
-    <child link="environment" />
-    <origin rpy="0 0 0" xyz="0 0 0" />
-  </joint>
-  <!-- External camera -->
-  <link name="external_camera_link" />
-  <joint name="external_camera_joint" type="fixed">
-    <parent link="world" />
-    <child link="external_camera_link" />
-    <origin xyz="1.1 -1.1 1.3" rpy="0.0 0.4 2.4" />
-  </joint>
-  <xacro:realsense_d435 parent="external_camera_link" name="scene_camera" visible="false" simulate_depth="true">
-    <origin xyz="0 0 0" rpy="0 0 0" />
-  </xacro:realsense_d435>
-  <!-- Additional Camera -->
-  <xacro:if value="$(arg use_extra_camera)">
-    <link name="extra_scene_camera_link" />
-    <joint name="extra_scene_camera_joint" type="fixed">
-      <parent link="world" />
-      <child link="extra_scene_camera_link" />
-      <origin xyz="-0.3 0.3 0.5" rpy="0.0 0.0 -3.14" />
-    </joint>
-    <xacro:realsense_d435 parent="extra_scene_camera_link" name="extra_camera" visible="false" simulate_depth="false">
-      <origin xyz="0 0 0" rpy="0 0 0" />
-    </xacro:realsense_d435>
-  </xacro:if>
-  <!-- Force/Torque Sensor -->
-  <link name="robot/wrist_3_joint/force_torque_sensor" />
-  <joint name="wrist_to_fts" type="fixed">
-    <parent link="wrist_3_link" />
-    <child link="robot/wrist_3_joint/force_torque_sensor" />
-    <origin rpy="0 0 0" xyz="0 0 0" />
-  </joint>
-  <gazebo reference="wrist_3_joint">
-    <sensor name="tcp_fts_sensor" type="force_torque">
-      <always_on>1</always_on>
-      <update_rate>50</update_rate>
-      <visualize>0</visualize>
-      <topic>tcp_fts_sensor/ft_data</topic>
-      <pose>0 0 0 0 0 0</pose>
-      <force_torque>
-        <frame>child</frame>
-        <measure_direction>parent_to_child</measure_direction>
-        <force>
-          <x>
-            <noise type="gaussian">
-              <mean>0</mean>
-              <stddev>0</stddev>
-            </noise>
-          </x>
-          <y>
-            <noise type="gaussian">
-              <mean>0</mean>
-              <stddev>0</stddev>
-            </noise>
-          </y>
-          <z>
-            <noise type="gaussian">
-              <mean>0</mean>
-              <stddev>0</stddev>
-            </noise>
-          </z>
-        </force>
-        <torque>
-          <x>
-            <noise type="gaussian">
-              <mean>0</mean>
-              <stddev>0</stddev>
-            </noise>
-          </x>
-          <y>
-            <noise type="gaussian">
-              <mean>0</mean>
-              <stddev>0</stddev>
-            </noise>
-          </y>
-          <z>
-            <noise type="gaussian">
-              <mean>0</mean>
-              <stddev>0</stddev>
-            </noise>
-          </z>
-        </torque>
-      </force_torque>
-    </sensor>
-  </gazebo>
-  <!-- Gazebo Plugins -->
-  <gazebo>
-    <plugin filename="ign_ros2_control-system" name="ign_ros2_control::IgnitionROS2ControlPlugin">
-      <parameters>$(find picknik_ur_gazebo_config)/config/control/picknik_ur5e.ros2_control.yaml</parameters>
-      <ros>
-        <remapping>/servo_controller/commands:=/robot_controllers/commands</remapping>
-        <remapping>/servo_controller/joint_trajectory:=/robot_controllers/joint_trajectory</remapping>
-      </ros>
-    </plugin>
-  </gazebo>
-  <gazebo>
-    <plugin filename="libignition-gazebo-sensors-system.so" name="ignition::gazebo::systems::Sensors">
-      <render_engine>${gazebo_renderer}</render_engine>
-    </plugin>
-  </gazebo>
+  <!-- Import UR and environment macros -->
+  <xacro:include filename="$(find picknik_ur_base_config)/description/picknik_ur_macro.xacro"/>
+  <xacro:include filename="$(find picknik_ur_base_config)/description/picknik_ur_attachments_macro.xacro"/>
+  <xacro:include filename="$(arg environment_xacro)"/>
+  <!-- Robot: contains robot description from the world frame to the tool frame -->
+  <xacro:picknik_ur parent="world"  child="tool0" initial_positions_file="$(arg initial_positions_file)" />
+  <!-- Gripper and UR adapter and realsense camera -->
+  <xacro:picknik_ur_attachments parent="tool0" child="grasp_link" has_tool_changer="$(arg has_tool_changer)"/>
+  <!-- Environment: contains scene geometry and external sensors, e.g. cameras -->
+  <xacro:environment parent="world"/>
 </robot>

Commit message: fix fake hardware gazebo issue
Signed-off-by: Paul Gesel <paulgesel@gmail.com>

File: src/picknik_ur_base_config/description/picknik_ur_attachments_macro.xacro (robot description, xacro)
@@ -24,6 +24,14 @@
         </xacro:realsense_d415>
         <xacro:ur_to_robotiq prefix="" parent="realsense_camera_adapter_tool0" child="gripper_mount_link" rotation="0"/>
+        <xacro:if value="${simulation == 'gazebo'}">
+            <xacro:property name="use_fake_hardware" default="false"/>
+            <xacro:property name="sim_ignition" default="true"/>
+        </xacro:if>
+        <xacro:if value="${not simulation == 'gazebo'}">
+            <xacro:property name="use_fake_hardware" default="(arg use_fake_hardware)"/>
+            <xacro:property name="sim_ignition" default="false"/>
+        </xacro:if>
         <xacro:robotiq_gripper name="RobotiqGripperHardwareInterface" prefix=""
-                               parent="gripper_mount_link" use_fake_hardware="$(arg use_fake_hardware)"
+                               parent="gripper_mount_link" use_fake_hardware="${use_fake_hardware}" sim_ignition="${sim_ignition}"
                                com_port="$(arg tool_device_name)">
             <origin xyz="0 0 0" rpy="0 0 0"/>

File: src/picknik_ur_base_config/description/picknik_ur_macro.xacro (robot description, xacro)
@@ -33,4 +33,22 @@
         <xacro:property name="initial_positions_file" default="$(arg initial_positions_file)"/>
         <xacro:property name="simulation" default="$(arg simulation)"/>
+        <xacro:property name="visual_parameters_file" default="$(arg visual_parameters_file)"/>
+        <xacro:if value="${not visual_parameters_file == ''}">
+            <xacro:property name="visual_parameters_file_full_path" default="$(arg visual_parameters_file)/$(arg name)/visual_parameters.yaml"/>
+        </xacro:if>
+        <xacro:property name="physical_parameters_file" default="$(arg physical_parameters_file)"/>
+        <xacro:if value="${not physical_parameters_file == ''}">
+            <xacro:property name="physical_parameters_file_full_path" default="$(arg physical_parameters_file)/$(arg name)/physical_parameters.yaml"/>
+        </xacro:if>
+        <xacro:property name="kinematics_parameters_file" default="$(arg kinematics_parameters_file)"/>
+        <xacro:if value="${not kinematics_parameters_file == ''}">
+            <xacro:property name="kinematics_parameters_file_full_path" default="$(arg kinematics_parameters_file)/$(arg name)/default_kinematics.yaml"/>
+        </xacro:if>
+        <xacro:if value="${simulation == 'gazebo'}">
+            <xacro:property name="use_fake_hardware" default="false"/>
+        </xacro:if>
+        <xacro:if value="${not simulation == 'gazebo'}">
+            <xacro:property name="use_fake_hardware" default="(arg use_fake_hardware)"/>
+        </xacro:if>
         <link name="${parent}"/>
         <!-- arm -->
@@ -40,8 +58,8 @@
                 parent="${parent}"
                 joint_limits_parameters_file="$(arg joint_limits_parameters_file)"
-                kinematics_parameters_file="$(arg kinematics_parameters_file)"
-                physical_parameters_file="$(arg physical_parameters_file)"
-                visual_parameters_file="$(arg visual_parameters_file)"
-                use_fake_hardware="$(arg use_fake_hardware)"
+                kinematics_parameters_file="${kinematics_parameters_file_full_path}"
+                physical_parameters_file="${physical_parameters_file_full_path}"
+                visual_parameters_file="${visual_parameters_file_full_path}"
+                use_fake_hardware="${use_fake_hardware}"
                 initial_positions="${xacro.load_yaml(initial_positions_file)}"
                 sim_ignition="${simulation == 'gazebo'}"

Commit message: add missing $
Signed-off-by: Paul Gesel <paulgesel@gmail.com>

File: src/picknik_ur_base_config/description/picknik_ur_attachments_macro.xacro (robot description, xacro)
@@ -29,5 +29,5 @@
         </xacro:if>
         <xacro:if value="${not simulation == 'gazebo'}">
-            <xacro:property name="use_fake_hardware" default="(arg use_fake_hardware)"/>
+            <xacro:property name="use_fake_hardware" default="$(arg use_fake_hardware)"/>
             <xacro:property name="sim_ignition" default="false"/>
         </xacro:if>

File: src/picknik_ur_base_config/description/picknik_ur_macro.xacro (robot description, xacro)
@@ -38,5 +38,5 @@
         </xacro:if>
         <xacro:if value="${not simulation == 'gazebo'}">
-            <xacro:property name="use_fake_hardware" default="(arg use_fake_hardware)"/>
+            <xacro:property name="use_fake_hardware" default="$(arg use_fake_hardware)"/>
         </xacro:if>
         <link name="${parent}"/>

Commit message: use gazebo_renderer to set use_mesh
Signed-off-by: Paul Gesel <paulgesel@gmail.com>

File: src/picknik_ur_base_config/description/picknik_ur_attachments_macro.xacro (robot description, xacro)
@@ -19,9 +19,10 @@
         <!-- wrist camera adapter and camera-->
         <xacro:ur_realsense_camera_adapter prefix="" parent="${ur_realsense_camera_adapter_parent}" child_tool="realsense_camera_adapter_tool0" child_camera="d415_mount_link" rotation="0"/>
-        <xacro:property name="simulation" default="$(arg simulation)"/>
-        <xacro:realsense_d415 parent="d415_mount_link" name="wrist_mounted_camera" use_mesh="${not simulation == 'gazebo'}">
+        <xacro:property name="gazebo_renderer" default="$(arg gazebo_renderer)"/>
+        <xacro:realsense_d415 parent="d415_mount_link" name="wrist_mounted_camera" use_mesh="${not gazebo_renderer == 'ogre'}">
             <origin xyz="0 0 0" rpy="0 0 0"/>
         </xacro:realsense_d415>
         <xacro:ur_to_robotiq prefix="" parent="realsense_camera_adapter_tool0" child="gripper_mount_link" rotation="0"/>
+        <xacro:property name="simulation" default="$(arg simulation)"/>
         <xacro:if value="${simulation == 'gazebo'}">
             <xacro:property name="use_fake_hardware" default="false"/>

File: src/picknik_ur_base_config/description/picknik_ur_macro.xacro (robot description, xacro)
@@ -18,4 +18,5 @@
         <xacro:arg name="tool_device_name" default="/dev/ttyUSB0"/>
         <xacro:arg name="simulation" default=""/>
+        <xacro:arg name="gazebo_renderer" default=""/>
         <xacro:if value="$(arg has_tool_changer)">
             <xacro:property name="camera_adapter_parent" value="tool_changer_tool0"/>

Commit message: Revert "use gazebo_renderer to set use_mesh"
This reverts commit d041f47b60935d5f2a5a861b5c924ad7436edc0f.

File: src/picknik_ur_base_config/description/picknik_ur_attachments_macro.xacro (robot description, xacro)
@@ -19,10 +19,9 @@
         <!-- wrist camera adapter and camera-->
         <xacro:ur_realsense_camera_adapter prefix="" parent="${ur_realsense_camera_adapter_parent}" child_tool="realsense_camera_adapter_tool0" child_camera="d415_mount_link" rotation="0"/>
-        <xacro:property name="gazebo_renderer" default="$(arg gazebo_renderer)"/>
-        <xacro:realsense_d415 parent="d415_mount_link" name="wrist_mounted_camera" use_mesh="${not gazebo_renderer == 'ogre'}">
+        <xacro:property name="simulation" default="$(arg simulation)"/>
+        <xacro:realsense_d415 parent="d415_mount_link" name="wrist_mounted_camera" use_mesh="${not simulation == 'gazebo'}">
             <origin xyz="0 0 0" rpy="0 0 0"/>
         </xacro:realsense_d415>
         <xacro:ur_to_robotiq prefix="" parent="realsense_camera_adapter_tool0" child="gripper_mount_link" rotation="0"/>
-        <xacro:property name="simulation" default="$(arg simulation)"/>
         <xacro:if value="${simulation == 'gazebo'}">
             <xacro:property name="use_fake_hardware" default="false"/>

File: src/picknik_ur_base_config/description/picknik_ur_macro.xacro (robot description, xacro)
@@ -18,5 +18,4 @@
         <xacro:arg name="tool_device_name" default="/dev/ttyUSB0"/>
         <xacro:arg name="simulation" default=""/>
-        <xacro:arg name="gazebo_renderer" default=""/>
         <xacro:if value="$(arg has_tool_changer)">
             <xacro:property name="camera_adapter_parent" value="tool_changer_tool0"/>
