Commit message: Address review

File: src/picknik_ur_base_config/description/picknik_ur_attachments_macro.xacro (robot description, xacro)
@@ -1,5 +1,7 @@
 <?xml version="1.0" encoding="utf-8"?>
 <robot xmlns:xacro="http://ros.org/wiki/xacro">
-    <xacro:macro name="picknik_ur_attachments" params="parent child has_tool_changer">
+    <xacro:macro name="picknik_ur_attachments" params="prefix:='' parent child has_tool_changer">
+        <!-- prefix property -->
+        <xacro:property name="prefix_" value='${prefix + "_" if prefix else ""}' />
         <!-- parameters -->
         <xacro:arg name="simulation" default=""/>
@@ -11,6 +13,6 @@
         <!-- tool changer-->
         <xacro:if value="$(arg has_tool_changer)">
-            <xacro:mtc_ur_tool_changer prefix="" parent="${parent}" child="tool_changer_tool0" rotation="0"/>
-            <xacro:property name="ur_realsense_camera_adapter_parent" value="tool_changer_tool0" />
+            <xacro:mtc_ur_tool_changer prefix="${prefix_}" parent="${parent}" child="${prefix_}tool_changer_tool0" rotation="0"/>
+            <xacro:property name="ur_realsense_camera_adapter_parent" value="${prefix_}tool_changer_tool0" />
         </xacro:if>
         <xacro:unless value="$(arg has_tool_changer)">
@@ -18,10 +20,11 @@
         </xacro:unless>
         <!-- wrist camera adapter and camera-->
-        <xacro:ur_realsense_camera_adapter prefix="" parent="${ur_realsense_camera_adapter_parent}" child_tool="realsense_camera_adapter_tool0" child_camera="d415_mount_link" rotation="0"/>
+        <xacro:ur_realsense_camera_adapter prefix="${prefix_}" parent="${ur_realsense_camera_adapter_parent}" child_tool="${prefix_}realsense_camera_adapter_tool0" child_camera="${prefix_}d415_mount_link" rotation="0"/>
         <xacro:property name="simulation" default="$(arg simulation)"/>
-        <xacro:realsense_d415 parent="d415_mount_link" name="wrist_mounted_camera" use_mesh="${not simulation == 'gazebo'}">
+        <xacro:realsense_d415 parent="${prefix_}d415_mount_link" name="${prefix_}wrist_mounted_camera" use_mesh="${not simulation == 'gazebo'}">
             <origin xyz="0 0 0" rpy="0 0 0"/>
         </xacro:realsense_d415>
-        <xacro:ur_to_robotiq prefix="" parent="realsense_camera_adapter_tool0" child="gripper_mount_link" rotation="0"/>
+        <!-- gripper and UR adapter-->
+        <xacro:ur_to_robotiq prefix="${prefix_}" parent="${prefix_}realsense_camera_adapter_tool0" child="${prefix_}gripper_mount_link" rotation="0"/>
         <xacro:if value="${simulation == 'gazebo'}">
             <xacro:property name="use_fake_hardware" default="false"/>
@@ -32,6 +35,6 @@
             <xacro:property name="sim_ignition" default="false"/>
         </xacro:if>
-        <xacro:robotiq_gripper name="RobotiqGripperHardwareInterface" prefix=""
-                               parent="gripper_mount_link" use_fake_hardware="${use_fake_hardware}" sim_ignition="${sim_ignition}"
+        <xacro:robotiq_gripper name="${prefix_}RobotiqGripperHardwareInterface" prefix="${prefix_}"
+                               parent="${prefix_}gripper_mount_link" use_fake_hardware="${use_fake_hardware}" sim_ignition="${sim_ignition}"
                                com_port="$(arg tool_device_name)">
             <origin xyz="0 0 0" rpy="0 0 0"/>
@@ -40,5 +43,5 @@
         <link name="${child}"/>
         <joint name="${child}_joint" type="fixed">
-            <parent link="robotiq_85_base_link"/>
+            <parent link="${prefix_}robotiq_85_base_link"/>
             <child link="${child}"/>
             <origin xyz="0.0 0.0 0.134" rpy="0.0 0.0 ${pi}"/>

File: src/picknik_ur_multi_arm_config/description/dual_arm_ur.xacro (robot description, xacro)
@@ -13,4 +13,7 @@
   <xacro:arg name="headless_mode" default="false" />
   <xacro:arg name="robot_ip" default="0.0.0.0" />
+  <xacro:arg name="use_tool_communication" default="false"/>
+  <xacro:arg name="tool_voltage" default="0"/>
+  <xacro:arg name="tool_device_name" default="/dev/ttyUSB0"/>
   <xacro:if value="$(arg has_tool_changer)">
     <xacro:property name="camera_adapter_parent" value="tool_changer_tool0" />
@@ -22,5 +25,5 @@
   <xacro:include filename="$(find ur_description)/urdf/ur_macro.xacro" />
   <xacro:include filename="$(find picknik_ur_multi_arm_config)/description/pinch_links.xacro" />
-  <xacro:include filename="$(find picknik_ur_multi_arm_config)/description/picknik_ur_attachments.xacro" />
+  <xacro:include filename="$(find picknik_ur_base_config)/description/picknik_ur_attachments_macro.xacro" />
   <xacro:include filename="$(find picknik_accessories)/descriptions/sensors/realsense_d435.urdf.xacro" />
   <!-- Initial positions for simulations (Mock Hardware and Gazebo) -->
@@ -53,8 +56,6 @@
     prefix="left"
     parent="left_tool0"
+    child="left_grasp_link"
     has_tool_changer="$(arg has_tool_changer)"
-    use_pinch_links="$(arg use_pinch_links)"
-    use_fake_hardware="$(arg use_fake_hardware)"
-    gripper_com_port="$/dev/ttyUSB0"
   />
   <!-- RIGHT ROBOT -->
@@ -80,8 +81,6 @@
     prefix="right"
     parent="right_tool0"
+    child="right_grasp_link"
     has_tool_changer="$(arg has_tool_changer)"
-    use_pinch_links="$(arg use_pinch_links)"
-    use_fake_hardware="$(arg use_fake_hardware)"
-    gripper_com_port="$/dev/ttyUSB0"
   />
   <!-- ENVIRONMENT -->

Commit message: Add dual arm configuration (#231)
---------

Co-authored-by: Sebastian Castro <4603398+sea-bass@users.noreply.github.com>

File: src/picknik_ur_base_config/description/picknik_ur_attachments_macro.xacro (robot description, xacro)
@@ -1,16 +1,18 @@
 <?xml version="1.0" encoding="utf-8"?>
 <robot xmlns:xacro="http://ros.org/wiki/xacro">
-    <xacro:macro name="picknik_ur_attachments" params="parent child has_tool_changer">
+    <xacro:include filename="$(find picknik_accessories)/descriptions/brackets/ur_realsense_camera_adapter/picknik_ur_camera_adapter.urdf.xacro"/>
+    <xacro:include filename="$(find picknik_accessories)/descriptions/sensors/realsense_d415.urdf.xacro"/>
+    <xacro:include filename="$(find robotiq_description)/urdf/ur_to_robotiq_adapter.urdf.xacro" />
+    <xacro:include filename="$(find robotiq_description)/urdf/robotiq_2f_85_macro.urdf.xacro" />
+    <xacro:include filename="$(find picknik_accessories)/descriptions/brackets/mtc_ur_tool_changer/mtc_ur_tool_changer.urdf.xacro"/>
+    <xacro:macro name="picknik_ur_attachments" params="prefix:='' parent child has_tool_changer">
+        <!-- prefix property -->
+        <xacro:property name="prefix_" value='${prefix + "_" if prefix else ""}' />
         <!-- parameters -->
         <xacro:arg name="simulation" default=""/>
-        <xacro:include filename="$(find picknik_accessories)/descriptions/brackets/ur_realsense_camera_adapter/picknik_ur_camera_adapter.urdf.xacro"/>
-        <xacro:include filename="$(find picknik_accessories)/descriptions/sensors/realsense_d415.urdf.xacro"/>
-        <xacro:include filename="$(find robotiq_description)/urdf/ur_to_robotiq_adapter.urdf.xacro" />
-        <xacro:include filename="$(find robotiq_description)/urdf/robotiq_2f_85_macro.urdf.xacro" />
-        <xacro:include filename="$(find picknik_accessories)/descriptions/brackets/mtc_ur_tool_changer/mtc_ur_tool_changer.urdf.xacro"/>
         <!-- tool changer-->
         <xacro:if value="$(arg has_tool_changer)">
-            <xacro:mtc_ur_tool_changer prefix="" parent="${parent}" child="tool_changer_tool0" rotation="0"/>
-            <xacro:property name="ur_realsense_camera_adapter_parent" value="tool_changer_tool0" />
+            <xacro:mtc_ur_tool_changer prefix="${prefix_}" parent="${parent}" child="${prefix_}tool_changer_tool0" rotation="0"/>
+            <xacro:property name="ur_realsense_camera_adapter_parent" value="${prefix_}tool_changer_tool0" />
         </xacro:if>
         <xacro:unless value="$(arg has_tool_changer)">
@@ -18,10 +20,11 @@
         </xacro:unless>
         <!-- wrist camera adapter and camera-->
-        <xacro:ur_realsense_camera_adapter prefix="" parent="${ur_realsense_camera_adapter_parent}" child_tool="realsense_camera_adapter_tool0" child_camera="d415_mount_link" rotation="0"/>
+        <xacro:ur_realsense_camera_adapter prefix="${prefix_}" parent="${ur_realsense_camera_adapter_parent}" child_tool="${prefix_}realsense_camera_adapter_tool0" child_camera="${prefix_}d415_mount_link" rotation="0"/>
         <xacro:property name="simulation" default="$(arg simulation)"/>
-        <xacro:realsense_d415 parent="d415_mount_link" name="wrist_mounted_camera" use_mesh="${not simulation == 'gazebo'}">
+        <xacro:realsense_d415 parent="${prefix_}d415_mount_link" name="${prefix_}wrist_mounted_camera" use_mesh="${not simulation == 'gazebo'}">
             <origin xyz="0 0 0" rpy="0 0 0"/>
         </xacro:realsense_d415>
-        <xacro:ur_to_robotiq prefix="" parent="realsense_camera_adapter_tool0" child="gripper_mount_link" rotation="0"/>
+        <!-- gripper and UR adapter-->
+        <xacro:ur_to_robotiq prefix="${prefix_}" parent="${prefix_}realsense_camera_adapter_tool0" child="${prefix_}gripper_mount_link" rotation="0"/>
         <xacro:if value="${simulation == 'gazebo'}">
             <xacro:property name="use_fake_hardware" default="false"/>
@@ -32,6 +35,6 @@
             <xacro:property name="sim_ignition" default="false"/>
         </xacro:if>
-        <xacro:robotiq_gripper name="RobotiqGripperHardwareInterface" prefix=""
-                               parent="gripper_mount_link" use_fake_hardware="${use_fake_hardware}" sim_ignition="${sim_ignition}"
+        <xacro:robotiq_gripper name="${prefix_}RobotiqGripperHardwareInterface" prefix="${prefix_}"
+                               parent="${prefix_}gripper_mount_link" use_fake_hardware="${use_fake_hardware}" sim_ignition="${sim_ignition}"
                                com_port="$(arg tool_device_name)">
             <origin xyz="0 0 0" rpy="0 0 0"/>
@@ -40,5 +43,5 @@
         <link name="${child}"/>
         <joint name="${child}_joint" type="fixed">
-            <parent link="robotiq_85_base_link"/>
+            <parent link="${prefix_}robotiq_85_base_link"/>
             <child link="${child}"/>
             <origin xyz="0.0 0.0 0.134" rpy="0.0 0.0 ${pi}"/>
