Commit message: Fix description for site config

File: src/picknik_ur_base_config/description/picknik_ur.xacro (robot description, xacro)
@@ -23,5 +23,7 @@
   <xacro:include filename="$(arg environment_xacro)"/>
   <!-- Robot: contains robot description from the world frame to the tool frame -->
-  <xacro:picknik_ur parent="world"  child="tool0" initial_positions_file="$(arg initial_positions_file)" />
+  <xacro:picknik_ur parent="world"  child="tool0" initial_positions_file="$(arg initial_positions_file)" >
+    <origin xyz="0 0 0" rpy="0 0 0" />
+  </xacro:picknik_ur>
   <!-- Gripper and UR adapter and realsense camera -->
   <xacro:picknik_ur_attachments parent="tool0" child="grasp_link" has_tool_changer="$(arg has_tool_changer)"/>

Commit message: Initial commit

File: src/picknik_ur_base_config/description/picknik_ur.xacro (robot description, xacro)
@@ -6,4 +6,5 @@
   <xacro:arg name="has_tool_changer" default="true"/>
   <xacro:arg name="use_pinch_links" default="true"/>
+  <xacro:arg name="generate_ros2_control_tag" default="true"/>
   <xacro:arg name="name" default=""/>
   <xacro:arg name="joint_limits_parameters_file" default=""/>
@@ -17,5 +18,4 @@
   <xacro:arg name="tool_device_name" default="/dev/ttyUSB0"/>
   <xacro:arg name="initial_positions_file" default="$(find picknik_ur_base_config)/config/initial_positions.yaml"/>
-  <xacro:arg name="environment_xacro" default="$(find picknik_ur_base_config)/description/environment.xacro"/>
   <!-- Import UR and environment macros -->
   <xacro:include filename="$(find picknik_ur_base_config)/description/picknik_ur_macro.xacro"/>
@@ -23,10 +23,8 @@
   <xacro:include filename="$(arg environment_xacro)"/>
   <!-- Robot: contains robot description from the world frame to the tool frame -->
-  <xacro:picknik_ur parent="world"  child="tool0" initial_positions_file="$(arg initial_positions_file)" >
+  <xacro:picknik_ur parent="world"  child="tool0" initial_positions_file="$(arg initial_positions_file)" generate_ros2_control_tag="$(arg generate_ros2_control_tag)" >
     <origin xyz="0 0 0" rpy="0 0 0" />
   </xacro:picknik_ur>
   <!-- Gripper and UR adapter and realsense camera -->
   <xacro:picknik_ur_attachments parent="tool0" child="grasp_link" has_tool_changer="$(arg has_tool_changer)"/>
-  <!-- Environment: contains scene geometry and external sensors, e.g. cameras -->
-  <xacro:environment parent="world"/>
 </robot>

File: src/picknik_ur_base_config/description/picknik_ur_macro.xacro (robot description, xacro)
@@ -1,5 +1,5 @@
 <?xml version="1.0" encoding="utf-8"?>
 <robot xmlns:xacro="http://ros.org/wiki/xacro">
-    <xacro:macro name="picknik_ur" params="parent child initial_positions_file *origin">
+    <xacro:macro name="picknik_ur" params="parent child initial_positions_file generate_ros2_control_tag *origin">
         <!-- parameters -->
         <xacro:arg name="use_fake_hardware" default="false"/>
@@ -7,4 +7,5 @@
         <xacro:arg name="has_tool_changer" default="true"/>
         <xacro:arg name="use_pinch_links" default="true"/>
+        <xacro:arg name="generate_ros2_control_tag" default="true"/>
         <xacro:arg name="name" default=""/>
         <xacro:arg name="joint_limits_parameters_file" default=""/>
@@ -44,5 +45,5 @@
                 physical_parameters_file="$(arg physical_parameters_file)"
                 visual_parameters_file="$(arg visual_parameters_file)"
-                use_fake_hardware="${use_fake_hardware}"
+                use_fake_hardware="false"
                 initial_positions="${xacro.load_yaml(initial_positions_file)}"
                 sim_ignition="${simulation == 'gazebo'}"
@@ -50,4 +51,5 @@
                 robot_ip="$(arg robot_ip)"
                 use_tool_communication="$(arg use_tool_communication)"
+                generate_ros2_control_tag="$(arg generate_ros2_control_tag)"
                 tool_voltage="$(arg tool_voltage)"
                 tool_device_name="$(arg tool_device_name)"

File: src/picknik_ur_gazebo_config/description/picknik_ur_gazebo.xacro (robot description, xacro)
@@ -6,4 +6,5 @@
   <xacro:arg name="has_tool_changer" default="true"/>
   <xacro:arg name="use_pinch_links" default="true"/>
+  <xacro:arg name="generate_ros2_control_tag" default="true"/>
   <xacro:arg name="name" default=""/>
   <xacro:arg name="joint_limits_parameters_file" default=""/>
@@ -30,5 +31,5 @@
   </xacro:picknik_ur>
   <!-- Gripper and UR adapter and realsense camera -->
-  <xacro:picknik_ur_attachments parent="tool0" child="grasp_link" has_tool_changer="$(arg has_tool_changer)"/>
+  <xacro:picknik_ur_attachments parent="tool0" child="grasp_link" has_tool_changer="$(arg has_tool_changer)" generate_ros2_control_tag="$(arg generate_ros2_control_tag)"/>
   <!-- Environment: contains scene geometry and external sensors, e.g. cameras -->
   <xacro:environment parent="world"/>
