Commit message: update objective
Signed-off-by: Paul Gesel <paulgesel@gmail.com>

File: src/picknik_ur_gazebo_peg_in_hole/config/moveit/picknik_ur_gazebo.srdf.xacro (robot description, xacro)
@@ -26,4 +26,8 @@
         <link name="$(arg gripper_name)_right_finger_link"/>
         <joint name="$(arg gripper_name)_left_knuckle_joint"/>
+        <joint name="peg_link_joint"/>
+        <joint name="peg_tip_link_joint"/>
+        <link name="peg_tip_link"/>
+        <link name="peg_link"/>
     </group>
     <!--GROUP STATES: Purpose: Define a named state for a particular group, in terms of joint values. This is useful to define states like 'folded arms'-->
