Commit message: find gazebo_renderer tag
Signed-off-by: Paul Gesel <paulgesel@gmail.com>

File: src/picknik_ur_gazebo_config/description/environment.xacro (robot description, xacro)
@@ -2,7 +2,4 @@
 <robot xmlns:xacro="http://ros.org/wiki/xacro">
   <xacro:macro name="environment" params="parent">
-    <!-- parameters -->
-    <xacro:arg name="gazebo_renderer" default="ogre"/>
-    <xacro:property name="gazebo_renderer" default="$(arg gazebo_renderer)"/>
     <!-- Import environment macros -->
     <xacro:include filename="$(find picknik_accessories)/descriptions/geometry/collision_and_visual/cube_collision_and_visual.urdf.xacro" />

File: src/picknik_ur_gazebo_config/description/picknik_ur_gazebo.xacro (robot description, xacro)
@@ -101,4 +101,5 @@
     </plugin>
   </gazebo>
+  <xacro:property name="gazebo_renderer" default="$(arg gazebo_renderer)"/>
   <gazebo>
     <plugin filename="libignition-gazebo-sensors-system.so" name="ignition::gazebo::systems::Sensors">
