Commit message: Move switch panel outside robot URDF, add Push Button

File: src/picknik_ur_gazebo_config/description/picknik_ur_gazebo.xacro (robot description, xacro)
@@ -19,5 +19,4 @@
   <!-- Import environment macros -->
   <xacro:include filename="$(find picknik_accessories)/descriptions/geometry/collision_and_visual/cube_collision_and_visual.urdf.xacro" />
-  <xacro:include filename="$(find picknik_accessories)/descriptions/furniture/switch_panel/switch_panel.urdf.xacro"/>
   <!-- initial position for simulations (Fake Hardware, Gazebo, Ignition) -->
   <xacro:arg name="initial_positions_file" default="$(find picknik_ur_gazebo_config)/config/initial_positions.yaml"/>
@@ -79,7 +78,4 @@
     <origin rpy="0 0 0" xyz="0 0 0" />
   </joint>
-  <xacro:picknik_switch_panel parent="world" >
-    <origin xyz="-0.8 0.0 0" rpy="0 0 -0.44"/>
-  </xacro:picknik_switch_panel>
   <!-- External camera -->
   <link name="external_camera_link" />

Commit message: Camera scene zoomed out and rotated.

File: src/picknik_ur_gazebo_config/description/picknik_ur_gazebo.xacro (robot description, xacro)
@@ -84,5 +84,5 @@
     <parent link="world" />
     <child link="external_camera_link" />
-    <origin xyz="0.3 -0.3 1.0" rpy="0.0 0.4 3.14" />
+    <origin xyz="1.1 -1.1 1.3" rpy="0.0 0.4 2.4" />
   </joint>
   <xacro:realsense_d435 parent="external_camera_link" name="scene_camera" visible="false" simulate_depth="true">

Commit message: Simulation with four cameras.

File: src/picknik_ur_gazebo_config/description/picknik_ur_gazebo.xacro (robot description, xacro)
@@ -16,5 +16,5 @@
   <xacro:include filename="$(find picknik_accessories)/descriptions/brackets/ur_realsense_camera_adapter/picknik_ur_camera_adapter.urdf.xacro" />
   <xacro:include filename="$(find picknik_accessories)/descriptions/sensors/realsense_d415.urdf.xacro" />
-  <xacro:include filename="$(find picknik_accessories)/descriptions/sensors/realsense_d435.urdf.xacro" />
+  <xacro:include filename="$(find picknik_accessories)/descriptions/sensors/realsense_d435.urdf.xacro"/>
   <!-- Import environment macros -->
   <xacro:include filename="$(find picknik_accessories)/descriptions/geometry/collision_and_visual/cube_collision_and_visual.urdf.xacro" />
@@ -45,5 +45,5 @@
   <!-- TODO: With ogre renderer and use_mesh="true",
   the camera image will be obstructed by the mesh-->
-  <xacro:realsense_d415 parent="d415_mount_link" name="wrist_mounted_camera" use_mesh="${gazebo_renderer == 'ogre2'}">
+  <xacro:realsense_d415 parent="d415_mount_link" name="wrist_mounted_camera" use_mesh="${gazebo_renderer == 'ogre2'}" gazebo_camera_fps="20">
     <origin xyz="0 0 0" rpy="0 0 0" />
   </xacro:realsense_d415>
@@ -79,26 +79,34 @@
     <origin rpy="0 0 0" xyz="0 0 0" />
   </joint>
-  <!-- External camera -->
-  <link name="external_camera_link" />
-  <joint name="external_camera_joint" type="fixed">
+  <!-- External camera_1 -->
+  <link name="camera_1" />
+  <joint name="camera_joint_1" type="fixed">
     <parent link="world" />
-    <child link="external_camera_link" />
-    <origin xyz="0.3 -0.3 1.0" rpy="0.0 0.4 3.14" />
+    <child link="camera_1" />
+    <origin xyz="1.1 -1.1 1.3" rpy="0.0 0.4 2.4" />
   </joint>
-  <xacro:realsense_d435 parent="external_camera_link" name="scene_camera" visible="false" simulate_depth="true">
+  <xacro:realsense_d435 parent="camera_1" name="camera_1" visible="false" simulate_depth="true" gazebo_camera_fps="20">
     <origin xyz="0 0 0" rpy="0 0 0" />
   </xacro:realsense_d435>
-  <!-- Additional Camera -->
-  <xacro:if value="$(arg use_extra_camera)">
-    <link name="extra_scene_camera_link" />
-    <joint name="extra_scene_camera_joint" type="fixed">
-      <parent link="world" />
-      <child link="extra_scene_camera_link" />
-      <origin xyz="-0.3 0.3 0.5" rpy="0.0 0.0 -3.14" />
-    </joint>
-    <xacro:realsense_d435 parent="extra_scene_camera_link" name="extra_camera" visible="false" simulate_depth="false">
-      <origin xyz="0 0 0" rpy="0 0 0" />
-    </xacro:realsense_d435>
-  </xacro:if>
+  <!-- External camera_2 -->
+  <link name="camera_2" />
+  <joint name="camera_joint_2" type="fixed">
+    <parent link="world" />
+    <child link="camera_2" />
+    <origin xyz="1.1 1.1 1.3" rpy="0.0 0.4 3.97" />
+  </joint>
+  <xacro:realsense_d435 parent="camera_2" name="camera_2" visible="false" simulate_depth="true" gazebo_camera_fps="20">
+    <origin xyz="0 0 0" rpy="0 0 0" />
+  </xacro:realsense_d435>
+  <!-- External camera_3 -->
+  <link name="camera_3" />
+  <joint name="camera_joint_3" type="fixed">
+    <parent link="world" />
+    <child link="camera_3" />
+    <origin xyz="1.5 0.0 1.0" rpy="0.0 0.4 3.14" />
+  </joint>
+  <xacro:realsense_d435 parent="camera_3" name="camera_3" visible="false" simulate_depth="true" gazebo_camera_fps="20">
+    <origin xyz="0 0 0" rpy="0 0 0" />
+  </xacro:realsense_d435>
   <!-- Force/Torque Sensor -->
   <link name="robot/wrist_3_joint/force_torque_sensor" />
