Commit message: Ran presubmit to prettify xml files

File: src/picknik_ur_gazebo_config/description/picknik_ur_gazebo.xacro (robot description, xacro)
@@ -1,37 +1,56 @@
-<?xml version="1.0"?>
+<?xml version="1.0" ?>
 <robot xmlns:xacro="http://wiki.ros.org/xacro" name="$(arg name)">
   <!-- parameters -->
-  <xacro:arg name="use_fake_hardware" default="false"/>
-  <xacro:arg name="external_camera" default="false"/>
-  <xacro:arg name="has_tool_changer" default="true"/>
-  <xacro:arg name="use_pinch_links" default="true"/>
-  <xacro:arg name="generate_ros2_control_tag" default="true"/>
-  <xacro:arg name="name" default=""/>
-  <xacro:arg name="joint_limits_parameters_file" default=""/>
-  <xacro:arg name="kinematics_parameters_file" default=""/>
-  <xacro:arg name="physical_parameters_file" default=""/>
-  <xacro:arg name="visual_parameters_file" default=""/>
-  <xacro:arg name="headless_mode" default="false"/>
-  <xacro:arg name="robot_ip" default="0.0.0.0"/>
-  <xacro:arg name="use_tool_communication" default="false"/>
-  <xacro:arg name="tool_voltage" default="0"/>
-  <xacro:arg name="tool_device_name" default="/dev/ttyUSB0"/>
-  <xacro:arg name="initial_positions_file" default="$(find picknik_ur_base_config)/config/initial_positions.yaml"/>
-  <xacro:arg name="environment_xacro" default="$(find picknik_ur_gazebo_config)/description/environment.xacro"/>
-  <xacro:arg name="simulation" default="gazebo"/>
-  <xacro:arg name="gazebo_renderer" default="ogre"/>
-  <xacro:arg name="use_extra_camera" default="false"/>
+  <xacro:arg name="use_fake_hardware" default="false" />
+  <xacro:arg name="external_camera" default="false" />
+  <xacro:arg name="has_tool_changer" default="true" />
+  <xacro:arg name="use_pinch_links" default="true" />
+  <xacro:arg name="generate_ros2_control_tag" default="true" />
+  <xacro:arg name="name" default="" />
+  <xacro:arg name="joint_limits_parameters_file" default="" />
+  <xacro:arg name="kinematics_parameters_file" default="" />
+  <xacro:arg name="physical_parameters_file" default="" />
+  <xacro:arg name="visual_parameters_file" default="" />
+  <xacro:arg name="headless_mode" default="false" />
+  <xacro:arg name="robot_ip" default="0.0.0.0" />
+  <xacro:arg name="use_tool_communication" default="false" />
+  <xacro:arg name="tool_voltage" default="0" />
+  <xacro:arg name="tool_device_name" default="/dev/ttyUSB0" />
+  <xacro:arg
+    name="initial_positions_file"
+    default="$(find picknik_ur_base_config)/config/initial_positions.yaml"
+  />
+  <xacro:arg
+    name="environment_xacro"
+    default="$(find picknik_ur_gazebo_config)/description/environment.xacro"
+  />
+  <xacro:arg name="simulation" default="gazebo" />
+  <xacro:arg name="gazebo_renderer" default="ogre" />
+  <xacro:arg name="use_extra_camera" default="false" />
   <!-- Import UR and environment macros -->
-  <xacro:include filename="$(find picknik_ur_base_config)/description/picknik_ur_macro.xacro"/>
-  <xacro:include filename="$(find picknik_ur_base_config)/description/picknik_ur_attachments_macro.xacro"/>
-  <xacro:include filename="$(arg environment_xacro)"/>
+  <xacro:include
+    filename="$(find picknik_ur_base_config)/description/picknik_ur_macro.xacro"
+  />
+  <xacro:include
+    filename="$(find picknik_ur_base_config)/description/picknik_ur_attachments_macro.xacro"
+  />
+  <xacro:include filename="$(arg environment_xacro)" />
   <!-- Robot: contains robot description from the world frame to the tool frame -->
-  <xacro:picknik_ur parent="world"  child="tool0" initial_positions_file="$(arg initial_positions_file)" generate_ros2_control_tag="$(arg generate_ros2_control_tag)">
+  <xacro:picknik_ur
+    parent="world"
+    child="tool0"
+    initial_positions_file="$(arg initial_positions_file)"
+    generate_ros2_control_tag="$(arg generate_ros2_control_tag)"
+  >
     <origin xyz="0 0 0" rpy="0 0 0" />
   </xacro:picknik_ur>
   <!-- Gripper and UR adapter and realsense camera -->
-  <xacro:picknik_ur_attachments parent="tool0" child="grasp_link" has_tool_changer="$(arg has_tool_changer)"/>
+  <xacro:picknik_ur_attachments
+    parent="tool0"
+    child="grasp_link"
+    has_tool_changer="$(arg has_tool_changer)"
+  />
   <!-- Environment: contains scene geometry and external sensors, e.g. cameras -->
-  <xacro:environment parent="world"/>
+  <xacro:environment parent="world" />
   <!-- Gazebo Force/Torque Sensor -->
   <link name="robot/wrist_3_joint/force_torque_sensor" />
@@ -96,15 +115,28 @@
   <!-- Gazebo Plugins -->
   <gazebo>
-    <plugin filename="ign_ros2_control-system" name="ign_ros2_control::IgnitionROS2ControlPlugin">
-      <parameters>$(find picknik_ur_gazebo_config)/config/control/picknik_ur5e.ros2_control.yaml</parameters>
+    <plugin
+      filename="ign_ros2_control-system"
+      name="ign_ros2_control::IgnitionROS2ControlPlugin"
+    >
+      <parameters>
+        $(find
+        picknik_ur_gazebo_config)/config/control/picknik_ur5e.ros2_control.yaml
+      </parameters>
       <ros>
-        <remapping>/servo_controller/commands:=/robot_controllers/commands</remapping>
-        <remapping>/servo_controller/joint_trajectory:=/robot_controllers/joint_trajectory</remapping>
+        <remapping>
+          /servo_controller/commands:=/robot_controllers/commands
+        </remapping>
+        <remapping>
+          /servo_controller/joint_trajectory:=/robot_controllers/joint_trajectory
+        </remapping>
       </ros>
     </plugin>
   </gazebo>
-  <xacro:property name="gazebo_renderer" default="$(arg gazebo_renderer)"/>
+  <xacro:property name="gazebo_renderer" default="$(arg gazebo_renderer)" />
   <gazebo>
-    <plugin filename="libignition-gazebo-sensors-system.so" name="ignition::gazebo::systems::Sensors">
+    <plugin
+      filename="libignition-gazebo-sensors-system.so"
+      name="ignition::gazebo::systems::Sensors"
+    >
       <render_engine>${gazebo_renderer}</render_engine>
     </plugin>

File: src/picknik_ur_mujoco_config/description/picknik_ur.xacro (robot description, xacro)
@@ -3,161 +3,185 @@
   <xacro:arg name="mujoco_model" default="description/scene.xml" />
   <material name="aluminum">
-    <color rgba="0.5 0.5 0.5 1"/>
+    <color rgba="0.5 0.5 0.5 1" />
   </material>
   <material name="plastic">
-    <color rgba="0.1 0.1 0.1 1"/>
+    <color rgba="0.1 0.1 0.1 1" />
   </material>
-  <link name="world"/>
+  <link name="world" />
   <joint name="tool_changer_joint" type="fixed">
     <!-- The parent link must be read from the robot model it is attached to. -->
-    <parent link="tool0"/>
-    <child link="tool_changer_link"/>
-    <origin rpy="0 0 0" xyz="0 0 0"/>
+    <parent link="tool0" />
+    <child link="tool_changer_link" />
+    <origin rpy="0 0 0" xyz="0 0 0" />
   </joint>
   <link name="tool_changer_link">
     <visual>
-      <origin rpy="0 0 0" xyz="0 0 0"/>
-      <geometry>
-        <mesh filename="package://picknik_accessories/descriptions/brackets/mtc_ur_tool_changer/mtc_ur3510_ur_toolchanger.dae"/>
-      </geometry>
-    </visual>
-    <collision>
-      <origin rpy="0 0 0" xyz="0 0 0"/>
-      <geometry>
-        <mesh filename="package://picknik_accessories/descriptions/brackets/mtc_ur_tool_changer/mtc_ur3510_ur_toolchanger_collision.stl"/>
+      <origin rpy="0 0 0" xyz="0 0 0" />
+      <geometry>
+        <mesh
+          filename="package://picknik_accessories/descriptions/brackets/mtc_ur_tool_changer/mtc_ur3510_ur_toolchanger.dae"
+        />
+      </geometry>
+    </visual>
+    <collision>
+      <origin rpy="0 0 0" xyz="0 0 0" />
+      <geometry>
+        <mesh
+          filename="package://picknik_accessories/descriptions/brackets/mtc_ur_tool_changer/mtc_ur3510_ur_toolchanger_collision.stl"
+        />
       </geometry>
     </collision>
   </link>
   <joint name="tool_side_joint" type="fixed">
-    <parent link="tool_changer_link"/>
-    <child link="tool_changer_tool0"/>
-    <origin rpy="0 0 0" xyz="0 0 0.0331"/>
-  </joint>
-  <link name="tool_changer_tool0"/>
+    <parent link="tool_changer_link" />
+    <child link="tool_changer_tool0" />
+    <origin rpy="0 0 0" xyz="0 0 0.0331" />
+  </joint>
+  <link name="tool_changer_tool0" />
   <joint name="realsense_camera_adapter_joint" type="fixed">
     <!-- The parent link must be read from the robot model it is attached to. -->
-    <parent link="tool_changer_tool0"/>
-    <child link="realsense_camera_adapter_link"/>
-    <origin rpy="0 0 0" xyz="0 0 0"/>
+    <parent link="tool_changer_tool0" />
+    <child link="realsense_camera_adapter_link" />
+    <origin rpy="0 0 0" xyz="0 0 0" />
   </joint>
   <link name="realsense_camera_adapter_link">
     <visual>
-      <origin rpy="0 0 0" xyz="0 0 0"/>
-      <geometry>
-        <mesh filename="package://picknik_accessories/descriptions/brackets/ur_realsense_camera_adapter/picknik_ur5_realsense_camera_adapter_rev2.dae"/>
-      </geometry>
-    </visual>
-    <collision>
-      <origin rpy="0 0 0" xyz="0 0 0"/>
-      <geometry>
-        <mesh filename="package://picknik_accessories/descriptions/brackets/ur_realsense_camera_adapter/picknik_ur5_realsense_camera_adapter_rev2_collision.stl"/>
-      </geometry>
-    </collision>
-  </link>
-  <link name="realsense_camera_adapter_tool0"/>
+      <origin rpy="0 0 0" xyz="0 0 0" />
+      <geometry>
+        <mesh
+          filename="package://picknik_accessories/descriptions/brackets/ur_realsense_camera_adapter/picknik_ur5_realsense_camera_adapter_rev2.dae"
+        />
+      </geometry>
+    </visual>
+    <collision>
+      <origin rpy="0 0 0" xyz="0 0 0" />
+      <geometry>
+        <mesh
+          filename="package://picknik_accessories/descriptions/brackets/ur_realsense_camera_adapter/picknik_ur5_realsense_camera_adapter_rev2_collision.stl"
+        />
+      </geometry>
+    </collision>
+  </link>
+  <link name="realsense_camera_adapter_tool0" />
   <joint name="realsense_camera_adapter_tool0_joint" type="fixed">
-    <parent link="realsense_camera_adapter_link"/>
-    <child link="realsense_camera_adapter_tool0"/>
-    <origin rpy="0 0 0" xyz="0 0 0.007"/>
-  </joint>
-  <link name="d415_mount_link"/>
+    <parent link="realsense_camera_adapter_link" />
+    <child link="realsense_camera_adapter_tool0" />
+    <origin rpy="0 0 0" xyz="0 0 0.007" />
+  </joint>
+  <link name="d415_mount_link" />
   <joint name="d415_mount_joint" type="fixed">
-    <parent link="realsense_camera_adapter_link"/>
-    <child link="d415_mount_link"/>
-    <origin rpy="0 -1.4660765716752369 1.5707963267948966" xyz="0 -0.067 0.0171"/>
-  </joint>
-  <link name="l515_mount_link"/>
+    <parent link="realsense_camera_adapter_link" />
+    <child link="d415_mount_link" />
+    <origin
+      rpy="0 -1.4660765716752369 1.5707963267948966"
+      xyz="0 -0.067 0.0171"
+    />
+  </joint>
+  <link name="l515_mount_link" />
   <joint name="l515_mount_joint" type="fixed">
-    <parent link="realsense_camera_adapter_link"/>
-    <child link="l515_mount_link"/>
-    <origin rpy="0 -1.4660765716752369 1.5707963267948966" xyz="0 -0.0406 0.0173"/>
+    <parent link="realsense_camera_adapter_link" />
+    <child link="l515_mount_link" />
+    <origin
+      rpy="0 -1.4660765716752369 1.5707963267948966"
+      xyz="0 -0.0406 0.0173"
+    />
   </joint>
   <!-- camera body, with origin at bottom screw mount -->
   <joint name="wrist_mounted_camera_joint" type="fixed">
-    <origin rpy="0 0 0" xyz="0 0 0"/>
-    <parent link="d415_mount_link"/>
-    <child link="wrist_mounted_camera_bottom_screw_frame"/>
-  </joint>
-  <link name="wrist_mounted_camera_bottom_screw_frame"/>
+    <origin rpy="0 0 0" xyz="0 0 0" />
+    <parent link="d415_mount_link" />
+    <child link="wrist_mounted_camera_bottom_screw_frame" />
+  </joint>
+  <link name="wrist_mounted_camera_bottom_screw_frame" />
   <joint name="wrist_mounted_camera_link_joint" type="fixed">
-    <origin rpy="0 0 0" xyz="0 0.02 0.0115"/>
-    <parent link="wrist_mounted_camera_bottom_screw_frame"/>
-    <child link="wrist_mounted_camera_link"/>
+    <origin rpy="0 0 0" xyz="0 0.02 0.0115" />
+    <parent link="wrist_mounted_camera_bottom_screw_frame" />
+    <child link="wrist_mounted_camera_link" />
   </joint>
   <link name="wrist_mounted_camera_link">
     <visual>
-      <origin rpy="1.5707963267948966 0 1.5707963267948966" xyz="0.00987 -0.02 0"/>
-      <geometry>
-        <mesh filename="package://realsense2_description/meshes/d415.stl"/>
+      <origin
+        rpy="1.5707963267948966 0 1.5707963267948966"
+        xyz="0.00987 -0.02 0"
+      />
+      <geometry>
+        <mesh filename="package://realsense2_description/meshes/d415.stl" />
       </geometry>
       <material name="rs_aluminum">
-        <color rgba="0.5 0.5 0.5 1.0"/>
+        <color rgba="0.5 0.5 0.5 1.0" />
       </material>
     </visual>
     <collision>
-      <origin rpy="0 0 0" xyz="0 -0.02 0"/>
-      <geometry>
-        <box size="0.02005 0.099 0.023"/>
-      </geometry>
-    </collision>
-    <inertial>
-      <mass value="0.072"/>
+      <origin rpy="0 0 0" xyz="0 -0.02 0" />
+      <geometry>
+        <box size="0.02005 0.099 0.023" />
+      </geometry>
+    </collision>
+    <inertial>
+      <mass value="0.072" />
       <!-- The following are not reliable values, and should not be used for modeling -->
-      <origin xyz="0 0 0"/>
-      <inertia ixx="0.003881243" ixy="0.0" ixz="0.0" iyy="0.000498940" iyz="0.0" izz="0.003879257"/>
+      <origin xyz="0 0 0" />
+      <inertia
+        ixx="0.003881243"
+        ixy="0.0"
+        ixz="0.0"
+        iyy="0.000498940"
+        iyz="0.0"
+        izz="0.003879257"
+      />
     </inertial>
   </link>
   <!-- camera depth joints and links -->
   <joint name="wrist_mounted_camera_depth_joint" type="fixed">
-    <origin rpy="0 0 0" xyz="0 0 0"/>
-    <parent link="wrist_mounted_camera_link"/>
-    <child link="wrist_mounted_camera_depth_frame"/>
-  </joint>
-  <link name="wrist_mounted_camera_depth_frame"/>
+    <origin rpy="0 0 0" xyz="0 0 0" />
+    <parent link="wrist_mounted_camera_link" />
+    <child link="wrist_mounted_camera_depth_frame" />
+  </joint>
+  <link name="wrist_mounted_camera_depth_frame" />
   <joint name="wrist_mounted_camera_depth_optical_joint" type="fixed">
-    <origin rpy="-1.5707963267948966 0 -1.5707963267948966" xyz="0 0 0"/>
-    <parent link="wrist_mounted_camera_depth_frame"/>
-    <child link="wrist_mounted_camera_depth_optical_frame"/>
-  </joint>
-  <link name="wrist_mounted_camera_depth_optical_frame"/>
+    <origin rpy="-1.5707963267948966 0 -1.5707963267948966" xyz="0 0 0" />
+    <parent link="wrist_mounted_camera_depth_frame" />
+    <child link="wrist_mounted_camera_depth_optical_frame" />
+  </joint>
+  <link name="wrist_mounted_camera_depth_optical_frame" />
   <!-- camera left IR joints and links -->
   <joint name="wrist_mounted_camera_infra1_joint" type="fixed">
-    <origin rpy="0 0 0" xyz="0 0.0 0"/>
-    <parent link="wrist_mounted_camera_link"/>
-    <child link="wrist_mounted_camera_infra1_frame"/>
-  </joint>
-  <link name="wrist_mounted_camera_infra1_frame"/>
+    <origin rpy="0 0 0" xyz="0 0.0 0" />
+    <parent link="wrist_mounted_camera_link" />
+    <child link="wrist_mounted_camera_infra1_frame" />
+  </joint>
+  <link name="wrist_mounted_camera_infra1_frame" />
   <joint name="wrist_mounted_camera_infra1_optical_joint" type="fixed">
-    <origin rpy="-1.5707963267948966 0 -1.5707963267948966" xyz="0 0 0"/>
-    <parent link="wrist_mounted_camera_infra1_frame"/>
-    <child link="wrist_mounted_camera_infra1_optical_frame"/>
-  </joint>
-  <link name="wrist_mounted_camera_infra1_optical_frame"/>
+    <origin rpy="-1.5707963267948966 0 -1.5707963267948966" xyz="0 0 0" />
+    <parent link="wrist_mounted_camera_infra1_frame" />
+    <child link="wrist_mounted_camera_infra1_optical_frame" />
+  </joint>
+  <link name="wrist_mounted_camera_infra1_optical_frame" />
   <!-- camera right IR joints and links -->
   <joint name="wrist_mounted_camera_infra2_joint" type="fixed">
-    <origin rpy="0 0 0" xyz="0 -0.055 0"/>
-    <parent link="wrist_mounted_camera_link"/>
-    <child link="wrist_mounted_camera_infra2_frame"/>
-  </joint>
-  <link name="wrist_mounted_camera_infra2_frame"/>
+    <origin rpy="0 0 0" xyz="0 -0.055 0" />
+    <parent link="wrist_mounted_camera_link" />
+    <child link="wrist_mounted_camera_infra2_frame" />
+  </joint>
+  <link name="wrist_mounted_camera_infra2_frame" />
   <joint name="wrist_mounted_camera_infra2_optical_joint" type="fixed">
-    <origin rpy="-1.5707963267948966 0 -1.5707963267948966" xyz="0 0 0"/>
-    <parent link="wrist_mounted_camera_infra2_frame"/>
-    <child link="wrist_mounted_camera_infra2_optical_frame"/>
-  </joint>
-  <link name="wrist_mounted_camera_infra2_optical_frame"/>
+    <origin rpy="-1.5707963267948966 0 -1.5707963267948966" xyz="0 0 0" />
+    <parent link="wrist_mounted_camera_infra2_frame" />
+    <child link="wrist_mounted_camera_infra2_optical_frame" />
+  </joint>
+  <link name="wrist_mounted_camera_infra2_optical_frame" />
   <!-- camera color joints and links -->
   <joint name="wrist_mounted_camera_color_joint" type="fixed">
-    <origin rpy="0 0 0" xyz="0 0.015 0"/>
-    <parent link="wrist_mounted_camera_link"/>
-    <child link="wrist_mounted_camera_color_frame"/>
-  </joint>
-  <link name="wrist_mounted_camera_color_frame"/>
+    <origin rpy="0 0 0" xyz="0 0.015 0" />
+    <parent link="wrist_mounted_camera_link" />
+    <child link="wrist_mounted_camera_color_frame" />
+  </joint>
+  <link name="wrist_mounted_camera_color_frame" />
   <joint name="wrist_mounted_camera_color_optical_joint" type="fixed">
-    <origin rpy="-1.5707963267948966 0 -1.5707963267948966" xyz="0 0 0"/>
-    <parent link="wrist_mounted_camera_color_frame"/>
-    <child link="wrist_mounted_camera_color_optical_frame"/>
-  </joint>
-  <link name="wrist_mounted_camera_color_optical_frame"/>
+    <origin rpy="-1.5707963267948966 0 -1.5707963267948966" xyz="0 0 0" />
+    <parent link="wrist_mounted_camera_color_frame" />
+    <child link="wrist_mounted_camera_color_optical_frame" />
+  </joint>
+  <link name="wrist_mounted_camera_color_optical_frame" />
   <gazebo reference="wrist_mounted_camera_color_frame">
     <sensor name="wrist_mounted_camera_rgbd_sensor" type="rgbd_camera">
@@ -211,5 +235,7 @@
           </clip>
         </depth_camera>
-        <optical_frame_id>wrist_mounted_camera_color_optical_frame</optical_frame_id>
+        <optical_frame_id>
+          wrist_mounted_camera_color_optical_frame
+        </optical_frame_id>
       </camera>
       <ignition_frame_id>wrist_mounted_camera_color_frame</ignition_frame_id>
@@ -223,50 +249,72 @@
   <joint name="ur_to_robotiq_joint" type="fixed">
     <!-- The parent link must be read from the robot model it is attached to. -->
-    <parent link="realsense_camera_adapter_tool0"/>
-    <child link="ur_to_robotiq_link"/>
-    <origin rpy="0 0 0" xyz="0 0 0"/>
+    <parent link="realsense_camera_adapter_tool0" />
+    <child link="ur_to_robotiq_link" />
+    <origin rpy="0 0 0" xyz="0 0 0" />
   </joint>
   <link name="ur_to_robotiq_link">
     <visual>
-      <origin rpy="0 0 0" xyz="0 0 0"/>
-      <geometry>
-        <mesh filename="package://robotiq_description/meshes/visual/2f_85/ur_to_robotiq_adapter.dae"/>
-      </geometry>
-    </visual>
-    <collision>
-      <origin rpy="0 0 0" xyz="0 0 0"/>
-      <geometry>
-        <mesh filename="package://robotiq_description/meshes/collision/2f_85/ur_to_robotiq_adapter.stl"/>
-      </geometry>
-    </collision>
-    <inertial>
-      <mass value="0.01"/>
-      <origin xyz="0 0 0"/>
-      <inertia ixx="0.000044" ixy="0.0" ixz="0.0" iyy="0.000027" iyz="0.0" izz="0.000027"/>
+      <origin rpy="0 0 0" xyz="0 0 0" />
+      <geometry>
+        <mesh
+          filename="package://robotiq_description/meshes/visual/2f_85/ur_to_robotiq_adapter.dae"
+        />
+      </geometry>
+    </visual>
+    <collision>
+      <origin rpy="0 0 0" xyz="0 0 0" />
+      <geometry>
+        <mesh
+          filename="package://robotiq_description/meshes/collision/2f_85/ur_to_robotiq_adapter.stl"
+        />
+      </geometry>
+    </collision>
+    <inertial>
+      <mass value="0.01" />
+      <origin xyz="0 0 0" />
+      <inertia
+        ixx="0.000044"
+        ixy="0.0"
+        ixz="0.0"
+        iyy="0.000027"
+        iyz="0.0"
+        izz="0.000027"
+      />
     </inertial>
   </link>
   <joint name="gripper_side_joint" type="fixed">
-    <parent link="ur_to_robotiq_link"/>
-    <child link="gripper_mount_link"/>
+    <parent link="ur_to_robotiq_link" />
+    <child link="gripper_mount_link" />
     <!-- <origin xyz="0 0 0.011" rpy="0 ${-pi/2} ${pi/2}"/> -->
-    <origin rpy="0 0 0" xyz="0 0 0.011"/>
-  </joint>
-  <link name="gripper_mount_link"/>
+    <origin rpy="0 0 0" xyz="0 0 0.011" />
+  </joint>
+  <link name="gripper_mount_link" />
   <!-- Add robotiq 2f 85 gripper model -->
   <link name="robotiq_85_base_link">
     <visual>
       <geometry>
-        <mesh filename="package://robotiq_description/meshes/visual/2f_85/robotiq_base.dae"/>
-      </geometry>
-    </visual>
-    <collision>
-      <geometry>
-        <mesh filename="package://robotiq_description/meshes/collision/2f_85/robotiq_base.stl"/>
-      </geometry>
-    </collision>
-    <inertial>
-      <origin rpy="0 0 0" xyz="0.0 2.274e-05 0.03232288"/>
-      <mass value="6.6320197e-01"/>
-      <inertia ixx="5.1617816e-04" ixy="2.936e-8" ixz="0.0" iyy="5.8802208e-04" iyz="-3.2296e-7" izz="3.9462776e-04"/>
+        <mesh
+          filename="package://robotiq_description/meshes/visual/2f_85/robotiq_base.dae"
+        />
+      </geometry>
+    </visual>
+    <collision>
+      <geometry>
+        <mesh
+          filename="package://robotiq_description/meshes/collision/2f_85/robotiq_base.stl"
+        />
+      </geometry>
+    </collision>
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