Commit message: swap robot positions

File: src/picknik_dual_ur_arm_config/description/dual_arm_ur.xacro (robot description, xacro)
@@ -52,5 +52,5 @@
     sim_ignition="true"
     initial_positions="${xacro.load_yaml(initial_positions_file)}">
-    <origin xyz="0 0.5 0" rpy="0 0 0" /> <!-- position robot in the world -->
+    <origin xyz="0 -0.5 0" rpy="0 0 0" /> <!-- position robot in the world -->
   </xacro:ur_robot>
   <!-- tool changer-->
@@ -86,5 +86,5 @@
     sim_ignition="true"
     initial_positions="${xacro.load_yaml(initial_positions_file)}">
-    <origin xyz="0 -0.5 0" rpy="0 0 0" /> <!-- position robot in the world -->
+    <origin xyz="0 0.5 0" rpy="0 0 0" /> <!-- position robot in the world -->
   </xacro:ur_robot>
   <!-- tool changer-->
