Commit message: updates for generic camera usage

File: src/picknik_ur_multi_arm_gazebo_config/description/dual_arm_ur.xacro (robot description, xacro)
@@ -27,4 +27,5 @@
   <xacro:include filename="$(find picknik_ur_base_config)/description/pinch_links.xacro" />
   <xacro:include filename="$(find picknik_ur_base_config)/description/picknik_ur_attachments_macro.xacro" />
+  <xacro:include filename="$(find picknik_ur_multi_arm_gazebo_config)/description/camera_and_gripper.xacro" />
   <xacro:include filename="$(find picknik_accessories)/descriptions/sensors/realsense_d435.urdf.xacro" />
   <!-- Initial positions for simulations (Mock Hardware and Gazebo) -->
@@ -34,7 +35,4 @@
   <xacro:include filename="$(find picknik_accessories)/descriptions/geometry/collision_and_visual/cube_collision_and_visual.urdf.xacro" />
   <xacro:include filename="$(find picknik_accessories)/descriptions/geometry/visual/cube_visual.urdf.xacro" />
-  <!-- Bring in realsense materials only once -->
-  <xacro:include filename="$(find realsense2_description)/urdf/_materials.urdf.xacro" />
-  <xacro:property name="realsense_materials_defined" value="true"/>
   <xacro:property name="gazebo_renderer" default="$(arg gazebo_renderer)"/>
   <link name="world" />
@@ -63,5 +61,5 @@
       <xacro:wrist_3_pinch_link  prefix="right"/>
   </xacro:if>
-  <xacro:picknik_ur_attachments
+  <xacro:camera_and_gripper
     prefix="left"
     parent="left_tool0"
@@ -93,5 +91,5 @@
     <xacro:wrist_3_pinch_link  prefix="left"/>
   </xacro:if>
-  <xacro:picknik_ur_attachments
+  <xacro:camera_and_gripper
     prefix="right"
     parent="right_tool0"

Commit message: added left gripper controller and updated objectives

File: src/picknik_ur_multi_arm_gazebo_config/description/dual_arm_ur.xacro (robot description, xacro)
@@ -105,10 +105,4 @@
       </geometry>
     </visual>
-    <collision>
-      <origin rpy="0 0 0" xyz="0 0 0"/>
-      <geometry>
-        <mesh filename="package://picknik_accessories/descriptions/furniture/generic_table/wood_block.dae" scale="0.25 0.25 0.1"/>
-      </geometry>
-    </collision>
   </link>
   <joint name="table_joint" type="fixed">
