Commit message: add camera frame to URDF
Signed-off-by: Paul Gesel <paulgesel@gmail.com>

File: src/picknik_panda_mujoco_config/description/panda.xacro (robot description, xacro)
@@ -253,4 +253,11 @@
         <color rgba="1. 1. 1. 1."/>
     </material>
+    <!--Add camera frame-->
+    <joint name="wrist_camera_joint" type="fixed">
+        <parent link="panda_hand"/>
+        <child link="wrist_camera_color_optical_frame"/>
+        <origin rpy="0 0 ${pi/2}" xyz="0.05 0 0"/>
+    </joint>
+    <link name="wrist_camera_color_optical_frame"/>
     <ros2_control name="picknik_mujoco_simulation" type="system">
         <joint name="panda_joint1">

Commit message: rename camera link
Signed-off-by: Paul Gesel <paulgesel@gmail.com>

File: src/picknik_panda_mujoco_config/description/panda.xacro (robot description, xacro)
@@ -256,8 +256,8 @@
     <joint name="wrist_camera_joint" type="fixed">
         <parent link="panda_hand"/>
-        <child link="wrist_camera_color_optical_frame"/>
+        <child link="wrist_camera_optical_frame"/>
         <origin rpy="0 0 ${pi/2}" xyz="0.05 0 0"/>
     </joint>
-    <link name="wrist_camera_color_optical_frame"/>
+    <link name="wrist_camera_optical_frame"/>
     <ros2_control name="picknik_mujoco_simulation" type="system">
         <joint name="panda_joint1">
