Commit message: Move to new hardware config

File: src/picknik_ur_mock_hw_config/description/picknik_ur_machine_tending.xacro (robot description, xacro)
@@ -51,5 +51,5 @@
     output_recipe_filename="$(find ur_robot_driver)/resources/rtde_output_recipe.txt"
     input_recipe_filename="$(find ur_robot_driver)/resources/rtde_input_recipe.txt">
-    <origin xyz="0 0 0" rpy="0 0 0" />
+    <origin xyz="0 0 0.8" rpy="0 0 0" />
   </xacro:ur_robot>
   <xacro:if value="$(arg has_tool_changer)">
@@ -85,78 +85,103 @@
     <origin xyz="0 0 0" rpy="${pi / 180.0 * 5} 0 0" />
   </joint>
-  <!-- Environment -->
-  <link name="environment">
+  <!-- CNC machine -->
+  <link name="cnc_machine">
     <visual>
       <origin xyz="0 0 0" rpy="0 0 0" />
       <geometry>
-        <mesh filename="package://picknik_accessories/descriptions/furniture/generic_table/wood_block.dae" scale="0.25 0.25 0.1"/>
+        <mesh filename="file://$(find picknik_ur_mock_hw_config)/meshes/cnc.dae" scale="1 1 1"/>
       </geometry>
     </visual>
     <collision>
-      <origin rpy="0 0 0" xyz="0 0 0"/>
+      <origin xyz="0 0 0" rpy="0 0 0"/>
       <geometry>
-        <mesh filename="package://picknik_accessories/descriptions/furniture/generic_table/wood_block.dae" scale="0.25 0.25 0.1"/>
+        <mesh filename="file://$(find picknik_ur_mock_hw_config)/meshes/cnc.dae" scale="1 1 1"/>
       </geometry>
     </collision>
   </link>
-  <joint name="table_joint" type="fixed">
-    <parent link="base" />
-    <child link="environment" />
-    <origin rpy="0 0 0" xyz="0 0 -0.05" />
+  <joint name="cnc_machine_joint" type="fixed">
+    <parent link="world" />
+    <child link="cnc_machine" />
+    <origin xyz="-0.1 -1 0" rpy="0 0 3.14"  />
   </joint>
-  <link name="box_1">
-    <xacro:cube_visual length="0.05" width="0.05" height="0.05">
+  <!-- Robot base -->
+  <link name="robot_base">
+    <visual>
       <origin xyz="0 0 0" rpy="0 0 0" />
-      <color rgba="0.1 0.1 0.1 0.9" />
-    </xacro:cube_visual>
+      <geometry>
+        <mesh filename="file://$(find picknik_ur_mock_hw_config)/meshes/base.dae" scale="1 1 1"/>
+      </geometry>
+    </visual>
+    <collision>
+      <origin xyz="0 0 0" rpy="0 0 0"/>
+      <geometry>
+        <mesh filename="file://$(find picknik_ur_mock_hw_config)/meshes/base.dae" scale="1 1 1"/>
+      </geometry>
+    </collision>
   </link>
-  <joint name="box1_on_table" type="fixed">
-    <parent link="environment" />
-    <child link="box_1" />
-    <origin rpy="0 0 0" xyz="0.65 -0.35 0.1" />
+  <joint name="robot_base_joint" type="fixed">
+    <parent link="world" />
+    <child link="robot_base" />
+    <origin xyz="0 0 0" rpy="0 0 0"  />
   </joint>
-  <link name="box_2">
-    <xacro:cube_visual length="0.05" width="0.05" height="0.05">
+  <!-- Hexagonal table 1 -->
+  <link name="hexagonal_table_1">
+    <visual>
       <origin xyz="0 0 0" rpy="0 0 0" />
-      <color rgba="0.5 0.5 0.5 0.9" />
-    </xacro:cube_visual>
+      <geometry>
+        <mesh filename="file://$(find picknik_ur_mock_hw_config)/meshes/table.dae" scale="1 1 1"/>
+      </geometry>
+    </visual>
+    <collision>
+      <origin xyz="0 0 0" rpy="0 0 0"/>
+      <geometry>
+        <mesh filename="file://$(find picknik_ur_mock_hw_config)/meshes/table.dae" scale="1 1 1"/>
+      </geometry>
+    </collision>
   </link>
-  <joint name="box2_on_table" type="fixed">
-    <parent link="environment" />
-    <child link="box_2" />
-    <origin rpy="0 0 0" xyz="0.65 0.35 0.1" />
+  <joint name="hexagonal_table_joint_1" type="fixed">
+    <parent link="world" />
+    <child link="hexagonal_table_1" />
+    <origin xyz="0.8 0 0" rpy="0 0 0"  />
   </joint>
-  <link name="box_3">
-    <xacro:cube_visual length="0.05" width="0.05" height="0.05">
+  <!-- Hexagonal table 2 -->
+  <link name="hexagonal_table_2">
+    <visual>
       <origin xyz="0 0 0" rpy="0 0 0" />
-      <color rgba="0.8 0.3 0.1 0.9" />
-    </xacro:cube_visual>
+      <geometry>
+        <mesh filename="file://$(find picknik_ur_mock_hw_config)/meshes/table.dae" scale="1 1 1"/>
+      </geometry>
+    </visual>
+    <collision>
+      <origin xyz="0 0 0" rpy="0 0 0"/>
+      <geometry>
+        <mesh filename="file://$(find picknik_ur_mock_hw_config)/meshes/table.dae" scale="1 1 1"/>
+      </geometry>
+    </collision>
   </link>
-  <joint name="box3_on_table" type="fixed">
-    <parent link="environment" />
-    <child link="box_3" />
-    <origin rpy="0 0 0" xyz="0.65 0 0.1" />
+  <joint name="hexagonal_table_joint_2" type="fixed">
+    <parent link="world" />
+    <child link="hexagonal_table_2" />
+    <origin xyz="-0.8 0 0" rpy="0 0 0"  />
   </joint>
-  <link name="box_4">
-    <xacro:cube_visual length="0.05" width="0.05" height="0.05">
+  <!-- Cylinder item -->
+  <link name="cylinder_item">
+    <visual>
       <origin xyz="0 0 0" rpy="0 0 0" />
-      <color rgba="0.8 0.3 0.1 0.9" />
-    </xacro:cube_visual>
+      <geometry>
+        <mesh filename="file://$(find picknik_ur_mock_hw_config)/meshes/cylinder-item.dae" scale="1 1 1"/>
+      </geometry>
+    </visual>
+    <collision>
+      <origin xyz="0 0 0" rpy="0 0 0"/>
+      <geometry>
+        <mesh filename="file://$(find picknik_ur_mock_hw_config)/meshes/cylinder-item.dae" scale="1 1 1"/>
+      </geometry>
+    </collision>
   </link>
-  <joint name="box4_on_table" type="fixed">
-    <parent link="environment" />
-    <child link="box_4" />
-    <origin rpy="0 0 0" xyz="-0.65 0.25 0.1" />
-  </joint>
-  <link name="box_5">
-    <xacro:cube_visual length="0.05" width="0.05" height="0.05">
-      <origin xyz="0 0 0" rpy="0 0 0" />
-      <color rgba="0.1 0.3 0.8 0.9" />
-    </xacro:cube_visual>
-  </link>
-  <joint name="box5_on_table" type="fixed">
-    <parent link="environment" />
-    <child link="box_5" />
-    <origin rpy="0 0 0" xyz="-0.65 -0.25 0.1" />
+  <joint name="cylinder_item_joint" type="fixed">
+    <parent link="world" />
+    <child link="cylinder_item" />
+    <origin xyz="0.73 0.06 0.5" rpy="0 0 0"  />
   </joint>
   <!-- External Camera -->

Commit message: Cleanup configs and inherited Objectives

File: src/picknik_ur_mock_hw_config/description/picknik_ur_machine_tending.xacro (robot description, xacro)
@@ -51,5 +51,5 @@
     output_recipe_filename="$(find ur_robot_driver)/resources/rtde_output_recipe.txt"
     input_recipe_filename="$(find ur_robot_driver)/resources/rtde_input_recipe.txt">
-    <origin xyz="0 0 0.8" rpy="0 0 0" />
+    <origin xyz="0 0 0.8" rpy="0 0 ${pi/2}" />
   </xacro:ur_robot>
   <xacro:if value="$(arg has_tool_changer)">

Commit message: PR comments and general cleanup

File: src/picknik_ur_mock_hw_config/description/picknik_ur_machine_tending.xacro (robot description, xacro)
@@ -103,5 +103,5 @@
     <parent link="world" />
     <child link="cnc_machine" />
-    <origin xyz="-0.1 -1 0" rpy="0 0 3.14"  />
+    <origin xyz="-0.1 -1.2 0" rpy="0 0 3.14"  />
   </joint>
   <!-- Robot base -->

Commit message: Modify scene positions and collisions, add cylinder on right

File: src/picknik_ur_mock_hw_config/description/picknik_ur_machine_tending.xacro (robot description, xacro)
@@ -26,12 +26,8 @@
   <xacro:include filename="$(find picknik_accessories)/descriptions/brackets/ur_realsense_camera_adapter/picknik_ur_camera_adapter.urdf.xacro" />
   <xacro:include filename="$(find picknik_accessories)/descriptions/sensors/realsense_d415.urdf.xacro" />
-  <xacro:include filename="$(find picknik_accessories)/descriptions/sensors/realsense_d435.urdf.xacro" />
   <xacro:include filename="$(find picknik_ur_base_config)/description/pinch_link.xacro" />
   <!-- Initial positions for simulations (Mock Hardware and Gazebo) -->
-  <xacro:arg name="initial_positions_file" default="$(find picknik_ur_base_config)/config/initial_positions.yaml"/>
+  <xacro:arg name="initial_positions_file" default="$(find picknik_ur_mock_hw_config)/config/initial_positions.yaml"/>
   <xacro:property name="initial_positions_file" default="$(arg initial_positions_file)"/>
-  <!-- Import environment macros -->
-  <xacro:include filename="$(find picknik_accessories)/descriptions/geometry/collision_and_visual/cube_collision_and_visual.urdf.xacro" />
-  <xacro:include filename="$(find picknik_accessories)/descriptions/geometry/visual/cube_visual.urdf.xacro" />
   <link name="world" />
   <!-- arm -->
@@ -51,5 +47,5 @@
     output_recipe_filename="$(find ur_robot_driver)/resources/rtde_output_recipe.txt"
     input_recipe_filename="$(find ur_robot_driver)/resources/rtde_input_recipe.txt">
-    <origin xyz="0 0 0.8" rpy="0 0 ${pi/2}" />
+    <origin xyz="0 0 0" rpy="0 0 ${pi/2}" />
   </xacro:ur_robot>
   <xacro:if value="$(arg has_tool_changer)">
@@ -103,5 +99,5 @@
     <parent link="world" />
     <child link="cnc_machine" />
-    <origin xyz="-0.1 -1.2 0" rpy="0 0 3.14"  />
+    <origin xyz="-0.1 -1.2 -0.8" rpy="0 0 3.14"  />
   </joint>
   <!-- Robot base -->
@@ -123,8 +119,8 @@
     <parent link="world" />
     <child link="robot_base" />
-    <origin xyz="0 0 0" rpy="0 0 0"  />
+    <origin xyz="0 0 -0.8" rpy="0 0 0"  />
   </joint>
-  <!-- Hexagonal table 1 -->
-  <link name="hexagonal_table_1">
+  <!-- Hexagonal tables -->
+  <link name="left_hexagonal_table">
     <visual>
       <origin xyz="0 0 0" rpy="0 0 0" />
@@ -134,17 +130,16 @@
     </visual>
     <collision>
-      <origin xyz="0 0 0" rpy="0 0 0"/>
+      <origin xyz="0 0 0.29" rpy="0 0 0"/>
       <geometry>
-        <mesh filename="file://$(find picknik_ur_mock_hw_config)/meshes/table.dae" scale="1 1 1"/>
+        <box size="1.0 1.0 0.58"/>
       </geometry>
     </collision>
   </link>
-  <joint name="hexagonal_table_joint_1" type="fixed">
+  <joint name="left_hexagonal_table_joint" type="fixed">
     <parent link="world" />
-    <child link="hexagonal_table_1" />
-    <origin xyz="0.8 0 0" rpy="0 0 0"  />
+    <child link="left_hexagonal_table" />
+    <origin xyz="0.8 0 -0.8" rpy="0 0 0"  />
   </joint>
-  <!-- Hexagonal table 2 -->
-  <link name="hexagonal_table_2">
+  <link name="right_hexagonal_table">
     <visual>
       <origin xyz="0 0 0" rpy="0 0 0" />
@@ -154,17 +149,17 @@
     </visual>
     <collision>
-      <origin xyz="0 0 0" rpy="0 0 0"/>
+      <origin xyz="0 0 0.29" rpy="0 0 0"/>
       <geometry>
-        <mesh filename="file://$(find picknik_ur_mock_hw_config)/meshes/table.dae" scale="1 1 1"/>
+        <box size="1.0 1.0 0.58"/>
       </geometry>
     </collision>
   </link>
-  <joint name="hexagonal_table_joint_2" type="fixed">
+  <joint name="right_hexagonal_table_joint" type="fixed">
     <parent link="world" />
-    <child link="hexagonal_table_2" />
-    <origin xyz="-0.8 0 0" rpy="0 0 0"  />
+    <child link="right_hexagonal_table" />
+    <origin xyz="-0.8 0 -0.8" rpy="0 0 0"  />
   </joint>
-  <!-- Cylinder item -->
-  <link name="cylinder_item">
+  <!-- Cylinder items -->
+  <link name="left_cylinder_item">
     <visual>
       <origin xyz="0 0 0" rpy="0 0 0" />
@@ -173,25 +168,24 @@
       </geometry>
     </visual>
-    <collision>
-      <origin xyz="0 0 0" rpy="0 0 0"/>
+    <!-- No collision geometry so the gripper can overlap with the object. -->
+  </link>
+  <joint name="left_cylinder_item_joint" type="fixed">
+    <parent link="world" />
+    <child link="left_cylinder_item" />
+    <origin xyz="0.73 0.06 -0.25" rpy="0 0 0"  />
+  </joint>
+  <link name="right_cylinder_item">
+    <visual>
+      <origin xyz="0 0 0" rpy="0 0 0" />
       <geometry>
         <mesh filename="file://$(find picknik_ur_mock_hw_config)/meshes/cylinder-item.dae" scale="1 1 1"/>
       </geometry>
-    </collision>
+    </visual>
+    <!-- No collision geometry so the gripper can overlap with the object. -->
   </link>
-  <joint name="cylinder_item_joint" type="fixed">
+  <joint name="right_cylinder_item_joint" type="fixed">
     <parent link="world" />
-    <child link="cylinder_item" />
-    <origin xyz="0.73 0.06 0.5" rpy="0 0 0"  />
+    <child link="right_cylinder_item" />
+    <origin xyz="-0.73 0.06 -0.25" rpy="0 0 0"  />
   </joint>
-  <!-- External Camera -->
-  <link name="external_camera_link" />
-  <joint name="external_camera_joint" type="fixed">
-    <parent link="world" />
-    <child link="external_camera_link" />
-    <origin xyz="-0.3 0.3 1.0" rpy="0.0 0.4 0" />
-  </joint>
-  <xacro:realsense_d435 parent="external_camera_link" name="scene_camera" visible="false">
-    <origin xyz="0 0 0" rpy="0 0 0" />
-  </xacro:realsense_d435>
 </robot>

Commit message: Updated CNC scene textures.

File: src/picknik_ur_mock_hw_config/description/picknik_ur_machine_tending.xacro (robot description, xacro)
@@ -119,5 +119,5 @@
     <parent link="world" />
     <child link="robot_base" />
-    <origin xyz="0 0 -0.8" rpy="0 0 0"  />
+    <origin xyz="0 0 -0.8" rpy="0 0 3.14"  />
   </joint>
   <!-- Hexagonal tables -->
@@ -139,5 +139,5 @@
     <parent link="world" />
     <child link="left_hexagonal_table" />
-    <origin xyz="0.8 0 -0.8" rpy="0 0 0"  />
+    <origin xyz="0.8 0 -0.8" rpy="0 0 3.14"  />
   </joint>
   <link name="right_hexagonal_table">
@@ -158,5 +158,5 @@
     <parent link="world" />
     <child link="right_hexagonal_table" />
-    <origin xyz="-0.8 0 -0.8" rpy="0 0 0"  />
+    <origin xyz="-0.8 0 -0.8" rpy="0 0 3.14"  />
   </joint>
   <!-- Cylinder items -->
@@ -173,5 +173,5 @@
     <parent link="world" />
     <child link="left_cylinder_item" />
-    <origin xyz="0.73 0.06 -0.25" rpy="0 0 0"  />
+    <origin xyz="0.73 0.06 -0.30" rpy="0 0 3.14"  />
   </joint>
   <link name="right_cylinder_item">
@@ -187,5 +187,5 @@
     <parent link="world" />
     <child link="right_cylinder_item" />
-    <origin xyz="-0.73 0.06 -0.25" rpy="0 0 0"  />
+    <origin xyz="-0.73 0.06 -0.30" rpy="0 0 3.14"  />
   </joint>
 </robot>

Commit message: Simplify CNC collision

File: src/picknik_ur_mock_hw_config/description/picknik_ur_machine_tending.xacro (robot description, xacro)
@@ -89,8 +89,30 @@
       </geometry>
     </visual>
-    <collision>
-      <origin xyz="0 0 0" rpy="0 0 0"/>
-      <geometry>
-        <mesh filename="file://$(find picknik_ur_mock_hw_config)/meshes/cnc.dae" scale="1 1 1"/>
+    <!-- CNC base collision -->
+    <collision>
+      <origin xyz="-0.2 0 0.45" rpy="0 0 0"/>
+      <geometry>
+        <box size="1.8 1.1 0.9"/>
+      </geometry>
+    </collision>
+    <!-- CNC left door collision -->
+    <collision>
+      <origin xyz="-0.8 -0.4 1.35" rpy="0 0 0"/>
+      <geometry>
+        <box size="0.6 0.3 0.9"/>
+      </geometry>
+    </collision>
+    <!-- CNC right door collision -->
+    <collision>
+      <origin xyz="0.5 -0.4 1.35" rpy="0 0 0"/>
+      <geometry>
+        <box size="0.4 0.3 0.9"/>
+      </geometry>
+    </collision>
+    <!-- CNC top -->
+    <collision>
+      <origin xyz="-0.2 0 1.85" rpy="0 0 0"/>
+      <geometry>
+        <box size="1.8 1.1 0.2"/>
       </geometry>
     </collision>

Commit message: Use simplifies collision DAE files

File: src/picknik_ur_mock_hw_config/description/picknik_ur_machine_tending.xacro (robot description, xacro)
@@ -91,28 +91,7 @@
     <!-- CNC base collision -->
     <collision>
-      <origin xyz="-0.2 0 0.45" rpy="0 0 0"/>
+      <origin xyz="0 0.1 0" rpy="0 0 0"/>
       <geometry>
-        <box size="1.8 1.1 0.9"/>
-      </geometry>
-    </collision>
-    <!-- CNC left door collision -->
-    <collision>
-      <origin xyz="-0.8 -0.4 1.35" rpy="0 0 0"/>
-      <geometry>
-        <box size="0.6 0.3 0.9"/>
-      </geometry>
-    </collision>
-    <!-- CNC right door collision -->
-    <collision>
-      <origin xyz="0.5 -0.4 1.35" rpy="0 0 0"/>
-      <geometry>
-        <box size="0.4 0.3 0.9"/>
-      </geometry>
-    </collision>
-    <!-- CNC top -->
-    <collision>
-      <origin xyz="-0.2 0 1.85" rpy="0 0 0"/>
-      <geometry>
-        <box size="1.8 1.1 0.2"/>
+        <mesh filename="file://$(find picknik_ur_mock_hw_config)/meshes/cnc-collision.dae" scale="1 1 1"/>
       </geometry>
     </collision>
@@ -152,7 +131,7 @@
     </visual>
     <collision>
-      <origin xyz="0 0 0.29" rpy="0 0 0"/>
+      <origin xyz="0 0 0" rpy="0 0 0" />
       <geometry>
-        <box size="1.0 1.0 0.58"/>
+        <mesh filename="file://$(find picknik_ur_mock_hw_config)/meshes/table-collision.dae" scale="1 1 1"/>
       </geometry>
     </collision>
@@ -171,7 +150,7 @@
     </visual>
     <collision>
-      <origin xyz="0 0 0.29" rpy="0 0 0"/>
+      <origin xyz="0 0 0" rpy="0 0 0" />
       <geometry>
-        <box size="1.0 1.0 0.58"/>
+        <mesh filename="file://$(find picknik_ur_mock_hw_config)/meshes/table-collision.dae" scale="1 1 1"/>
       </geometry>
     </collision>

Commit message: Simplify CNC collision to fix motion planning failures when moving between `Grasp Left` and `Grasp Right` (#77)
* Simplify CNC collision

* Enable parallel planning

* Use simplifies collision DAE files

File: src/picknik_ur_mock_hw_config/description/picknik_ur_machine_tending.xacro (robot description, xacro)
@@ -89,8 +89,9 @@
       </geometry>
     </visual>
+    <!-- CNC base collision -->
     <collision>
-      <origin xyz="0 0 0" rpy="0 0 0"/>
+      <origin xyz="0 0.1 0" rpy="0 0 0"/>
       <geometry>
-        <mesh filename="file://$(find picknik_ur_mock_hw_config)/meshes/cnc.dae" scale="1 1 1"/>
+        <mesh filename="file://$(find picknik_ur_mock_hw_config)/meshes/cnc-collision.dae" scale="1 1 1"/>
       </geometry>
     </collision>
@@ -130,7 +131,7 @@
     </visual>
     <collision>
-      <origin xyz="0 0 0.29" rpy="0 0 0"/>
+      <origin xyz="0 0 0" rpy="0 0 0" />
       <geometry>
-        <box size="1.0 1.0 0.58"/>
+        <mesh filename="file://$(find picknik_ur_mock_hw_config)/meshes/table-collision.dae" scale="1 1 1"/>
       </geometry>
     </collision>
@@ -149,7 +150,7 @@
     </visual>
     <collision>
-      <origin xyz="0 0 0.29" rpy="0 0 0"/>
+      <origin xyz="0 0 0" rpy="0 0 0" />
       <geometry>
-        <box size="1.0 1.0 0.58"/>
+        <mesh filename="file://$(find picknik_ur_mock_hw_config)/meshes/table-collision.dae" scale="1 1 1"/>
       </geometry>
     </collision>

Commit message: fix offset between CNC mesh and CNC collision mesh

File: src/picknik_ur_mock_hw_config/description/picknik_ur_machine_tending.xacro (robot description, xacro)
@@ -91,5 +91,5 @@
     <!-- CNC base collision -->
     <collision>
-      <origin xyz="0 0.1 0" rpy="0 0 0"/>
+      <origin xyz="0 0 0" rpy="0 0 0"/>
       <geometry>
         <mesh filename="file://$(find picknik_ur_mock_hw_config)/meshes/cnc-collision.dae" scale="1 1 1"/>

Commit message: Move CNC machine back 5cm

File: src/picknik_ur_mock_hw_config/description/picknik_ur_machine_tending.xacro (robot description, xacro)
@@ -159,5 +159,5 @@
     <parent link="world" />
     <child link="right_hexagonal_table" />
-    <origin xyz="-0.8 0 -0.8" rpy="0 0 3.14"  />
+    <origin xyz="-0.8 0 -0.85" rpy="0 0 3.14"  />
   </joint>
   <!-- Cylinder items -->

Commit message: Whoops, bad copy-pasta

File: src/picknik_ur_mock_hw_config/description/picknik_ur_machine_tending.xacro (robot description, xacro)
@@ -100,5 +100,5 @@
     <parent link="world" />
     <child link="cnc_machine" />
-    <origin xyz="-0.1 -1.2 -0.8" rpy="0 0 3.14"  />
+    <origin xyz="-0.1 -1.25 -0.8" rpy="0 0 3.14"  />
   </joint>
   <!-- Robot base -->
@@ -159,5 +159,5 @@
     <parent link="world" />
     <child link="right_hexagonal_table" />
-    <origin xyz="-0.8 0 -0.85" rpy="0 0 3.14"  />
+    <origin xyz="-0.8 0 -0.8" rpy="0 0 3.14"  />
   </joint>
   <!-- Cylinder items -->

Commit message: Mock Hardware Scene v2.5 Cleanup (#82)
* Move CNC machine back 5cm

* Clear out waypoints

* Whoops, bad copy-pasta

* Adjust the look at machine waypoint

File: src/picknik_ur_mock_hw_config/description/picknik_ur_machine_tending.xacro (robot description, xacro)
@@ -100,5 +100,5 @@
     <parent link="world" />
     <child link="cnc_machine" />
-    <origin xyz="-0.1 -1.2 -0.8" rpy="0 0 3.14"  />
+    <origin xyz="-0.1 -1.25 -0.8" rpy="0 0 3.14"  />
   </joint>
   <!-- Robot base -->
