Commit message: Include ridgeback

File: src/picknik_ur_mobile_config/description/picknik_ur.xacro (robot description, xacro)
@@ -22,9 +22,10 @@
   <xacro:include filename="$(find picknik_ur_mujoco_config)/description/picknik_ur_attachments_macro.xacro"/>
   <xacro:include filename="$(find picknik_ur_mujoco_config)/description/picknik_ur_mujoco_ros2_control.xacro"/>
+  <xacro:include filename="$(find ridgeback_description)/urdf/ridgeback.urdf.xacro"/>
   <link name="world"/>
   <!-- Gripper and UR adapter and realsense camera -->
   <xacro:picknik_ur_attachments parent="tool0" child="grasp_link" has_tool_changer="$(arg has_tool_changer)"/>
   <!-- Linear rail -->
-  <link name="linear_rail">
+  <!--<link name="linear_rail">
     <visual>
       <origin xyz="0 0 0.05" rpy="0 0 0"/>
@@ -42,43 +43,22 @@
       </geometry>
     </collision>
-  </link>
-  <joint name="world-rail" type="fixed">
+  </link>-->
+  <!-- Ridgeback -->
+  <xacro:ridgeback/>
+  <!--<joint name="world-rail" type="fixed">
     <parent link="world" />
     <child link="linear_rail" />
     <origin xyz="0.0 0 0.6" rpy="0 0 0" />
+  </joint>-->
+  <joint name="arm_mount_joint" type="fixed">
+    <parent link="mid_mount" />
+    <child link="ur_arm_base_link" />
+    <origin xyz="0 0 0" rpy="0 0 0" />
   </joint>
   <!-- Robot: contains robot description from the world frame to the tool frame -->
-  <xacro:picknik_ur parent="ur_linear_rail_base"  child="tool0" initial_positions_file="$(arg initial_positions_file)" generate_ros2_control_tag="$(arg generate_ros2_control_tag)" >
+  <xacro:picknik_ur parent="ur_arm_base_link"  child="tool0" initial_positions_file="$(arg initial_positions_file)" generate_ros2_control_tag="$(arg generate_ros2_control_tag)" >
     <!-- Guesstimates below -->
     <origin xyz="0 -0.4 0.0" rpy="0 0 0" />
   </xacro:picknik_ur>
-  <joint name="linear_rail_joint" type="prismatic">
-    <axis xyz="0 1 0"/>
-    <parent link="linear_rail" />
-    <child link="ur_linear_rail_base" />
-    <origin xyz="0 0 0" rpy="0 0 0" />
-    <limit effort="1000.0" lower="-5.0" upper="5.0" velocity="0.175" acceleration="10.0"/>
-    <dynamics damping="20.0" friction="500.0" />
-  </joint>
-  <!-- Table -->
-  <link name="table">
-    <visual>
-      <origin xyz="0 0 0" rpy="0 0 0" />
-      <geometry>
-        <mesh filename="package://picknik_accessories/descriptions/furniture/generic_table/wood_block.dae" scale="0.125 0.125 0.00625"/>
-      </geometry>
-    </visual>
-    <collision>
-      <origin rpy="0 0 0" xyz="0 0 0"/>
-      <geometry>
-        <mesh filename="package://picknik_accessories/descriptions/furniture/generic_table/wood_block.dae" scale="0.125 0.125 0.00625"/>
-      </geometry>
-    </collision>
-  </link>
-  <joint name="table_joint" type="fixed">
-    <parent link="world" />
-    <child link="table" />
-    <origin rpy="0 0 0" xyz="1 0 0.5" />
-  </joint>
   <!-- MuJoCo Hardware interface -->
   <xacro:picknik_ur_mujoco_ros2_control />

Commit message: Move arm on ridgeback

File: src/picknik_ur_mobile_config/description/picknik_ur.xacro (robot description, xacro)
@@ -45,20 +45,23 @@
   </link>-->
   <!-- Ridgeback -->
-  <xacro:ridgeback/>
-  <!--<joint name="world-rail" type="fixed">
+  <xacro:ridgeback parent="ridgeback_base_link"/>
+  <joint name="world-rail" type="fixed">
     <parent link="world" />
-    <child link="linear_rail" />
+    <child link="ridgeback_base_link" />
     <origin xyz="0.0 0 0.6" rpy="0 0 0" />
-  </joint>-->
-  <joint name="arm_mount_joint" type="fixed">
-    <parent link="mid_mount" />
-    <child link="ur_arm_base_link" />
-    <origin xyz="0 0 0" rpy="0 0 0" />
   </joint>
   <!-- Robot: contains robot description from the world frame to the tool frame -->
-  <xacro:picknik_ur parent="ur_arm_base_link"  child="tool0" initial_positions_file="$(arg initial_positions_file)" generate_ros2_control_tag="$(arg generate_ros2_control_tag)" >
+  <xacro:picknik_ur parent="ur_linear_rail_base"  child="tool0" initial_positions_file="$(arg initial_positions_file)" generate_ros2_control_tag="$(arg generate_ros2_control_tag)" >
     <!-- Guesstimates below -->
-    <origin xyz="0 -0.4 0.0" rpy="0 0 0" />
+    <origin xyz="0 0.0 0.0" rpy="0 0 0" />
   </xacro:picknik_ur>
+  <joint name="linear_rail_joint" type="prismatic">
+    <axis xyz="0 1 0"/>
+    <parent link="mid_mount" />
+    <child link="ur_linear_rail_base" />
+    <origin xyz="0 0 0" rpy="0 0 0" />
+    <limit effort="1000.0" lower="-5.0" upper="5.0" velocity="0.175" acceleration="10.0"/>
+    <dynamics damping="20.0" friction="500.0" />
+  </joint>
   <!-- MuJoCo Hardware interface -->
   <xacro:picknik_ur_mujoco_ros2_control />

Commit message: Make ridgeback base movable

File: src/picknik_ur_mobile_config/description/picknik_ur.xacro (robot description, xacro)
@@ -46,8 +46,10 @@
   <!-- Ridgeback -->
   <xacro:ridgeback parent="ridgeback_base_link"/>
-  <joint name="world-rail" type="fixed">
+  <joint name="linear_rail_joint" type="prismatic">
     <parent link="world" />
     <child link="ridgeback_base_link" />
-    <origin xyz="0.0 0 0.6" rpy="0 0 0" />
+    <origin xyz="0 0 0" rpy="0 0 0" />
+    <limit effort="1000.0" lower="-5.0" upper="5.0" velocity="0.175" acceleration="10.0"/>
+    <dynamics damping="20.0" friction="500.0" />
   </joint>
   <!-- Robot: contains robot description from the world frame to the tool frame -->
@@ -56,11 +58,9 @@
     <origin xyz="0 0.0 0.0" rpy="0 0 0" />
   </xacro:picknik_ur>
-  <joint name="linear_rail_joint" type="prismatic">
+  <joint name="ur_ridgeback_mount" type="fixed">
     <axis xyz="0 1 0"/>
     <parent link="mid_mount" />
     <child link="ur_linear_rail_base" />
     <origin xyz="0 0 0" rpy="0 0 0" />
-    <limit effort="1000.0" lower="-5.0" upper="5.0" velocity="0.175" acceleration="10.0"/>
-    <dynamics damping="20.0" friction="500.0" />
   </joint>
   <!-- MuJoCo Hardware interface -->

Commit message: Remove rail

File: src/picknik_ur_mobile_config/description/picknik_ur.xacro (robot description, xacro)
@@ -20,28 +20,10 @@
   <!-- Import UR and environment macros -->
   <xacro:include filename="$(find picknik_ur_base_config)/description/picknik_ur_macro.xacro"/>
-  <xacro:include filename="$(find picknik_ur_mujoco_config)/description/picknik_ur_attachments_macro.xacro"/>
-  <xacro:include filename="$(find picknik_ur_mujoco_config)/description/picknik_ur_mujoco_ros2_control.xacro"/>
+  <xacro:include filename="$(find picknik_ur_mobile_config)/description/picknik_ur_attachments_macro.xacro"/>
+  <xacro:include filename="$(find picknik_ur_mobile_config)/description/picknik_ur_mujoco_ros2_control.xacro"/>
   <xacro:include filename="$(find ridgeback_description)/urdf/ridgeback.urdf.xacro"/>
   <link name="world"/>
   <!-- Gripper and UR adapter and realsense camera -->
   <xacro:picknik_ur_attachments parent="tool0" child="grasp_link" has_tool_changer="$(arg has_tool_changer)"/>
-  <!-- Linear rail -->
-  <!--<link name="linear_rail">
-    <visual>
-      <origin xyz="0 0 0.05" rpy="0 0 0"/>
-      <geometry>
-        <mesh filename="package://picknik_ur_mujoco_config/description/assets/rail.stl" />
-      </geometry>
-      <material name="grey">
-          <color rgba="0.1 0.1 0.1 1.0"/>
-        </material>
-    </visual>
-    <collision>
-      <origin xyz="0 0 0.05" rpy="0 0 0"/>
-      <geometry>
-        <mesh filename="package://picknik_ur_mujoco_config/description/assets/rail.stl" />
-      </geometry>
-    </collision>
-  </link>-->
   <!-- Ridgeback -->
   <xacro:ridgeback parent="ridgeback_base_link"/>

Commit message: Add multi-dof rail

File: src/picknik_ur_mobile_config/description/picknik_ur.xacro (robot description, xacro)
@@ -28,8 +28,17 @@
   <!-- Ridgeback -->
   <xacro:ridgeback parent="ridgeback_base_link"/>
-  <joint name="linear_rail_joint" type="prismatic">
-    <parent link="world" />
+  <link name="virual_rail_link_1"/>
+  <joint name="linear_x_joint" type="prismatic">
+    <parent link="virual_rail_link_1" />
+    <child link="virual_rail_link_2" />
+    <origin xyz="0 0 0" rpy="0 0 0" />
+    <limit effort="1000.0" lower="-5.0" upper="5.0" velocity="0.175" acceleration="10.0"/>
+    <dynamics damping="20.0" friction="500.0" />
+  </joint>
+  <link name="virual_rail_link_2"/>
+  <joint name="linear_y_joint" type="prismatic">
+    <parent link="virual_rail_link_2" />
     <child link="ridgeback_base_link" />
-    <origin xyz="0 0 0" rpy="0 0 0" />
+    <origin xyz="0 0 0" rpy="0 0 -1.5707963267948966" />
     <limit effort="1000.0" lower="-5.0" upper="5.0" velocity="0.175" acceleration="10.0"/>
     <dynamics damping="20.0" friction="500.0" />

File: src/picknik_ur_mobile_config/description/picknik_ur_mujoco_ros2_control.xacro (robot description, xacro)
@@ -3,5 +3,13 @@
   <xacro:macro name="picknik_ur_mujoco_ros2_control" >
     <ros2_control name="ur_mujoco_control" type="system">
-      <joint name="linear_rail_joint">
+      <joint name="linear_x_joint">
+          <param name="axis">1</param>
+          <command_interface name="position"/>
+          <state_interface name="position">
+          <param name="initial_value">0.0</param>
+          </state_interface>
+          <state_interface name="velocity"/>
+      </joint>
+      <joint name="linear_y_joint">
           <param name="axis">1</param>
           <command_interface name="position"/>

Commit message: Clean-up + move ground closer to robot

File: src/picknik_ur_mobile_config/description/picknik_ur.xacro (robot description, xacro)
@@ -28,4 +28,12 @@
   <!-- Ridgeback -->
   <xacro:ridgeback parent="ridgeback_base_link"/>
+  <joint name="rotational_yaw_joint" type="revolute">
+    <parent link="world"/>
+    <child link="virual_rail_link_1"/>
+    <origin rpy="0 0 0" xyz="0 0 0"/>
+    <axis xyz="0 0 1"/>
+    <limit effort="150.0" lower="-3.141592653589793" upper="3.141592653589793" velocity="0.5235987755982988"/>
+    <dynamics damping="0" friction="0"/>
+  </joint>
   <link name="virual_rail_link_1"/>
   <joint name="linear_x_joint" type="prismatic">

Commit message: Address review

File: src/picknik_ur_mobile_config/description/picknik_ur.xacro (robot description, xacro)
@@ -29,8 +29,8 @@
   <xacro:ridgeback parent="ridgeback_base_link"/>
   <joint name="rotational_yaw_joint" type="revolute">
+    <axis xyz="0 0 1"/>
     <parent link="world"/>
     <child link="virual_rail_link_1"/>
     <origin rpy="0 0 0" xyz="0 0 0"/>
-    <axis xyz="0 0 1"/>
     <limit effort="150.0" lower="-3.141592653589793" upper="3.141592653589793" velocity="0.5235987755982988"/>
     <dynamics damping="0" friction="0"/>
@@ -38,4 +38,5 @@
   <link name="virual_rail_link_1"/>
   <joint name="linear_x_joint" type="prismatic">
+    <axis xyz="1 0 0"/>
     <parent link="virual_rail_link_1" />
     <child link="virual_rail_link_2" />
@@ -46,7 +47,8 @@
   <link name="virual_rail_link_2"/>
   <joint name="linear_y_joint" type="prismatic">
+    <axis xyz="0 1 0"/>
     <parent link="virual_rail_link_2" />
     <child link="ridgeback_base_link" />
-    <origin xyz="0 0 0" rpy="0 0 -1.5707963267948966" />
+    <origin xyz="0 0 0" rpy="0 0 0" />
     <limit effort="1000.0" lower="-5.0" upper="5.0" velocity="0.175" acceleration="10.0"/>
     <dynamics damping="20.0" friction="500.0" />
