Commit message: robot and rail

File: src/picknik_ur_mujoco_config/description/picknik_ur.xacro (robot description, xacro)
@@ -22,11 +22,43 @@
   <xacro:include filename="$(find picknik_ur_mujoco_config)/description/picknik_ur_attachments_macro.xacro"/>
   <xacro:include filename="$(find picknik_ur_mujoco_config)/description/picknik_ur_mujoco_ros2_control.xacro"/>
+  <link name="world"/>
+  <!-- Gripper and UR adapter and realsense camera -->
+  <xacro:picknik_ur_attachments parent="tool0" child="grasp_link" has_tool_changer="$(arg has_tool_changer)"/>
+  <!-- Linear rail -->
+  <link name="linear_rail">
+    <visual>
+      <origin xyz="0 0 0.05" rpy="0 0 0"/>
+      <geometry>
+        <mesh filename="package://picknik_ur_mujoco_config/meshes/rail.stl" scale="0.9 0.6 0.9" />
+      </geometry>
+      <material name="grey">
+          <color rgba="0.1 0.1 0.1 1.0"/>
+        </material>
+    </visual>
+    <collision>
+      <origin xyz="0 0 0.05" rpy="0 0 0"/>
+      <geometry>
+        <mesh filename="package://picknik_ur_mujoco_config/meshes/rail.stl" scale="0.9 0.6 0.9"/>
+      </geometry>
+    </collision>
+  </link>
+  <joint name="world-rail" type="fixed">
+    <parent link="world" />
+    <child link="linear_rail" />
+    <origin xyz="0.0 0 0.6" rpy="0 0 ${pi}" />
+  </joint>
   <!-- Robot: contains robot description from the world frame to the tool frame -->
-  <xacro:picknik_ur parent="world"  child="tool0" initial_positions_file="$(arg initial_positions_file)" generate_ros2_control_tag="$(arg generate_ros2_control_tag)" >
+  <xacro:picknik_ur parent="ur_linear_rail_base"  child="tool0" initial_positions_file="$(arg initial_positions_file)" generate_ros2_control_tag="$(arg generate_ros2_control_tag)" >
     <!-- Guesstimates below -->
     <origin xyz="0 -0.4 0.0" rpy="0 0 0" />
   </xacro:picknik_ur>
-  <!-- Gripper and UR adapter and realsense camera -->
-  <xacro:picknik_ur_attachments parent="tool0" child="grasp_link" has_tool_changer="$(arg has_tool_changer)"/>
+  <joint name="linear_rail_joint" type="prismatic">
+    <axis xyz="0 1 0"/>
+    <parent link="linear_rail" />
+    <child link="ur_linear_rail_base" />
+    <origin xyz="0 0 0" rpy="0 0 0" />
+    <limit effort="1000.0" lower="-1.0" upper="1.0" velocity="0.175"/>
+    <dynamics damping="20.0" friction="500.0" />
+  </joint>
   <!-- MuJoCo Hardware interface -->
   <xacro:picknik_ur_mujoco_ros2_control />

File: src/picknik_ur_mujoco_config/description/picknik_ur_mujoco_ros2_control.xacro (robot description, xacro)
@@ -3,4 +3,12 @@
   <xacro:macro name="picknik_ur_mujoco_ros2_control" >
     <ros2_control name="ur_mujoco_control" type="system">
+      <joint name="linear_rail_joint">
+          <param name="axis">1</param>
+          <command_interface name="position"/>
+          <state_interface name="position">
+          <param name="initial_value">0.0</param>
+          </state_interface>
+          <state_interface name="velocity"/>
+      </joint>
       <joint name="shoulder_pan_joint">
           <command_interface name="position">
@@ -100,5 +108,5 @@
           <plugin>picknik_mujoco_ros/MujocoSystem</plugin>
           <param name="mujoco_model">description/scene.xml</param>
-          <param name="mujoco_model_package">picknik_ur_mujoco_config</param>
+          <param name="mujoco_model_package">picknik_ur_mujoco_kitchen_config</param>
           <param name="render_publish_rate">10</param>
           <param name="tf_publish_rate">60</param>

Commit message: formatting

File: src/picknik_ur_mujoco_config/description/picknik_ur.xacro (robot description, xacro)
@@ -30,5 +30,5 @@
       <origin xyz="0 0 0.05" rpy="0 0 0"/>
       <geometry>
-        <mesh filename="package://picknik_ur_mujoco_config/meshes/rail.stl" scale="0.9 0.6 0.9" />
+        <mesh filename="package://picknik_ur_mujoco_config/description/assets/rail.stl" scale="0.9 0.6 0.9" />
       </geometry>
       <material name="grey">
@@ -39,5 +39,5 @@
       <origin xyz="0 0 0.05" rpy="0 0 0"/>
       <geometry>
-        <mesh filename="package://picknik_ur_mujoco_config/meshes/rail.stl" scale="0.9 0.6 0.9"/>
+        <mesh filename="package://picknik_ur_mujoco_config/description/assets/rail.stl" scale="0.9 0.6 0.9"/>
       </geometry>
     </collision>
@@ -58,5 +58,5 @@
     <child link="ur_linear_rail_base" />
     <origin xyz="0 0 0" rpy="0 0 0" />
-    <limit effort="1000.0" lower="-1.0" upper="1.0" velocity="0.175"/>
+    <limit effort="1000.0" lower="-1.0" upper="1.0" velocity="0.175" acceleration="10.0"/>
     <dynamics damping="20.0" friction="500.0" />
   </joint>

File: src/picknik_ur_mujoco_config/description/picknik_ur_attachments_macro.xacro (robot description, xacro)
@@ -35,254 +35,254 @@
             <xacro:property name="sim_ignition" default="false"/>
         </xacro:if>
-        <!-- Add robotiq 2f 85 gripper model -->
-        <link name="robotiq_85_base_link">
-        <visual>
-            <geometry>
-            <mesh filename="package://robotiq_description/meshes/visual/2f_85/robotiq_base.dae"/>
-            </geometry>
-        </visual>
-        <collision>
-            <geometry>
-            <mesh filename="package://robotiq_description/meshes/collision/2f_85/robotiq_base.stl"/>
-            </geometry>
-        </collision>
-        <inertial>
-            <origin rpy="0 0 0" xyz="0.0 2.274e-05 0.03232288"/>
-            <mass value="6.6320197e-01"/>
-            <inertia ixx="5.1617816e-04" ixy="2.936e-8" ixz="0.0" iyy="5.8802208e-04" iyz="-3.2296e-7" izz="3.9462776e-04"/>
-        </inertial>
-        </link>
-        <link name="robotiq_85_left_knuckle_link">
-        <visual>
-            <geometry>
-            <mesh filename="package://robotiq_description/meshes/visual/2f_85/left_knuckle.dae"/>
-            </geometry>
-        </visual>
-        <collision>
-            <geometry>
-            <mesh filename="package://robotiq_description/meshes/collision/2f_85/left_knuckle.stl"/>
-            </geometry>
-        </collision>
-        <inertial>
-            <origin rpy="0 0 0" xyz="0.01213197 0.0002 -0.00058647"/>
-            <mass value="1.384773208e-02"/>
-            <inertia ixx="3.5232e-7" ixy="0.0" ixz="1.1744e-7" iyy="2.31944e-6" iyz="0" izz="2.23136e-6"/>
-        </inertial>
-        </link>
-        <link name="robotiq_85_right_knuckle_link">
-        <visual>
-            <geometry>
-            <mesh filename="package://robotiq_description/meshes/visual/2f_85/right_knuckle.dae"/>
-            </geometry>
-        </visual>
-        <collision>
-            <geometry>
-            <mesh filename="package://robotiq_description/meshes/collision/2f_85/right_knuckle.stl"/>
-            </geometry>
-        </collision>
-        <inertial>
-            <origin rpy="0 0 0" xyz="-0.01213197 0.0002 -0.00058647"/>
-            <mass value="1.384773208e-02"/>
-            <inertia ixx="3.5232e-7" ixy="0.0" ixz="-1.1744e-7" iyy="2.31944e-6" iyz="0.0" izz="2.23136e-6"/>
-        </inertial>
-        </link>
-        <link name="robotiq_85_left_finger_link">
-        <visual>
-            <geometry>
-            <mesh filename="package://robotiq_description/meshes/visual/2f_85/left_finger.dae"/>
-            </geometry>
-        </visual>
-        <collision>
-            <geometry>
-            <mesh filename="package://robotiq_description/meshes/collision/2f_85/left_finger.stl"/>
-            </geometry>
-        </collision>
-        <inertial>
-            <origin rpy="0 0 0" xyz="0.00346899 -0.00079447 0.01867121"/>
-            <mass value="4.260376752e-02"/>
-            <inertia ixx="1.385792000000000e-05" ixy="0.0" ixz="-2.17264e-06" iyy="1.183208e-05" iyz="0.0" izz="5.19672e-06"/>
-        </inertial>
-        </link>
-        <link name="robotiq_85_right_finger_link">
-        <visual>
-            <geometry>
-            <mesh filename="package://robotiq_description/meshes/visual/2f_85/right_finger.dae"/>
-            </geometry>
-        </visual>
-        <collision>
-            <geometry>
-            <mesh filename="package://robotiq_description/meshes/collision/2f_85/right_finger.stl"/>
-            </geometry>
-        </collision>
-        <inertial>
-            <origin rpy="0 0 0" xyz="-0.00346899 -5.53e-06 0.01867121"/>
-            <mass value="4.260376752000000e-02"/>
-            <inertia ixx="1.385792e-05" ixy="0.0" ixz="2.17264e-06" iyy="1.183208e-05" iyz="0.0" izz="5.19672e-06"/>
-        </inertial>
-        </link>
-        <link name="robotiq_85_left_inner_knuckle_link">
-        <visual>
-            <geometry>
-            <mesh filename="package://robotiq_description/meshes/visual/2f_85/left_inner_knuckle.dae"/>
-            </geometry>
-        </visual>
-        <collision>
-            <geometry>
-            <mesh filename="package://robotiq_description/meshes/collision/2f_85/left_inner_knuckle.stl"/>
-            </geometry>
-        </collision>
-        <inertial>
-            <origin rpy="0 0 0" xyz="0.01897699 0.00015001 0.02247101"/>
-            <mass value="2.969376448e-02"/>
-            <inertia ixx="9.57136e-06" ixy="0.0" ixz="-3.93424e-06" iyy="8.69056e-06" iyz="0.0" izz="8.19144e-06"/>
-        </inertial>
-        </link>
-        <link name="robotiq_85_right_inner_knuckle_link">
-        <visual>
-            <geometry>
-            <mesh filename="package://robotiq_description/meshes/visual/2f_85/right_inner_knuckle.dae"/>
-            </geometry>
-        </visual>
-        <collision>
-            <geometry>
-            <mesh filename="package://robotiq_description/meshes/collision/2f_85/right_inner_knuckle.stl"/>
-            </geometry>
-        </collision>
-        <inertial>
-            <origin rpy="0 0 0" xyz="-0.01926824 5.001e-05 0.02222178"/>
-            <mass value="2.969376448e-02"/>
-            <inertia ixx="9.42456e-06" ixy="0.0" ixz="3.9636e-06" iyy="8.69056e-06" iyz="0.0" izz="8.33824e-06"/>
-        </inertial>
-        </link>
-        <link name="robotiq_85_left_finger_tip_link">
-        <visual>
-            <geometry>
-            <mesh filename="package://robotiq_description/meshes/visual/2f_85/left_finger_tip.dae"/>
-            </geometry>
-        </visual>
-        <collision>
-            <geometry>
-            <mesh filename="package://robotiq_description/meshes/collision/2f_85/left_finger_tip.stl"/>
-            </geometry>
-            <surface>
-            <friction>
-                <ode>
-                <mu1>100000.0</mu1>
-                <mu2>100000.0</mu2>
-                </ode>
-            </friction>
-            <contact>
-                <ode>
-                <kp>1e+5</kp>
-                <kd>1</kd>
-                <soft_cfm>0</soft_cfm>
-                <soft_erp>0.2</soft_erp>
-                <minDepth>0.002</minDepth>
-                <maxVel>0</maxVel>
-                </ode>
-            </contact>
-            </surface>
-        </collision>
-        <inertial>
-            <origin rpy="0 0 0" xyz="-0.01456706 -0.0008 0.01649701"/>
-            <mass value="4.268588744e-02"/>
-            <inertia ixx="1.048152e-05" ixy="0.0" ixz="3.5232e-6" iyy="1.197888e-05" iyz="0.0" izz="4.22784e-06"/>
-        </inertial>
-        </link>
-        <link name="robotiq_85_right_finger_tip_link">
-        <visual>
-            <geometry>
-            <mesh filename="package://robotiq_description/meshes/visual/2f_85/right_finger_tip.dae"/>
-            </geometry>
-        </visual>
-        <collision>
-            <geometry>
-            <mesh filename="package://robotiq_description/meshes/collision/2f_85/right_finger_tip.stl"/>
-            </geometry>
-            <surface>
-            <friction>
-                <ode>
-                <mu1>100000.0</mu1>
-                <mu2>100000.0</mu2>
-                </ode>
-            </friction>
-            <contact>
-                <ode>
-                <kp>1e+5</kp>
-                <kd>1</kd>
-                <soft_cfm>0</soft_cfm>
-                <soft_erp>0.2</soft_erp>
-                <minDepth>0.002</minDepth>
-                <maxVel>0</maxVel>
-                </ode>
-            </contact>
-            </surface>
-        </collision>
-        <inertial>
-            <origin rpy="0 0 0" xyz="0.01456706 5e-05 0.01649701"/>
-            <mass value="4.268588744e-02"/>
-            <inertia ixx="1.048152e-05" ixy="0.0" ixz="-3.5232e-06" iyy="1.197888e-05" iyz="0.0" izz="4.22784e-06"/>
-        </inertial>
-        </link>
-        <joint name="robotiq_85_base_joint" type="fixed">
-        <parent link="${prefix_}gripper_mount_link"/>
-        <child link="robotiq_85_base_link"/>
-        <origin rpy="0 0 0" xyz="0 0 0"/>
-        </joint>
-        <joint name="robotiq_85_left_knuckle_joint" type="revolute">
-        <parent link="robotiq_85_base_link"/>
-        <child link="robotiq_85_left_knuckle_link"/>
-        <axis xyz="0 -1 0"/>
-        <origin rpy="0 0 0" xyz="0.03060114 0.0 0.05490452"/>
-        <limit effort="50" lower="0.0" upper="0.8" velocity="0.5"/>
-        </joint>
-        <joint name="robotiq_85_right_knuckle_joint" type="revolute">
-        <parent link="robotiq_85_base_link"/>
-        <child link="robotiq_85_right_knuckle_link"/>
-        <axis xyz="0 1 0"/>
-        <origin rpy="0 0 0" xyz="-0.03060114 0.0 0.05490452"/>
-        <limit effort="50" lower="0.0" upper="0.8" velocity="0.5"/>
-        <mimic joint="robotiq_85_left_knuckle_joint" multiplier="1"/>
-        </joint>
-        <joint name="robotiq_85_left_finger_joint" type="continuous">
-        <parent link="robotiq_85_left_knuckle_link"/>
-        <child link="robotiq_85_left_finger_link"/>
-        <axis xyz="0 -1 0"/>
-        <origin rpy="0 0 0" xyz="0.03152616 0.0 -0.00376347"/>
-        </joint>
-        <joint name="robotiq_85_right_finger_joint" type="continuous">
-        <parent link="robotiq_85_right_knuckle_link"/>
-        <child link="robotiq_85_right_finger_link"/>
-        <axis xyz="0 1 0"/>
-        <origin rpy="0 0 0" xyz="-0.03152616 0.0 -0.00376347"/>
-        </joint>
-        <joint name="robotiq_85_left_inner_knuckle_joint" type="continuous">
-        <parent link="robotiq_85_base_link"/>
-        <child link="robotiq_85_left_inner_knuckle_link"/>
-        <axis xyz="0 -1 0"/>
-        <origin rpy="0 0 0" xyz="0.0127 0.0 0.06142"/>
-        <mimic joint="robotiq_85_left_knuckle_joint" multiplier="1"/>
-        </joint>
-        <joint name="robotiq_85_right_inner_knuckle_joint" type="continuous">
-        <parent link="robotiq_85_base_link"/>
-        <child link="robotiq_85_right_inner_knuckle_link"/>
-        <axis xyz="0 1 0"/>
-        <origin rpy="0 0 0" xyz="-0.0127 0.0 0.06142"/>
-        <mimic joint="robotiq_85_left_knuckle_joint" multiplier="1"/>
-        </joint>
-        <joint name="robotiq_85_left_finger_tip_joint" type="continuous">
-        <parent link="robotiq_85_left_finger_link"/>
-        <child link="robotiq_85_left_finger_tip_link"/>
-        <axis xyz="0 -1 0"/>
-        <origin rpy="0 0 0" xyz="0.00563134 0.0 0.04718515"/>
-        <mimic joint="robotiq_85_left_knuckle_joint" multiplier="-1"/>
-        </joint>
-        <joint name="robotiq_85_right_finger_tip_joint" type="continuous">
-        <parent link="robotiq_85_right_finger_link"/>
-        <child link="robotiq_85_right_finger_tip_link"/>
-        <axis xyz="0 1 0"/>
-        <origin rpy="0 0 0" xyz="-0.00563134 0.0 0.04718515"/>
-        <mimic joint="robotiq_85_left_knuckle_joint" multiplier="-1"/>
-        </joint>
+    <!-- Add robotiq 2f 85 gripper model -->
+    <link name="robotiq_85_base_link">
+      <visual>
+        <geometry>
+          <mesh filename="package://robotiq_description/meshes/visual/2f_85/robotiq_base.dae"/>
+        </geometry>
+      </visual>
+      <collision>
+        <geometry>
+          <mesh filename="package://robotiq_description/meshes/collision/2f_85/robotiq_base.stl"/>
+        </geometry>
+      </collision>
+      <inertial>
+        <origin rpy="0 0 0" xyz="0.0 2.274e-05 0.03232288"/>
+        <mass value="6.6320197e-01"/>
+        <inertia ixx="5.1617816e-04" ixy="2.936e-8" ixz="0.0" iyy="5.8802208e-04" iyz="-3.2296e-7" izz="3.9462776e-04"/>
+      </inertial>
+    </link>
+    <link name="robotiq_85_left_knuckle_link">
+      <visual>
+        <geometry>
+          <mesh filename="package://robotiq_description/meshes/visual/2f_85/left_knuckle.dae"/>
+        </geometry>
+      </visual>
+      <collision>
+        <geometry>
+          <mesh filename="package://robotiq_description/meshes/collision/2f_85/left_knuckle.stl"/>
+        </geometry>
+      </collision>
+      <inertial>
+        <origin rpy="0 0 0" xyz="0.01213197 0.0002 -0.00058647"/>
+        <mass value="1.384773208e-02"/>
+        <inertia ixx="3.5232e-7" ixy="0.0" ixz="1.1744e-7" iyy="2.31944e-6" iyz="0" izz="2.23136e-6"/>
+      </inertial>
+    </link>
+    <link name="robotiq_85_right_knuckle_link">
+      <visual>
+        <geometry>
+          <mesh filename="package://robotiq_description/meshes/visual/2f_85/right_knuckle.dae"/>
+        </geometry>
+      </visual>
+      <collision>
+        <geometry>
+          <mesh filename="package://robotiq_description/meshes/collision/2f_85/right_knuckle.stl"/>
+        </geometry>
+      </collision>
+      <inertial>
+        <origin rpy="0 0 0" xyz="-0.01213197 0.0002 -0.00058647"/>
+        <mass value="1.384773208e-02"/>
+        <inertia ixx="3.5232e-7" ixy="0.0" ixz="-1.1744e-7" iyy="2.31944e-6" iyz="0.0" izz="2.23136e-6"/>
+      </inertial>
+    </link>
+    <link name="robotiq_85_left_finger_link">
+      <visual>
+        <geometry>
+          <mesh filename="package://robotiq_description/meshes/visual/2f_85/left_finger.dae"/>
+        </geometry>
+      </visual>
+      <collision>
+        <geometry>
+          <mesh filename="package://robotiq_description/meshes/collision/2f_85/left_finger.stl"/>
+        </geometry>
+      </collision>
+      <inertial>
+        <origin rpy="0 0 0" xyz="0.00346899 -0.00079447 0.01867121"/>
+        <mass value="4.260376752e-02"/>
+        <inertia ixx="1.385792000000000e-05" ixy="0.0" ixz="-2.17264e-06" iyy="1.183208e-05" iyz="0.0" izz="5.19672e-06"/>
+      </inertial>
+    </link>
+    <link name="robotiq_85_right_finger_link">
+      <visual>
+        <geometry>
+          <mesh filename="package://robotiq_description/meshes/visual/2f_85/right_finger.dae"/>
+        </geometry>
+      </visual>
+      <collision>
+        <geometry>
+          <mesh filename="package://robotiq_description/meshes/collision/2f_85/right_finger.stl"/>
+        </geometry>
+      </collision>
+      <inertial>
+        <origin rpy="0 0 0" xyz="-0.00346899 -5.53e-06 0.01867121"/>
+        <mass value="4.260376752000000e-02"/>
+        <inertia ixx="1.385792e-05" ixy="0.0" ixz="2.17264e-06" iyy="1.183208e-05" iyz="0.0" izz="5.19672e-06"/>
+      </inertial>
+    </link>
+    <link name="robotiq_85_left_inner_knuckle_link">
+      <visual>
+        <geometry>
+          <mesh filename="package://robotiq_description/meshes/visual/2f_85/left_inner_knuckle.dae"/>
+        </geometry>
+      </visual>
+      <collision>
+        <geometry>
+          <mesh filename="package://robotiq_description/meshes/collision/2f_85/left_inner_knuckle.stl"/>
+        </geometry>
+      </collision>
+      <inertial>
+        <origin rpy="0 0 0" xyz="0.01897699 0.00015001 0.02247101"/>
+        <mass value="2.969376448e-02"/>
+        <inertia ixx="9.57136e-06" ixy="0.0" ixz="-3.93424e-06" iyy="8.69056e-06" iyz="0.0" izz="8.19144e-06"/>
+      </inertial>
+    </link>
+    <link name="robotiq_85_right_inner_knuckle_link">
+      <visual>
+        <geometry>
+          <mesh filename="package://robotiq_description/meshes/visual/2f_85/right_inner_knuckle.dae"/>
+        </geometry>
+      </visual>
+      <collision>
+        <geometry>
+          <mesh filename="package://robotiq_description/meshes/collision/2f_85/right_inner_knuckle.stl"/>
+        </geometry>
+      </collision>
+      <inertial>
+        <origin rpy="0 0 0" xyz="-0.01926824 5.001e-05 0.02222178"/>
+        <mass value="2.969376448e-02"/>
+        <inertia ixx="9.42456e-06" ixy="0.0" ixz="3.9636e-06" iyy="8.69056e-06" iyz="0.0" izz="8.33824e-06"/>
+      </inertial>
+    </link>
+    <link name="robotiq_85_left_finger_tip_link">
+      <visual>
+        <geometry>
+          <mesh filename="package://robotiq_description/meshes/visual/2f_85/left_finger_tip.dae"/>
+        </geometry>
+      </visual>
+      <collision>
+        <geometry>
+          <mesh filename="package://robotiq_description/meshes/collision/2f_85/left_finger_tip.stl"/>
+        </geometry>
+        <surface>
+          <friction>
+            <ode>
+              <mu1>100000.0</mu1>
+              <mu2>100000.0</mu2>
+            </ode>
+          </friction>
+          <contact>
+            <ode>
+              <kp>1e+5</kp>
+              <kd>1</kd>
+              <soft_cfm>0</soft_cfm>
+              <soft_erp>0.2</soft_erp>
+              <minDepth>0.002</minDepth>
+              <maxVel>0</maxVel>
+            </ode>
+          </contact>
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
File: src/picknik_ur_mujoco_config/description/picknik_ur_mujoco_ros2_control.xacro (robot description, xacro)
@@ -89,24 +89,8 @@
           <state_interface name="velocity"/>
       </joint>
-      <joint name="robotiq_85_left_inner_knuckle_joint">
-          <state_interface name="position"/>
-          <state_interface name="velocity"/>
-      </joint>
-      <joint name="robotiq_85_right_inner_knuckle_joint">
-          <state_interface name="position"/>
-          <state_interface name="velocity"/>
-      </joint>
-      <joint name="robotiq_85_left_finger_tip_joint">
-          <state_interface name="position"/>
-          <state_interface name="velocity"/>
-      </joint>
-      <joint name="robotiq_85_right_finger_tip_joint">
-          <state_interface name="position"/>
-          <state_interface name="velocity"/>
-      </joint>
       <hardware>
           <plugin>picknik_mujoco_ros/MujocoSystem</plugin>
           <param name="mujoco_model">description/scene.xml</param>
-          <param name="mujoco_model_package">picknik_ur_mujoco_kitchen_config</param>
+          <param name="mujoco_model_package">picknik_ur_mujoco_config</param>
           <param name="render_publish_rate">10</param>
           <param name="tf_publish_rate">60</param>
