Commit message: wip

File: src/picknik_ur_mujoco_config/description/picknik_ur.xacro (robot description, xacro)
@@ -30,5 +30,5 @@
       <origin xyz="0 0 0.05" rpy="0 0 0"/>
       <geometry>
-        <mesh filename="package://picknik_ur_mujoco_config/description/assets/rail.stl" scale="0.9 0.6 0.9" />
+        <mesh filename="package://picknik_ur_mujoco_config/description/assets/rail.stl" />
       </geometry>
       <material name="grey">
@@ -39,5 +39,5 @@
       <origin xyz="0 0 0.05" rpy="0 0 0"/>
       <geometry>
-        <mesh filename="package://picknik_ur_mujoco_config/description/assets/rail.stl" scale="0.9 0.6 0.9"/>
+        <mesh filename="package://picknik_ur_mujoco_config/description/assets/rail.stl" />
       </geometry>
     </collision>
@@ -46,5 +46,5 @@
     <parent link="world" />
     <child link="linear_rail" />
-    <origin xyz="0.0 0 0.6" rpy="0 0 ${pi}" />
+    <origin xyz="0.0 0 0.6" rpy="0 0 0" />
   </joint>
   <!-- Robot: contains robot description from the world frame to the tool frame -->
@@ -61,4 +61,24 @@
     <dynamics damping="20.0" friction="500.0" />
   </joint>
+  <!-- Table -->
+  <link name="table">
+    <visual>
+      <origin xyz="0 0 0" rpy="0 0 0" />
+      <geometry>
+        <mesh filename="package://picknik_accessories/descriptions/furniture/generic_table/wood_block.dae" scale="0.125 0.125 0.00625"/>
+      </geometry>
+    </visual>
+    <collision>
+      <origin rpy="0 0 0" xyz="0 0 0"/>
+      <geometry>
+        <mesh filename="package://picknik_accessories/descriptions/furniture/generic_table/wood_block.dae" scale="0.125 0.125 0.00625"/>
+      </geometry>
+    </collision>
+  </link>
+  <joint name="table_joint" type="fixed">
+    <parent link="world" />
+    <child link="table" />
+    <origin rpy="0 0 0" xyz="1 0 0.5" />
+  </joint>
   <!-- MuJoCo Hardware interface -->
   <xacro:picknik_ur_mujoco_ros2_control />

Commit message: Updated linear rail limits

File: src/picknik_ur_mujoco_config/description/picknik_ur.xacro (robot description, xacro)
@@ -58,5 +58,5 @@
     <child link="ur_linear_rail_base" />
     <origin xyz="0 0 0" rpy="0 0 0" />
-    <limit effort="1000.0" lower="-1.0" upper="1.0" velocity="0.175" acceleration="10.0"/>
+    <limit effort="1000.0" lower="-5.0" upper="5.0" velocity="0.175" acceleration="10.0"/>
     <dynamics damping="20.0" friction="500.0" />
   </joint>

Commit message: Use auto-generated description file

File: src/picknik_ur_mujoco_config/description/picknik_ur.xacro (robot description, xacro)
@@ -1,68 +1,875 @@
-<?xml version="1.0"?>
-<robot xmlns:xacro="http://wiki.ros.org/xacro" name="$(arg name)">
-  <!-- parameters -->
-  <xacro:arg name="use_fake_hardware" default="false"/>
-  <xacro:arg name="external_camera" default="false"/>
-  <xacro:arg name="has_tool_changer" default="true"/>
-  <xacro:arg name="use_pinch_links" default="true"/>
-  <xacro:arg name="generate_ros2_control_tag" default="false"/>
-  <xacro:arg name="name" default=""/>
-  <xacro:arg name="joint_limits_parameters_file" default=""/>
-  <xacro:arg name="kinematics_parameters_file" default=""/>
-  <xacro:arg name="physical_parameters_file" default=""/>
-  <xacro:arg name="visual_parameters_file" default=""/>
-  <xacro:arg name="headless_mode" default="false"/>
-  <xacro:arg name="robot_ip" default="0.0.0.0"/>
-  <xacro:arg name="use_tool_communication" default="false"/>
-  <xacro:arg name="tool_voltage" default="0"/>
-  <xacro:arg name="tool_device_name" default="/dev/ttyUSB0"/>
-  <xacro:arg name="initial_positions_file" default="$(find picknik_ur_base_config)/config/initial_positions.yaml"/>
-  <!-- Import UR and environment macros -->
-  <xacro:include filename="$(find picknik_ur_base_config)/description/picknik_ur_macro.xacro"/>
-  <xacro:include filename="$(find picknik_ur_mujoco_config)/description/picknik_ur_attachments_macro.xacro"/>
-  <xacro:include filename="$(find picknik_ur_mujoco_config)/description/picknik_ur_mujoco_ros2_control.xacro"/>
+<?xml version="1.0" ?>
+<robot name="ur5e" xmlns:xacro="http://ros.org/wiki/xacro">
+  <xacro:arg name="mujoco_model" default="description/scene.xml" />
+  <material name="aluminum">
+    <color rgba="0.5 0.5 0.5 1"/>
+  </material>
+  <material name="plastic">
+    <color rgba="0.1 0.1 0.1 1"/>
+  </material>
   <link name="world"/>
-  <!-- Gripper and UR adapter and realsense camera -->
-  <xacro:picknik_ur_attachments parent="tool0" child="grasp_link" has_tool_changer="$(arg has_tool_changer)"/>
+  <joint name="tool_changer_joint" type="fixed">
+    <!-- The parent link must be read from the robot model it is attached to. -->
+    <parent link="tool0"/>
+    <child link="tool_changer_link"/>
+    <origin rpy="0 0 0" xyz="0 0 0"/>
+  </joint>
+  <link name="tool_changer_link">
+    <visual>
+      <origin rpy="0 0 0" xyz="0 0 0"/>
+      <geometry>
+        <mesh filename="package://picknik_accessories/descriptions/brackets/mtc_ur_tool_changer/mtc_ur3510_ur_toolchanger.dae"/>
+      </geometry>
+    </visual>
+    <collision>
+      <origin rpy="0 0 0" xyz="0 0 0"/>
+      <geometry>
+        <mesh filename="package://picknik_accessories/descriptions/brackets/mtc_ur_tool_changer/mtc_ur3510_ur_toolchanger_collision.stl"/>
+      </geometry>
+    </collision>
+  </link>
+  <joint name="tool_side_joint" type="fixed">
+    <parent link="tool_changer_link"/>
+    <child link="tool_changer_tool0"/>
+    <origin rpy="0 0 0" xyz="0 0 0.0331"/>
+  </joint>
+  <link name="tool_changer_tool0"/>
+  <joint name="realsense_camera_adapter_joint" type="fixed">
+    <!-- The parent link must be read from the robot model it is attached to. -->
+    <parent link="tool_changer_tool0"/>
+    <child link="realsense_camera_adapter_link"/>
+    <origin rpy="0 0 0" xyz="0 0 0"/>
+  </joint>
+  <link name="realsense_camera_adapter_link">
+    <visual>
+      <origin rpy="0 0 0" xyz="0 0 0"/>
+      <geometry>
+        <mesh filename="package://picknik_accessories/descriptions/brackets/ur_realsense_camera_adapter/picknik_ur5_realsense_camera_adapter_rev2.dae"/>
+      </geometry>
+    </visual>
+    <collision>
+      <origin rpy="0 0 0" xyz="0 0 0"/>
+      <geometry>
+        <mesh filename="package://picknik_accessories/descriptions/brackets/ur_realsense_camera_adapter/picknik_ur5_realsense_camera_adapter_rev2_collision.stl"/>
+      </geometry>
+    </collision>
+  </link>
+  <link name="realsense_camera_adapter_tool0"/>
+  <joint name="realsense_camera_adapter_tool0_joint" type="fixed">
+    <parent link="realsense_camera_adapter_link"/>
+    <child link="realsense_camera_adapter_tool0"/>
+    <origin rpy="0 0 0" xyz="0 0 0.007"/>
+  </joint>
+  <link name="d415_mount_link"/>
+  <joint name="d415_mount_joint" type="fixed">
+    <parent link="realsense_camera_adapter_link"/>
+    <child link="d415_mount_link"/>
+    <origin rpy="0 -1.4660765716752369 1.5707963267948966" xyz="0 -0.067 0.0171"/>
+  </joint>
+  <link name="l515_mount_link"/>
+  <joint name="l515_mount_joint" type="fixed">
+    <parent link="realsense_camera_adapter_link"/>
+    <child link="l515_mount_link"/>
+    <origin rpy="0 -1.4660765716752369 1.5707963267948966" xyz="0 -0.0406 0.0173"/>
+  </joint>
+  <!-- camera body, with origin at bottom screw mount -->
+  <joint name="wrist_mounted_camera_joint" type="fixed">
+    <origin rpy="0 0 0" xyz="0 0 0"/>
+    <parent link="d415_mount_link"/>
+    <child link="wrist_mounted_camera_bottom_screw_frame"/>
+  </joint>
+  <link name="wrist_mounted_camera_bottom_screw_frame"/>
+  <joint name="wrist_mounted_camera_link_joint" type="fixed">
+    <origin rpy="0 0 0" xyz="0 0.02 0.0115"/>
+    <parent link="wrist_mounted_camera_bottom_screw_frame"/>
+    <child link="wrist_mounted_camera_link"/>
+  </joint>
+  <link name="wrist_mounted_camera_link">
+    <visual>
+      <origin rpy="1.5707963267948966 0 1.5707963267948966" xyz="0.00987 -0.02 0"/>
+      <geometry>
+        <mesh filename="package://realsense2_description/meshes/d415.stl"/>
+      </geometry>
+      <material name="rs_aluminum">
+        <color rgba="0.5 0.5 0.5 1.0"/>
+      </material>
+    </visual>
+    <collision>
+      <origin rpy="0 0 0" xyz="0 -0.02 0"/>
+      <geometry>
+        <box size="0.02005 0.099 0.023"/>
+      </geometry>
+    </collision>
+    <inertial>
+      <mass value="0.072"/>
+      <!-- The following are not reliable values, and should not be used for modeling -->
+      <origin xyz="0 0 0"/>
+      <inertia ixx="0.003881243" ixy="0.0" ixz="0.0" iyy="0.000498940" iyz="0.0" izz="0.003879257"/>
+    </inertial>
+  </link>
+  <!-- camera depth joints and links -->
+  <joint name="wrist_mounted_camera_depth_joint" type="fixed">
+    <origin rpy="0 0 0" xyz="0 0 0"/>
+    <parent link="wrist_mounted_camera_link"/>
+    <child link="wrist_mounted_camera_depth_frame"/>
+  </joint>
+  <link name="wrist_mounted_camera_depth_frame"/>
+  <joint name="wrist_mounted_camera_depth_optical_joint" type="fixed">
+    <origin rpy="-1.5707963267948966 0 -1.5707963267948966" xyz="0 0 0"/>
+    <parent link="wrist_mounted_camera_depth_frame"/>
+    <child link="wrist_mounted_camera_depth_optical_frame"/>
+  </joint>
+  <link name="wrist_mounted_camera_depth_optical_frame"/>
+  <!-- camera left IR joints and links -->
+  <joint name="wrist_mounted_camera_infra1_joint" type="fixed">
+    <origin rpy="0 0 0" xyz="0 0.0 0"/>
+    <parent link="wrist_mounted_camera_link"/>
+    <child link="wrist_mounted_camera_infra1_frame"/>
+  </joint>
+  <link name="wrist_mounted_camera_infra1_frame"/>
+  <joint name="wrist_mounted_camera_infra1_optical_joint" type="fixed">
+    <origin rpy="-1.5707963267948966 0 -1.5707963267948966" xyz="0 0 0"/>
+    <parent link="wrist_mounted_camera_infra1_frame"/>
+    <child link="wrist_mounted_camera_infra1_optical_frame"/>
+  </joint>
+  <link name="wrist_mounted_camera_infra1_optical_frame"/>
+  <!-- camera right IR joints and links -->
+  <joint name="wrist_mounted_camera_infra2_joint" type="fixed">
+    <origin rpy="0 0 0" xyz="0 -0.055 0"/>
+    <parent link="wrist_mounted_camera_link"/>
+    <child link="wrist_mounted_camera_infra2_frame"/>
+  </joint>
+  <link name="wrist_mounted_camera_infra2_frame"/>
+  <joint name="wrist_mounted_camera_infra2_optical_joint" type="fixed">
+    <origin rpy="-1.5707963267948966 0 -1.5707963267948966" xyz="0 0 0"/>
+    <parent link="wrist_mounted_camera_infra2_frame"/>
+    <child link="wrist_mounted_camera_infra2_optical_frame"/>
+  </joint>
+  <link name="wrist_mounted_camera_infra2_optical_frame"/>
+  <!-- camera color joints and links -->
+  <joint name="wrist_mounted_camera_color_joint" type="fixed">
+    <origin rpy="0 0 0" xyz="0 0.015 0"/>
+    <parent link="wrist_mounted_camera_link"/>
+    <child link="wrist_mounted_camera_color_frame"/>
+  </joint>
+  <link name="wrist_mounted_camera_color_frame"/>
+  <joint name="wrist_mounted_camera_color_optical_joint" type="fixed">
+    <origin rpy="-1.5707963267948966 0 -1.5707963267948966" xyz="0 0 0"/>
+    <parent link="wrist_mounted_camera_color_frame"/>
+    <child link="wrist_mounted_camera_color_optical_frame"/>
+  </joint>
+  <link name="wrist_mounted_camera_color_optical_frame"/>
+  <gazebo reference="wrist_mounted_camera_color_frame">
+    <sensor name="wrist_mounted_camera_rgbd_sensor" type="rgbd_camera">
+      <camera>
+        <horizontal_fov>1.047</horizontal_fov>
+        <image>
+          <width>640</width>
+          <height>480</height>
+          <format>RGB_INT8</format>
+        </image>
+        <clip>
+          <near>0.1</near>
+          <far>5</far>
+        </clip>
+        <distortion>
+          <k1>0.0</k1>
+          <k2>0.0</k2>
+          <k3>0.0</k3>
+          <p1>0.0</p1>
+          <p2>0.0</p2>
+          <center>0.5 0.5</center>
+        </distortion>
+        <lens>
+          <intrinsics>
+            <fx>554.25469</fx>
+            <fy>554.25469</fy>
+            <cx>320.5</cx>
+            <cy>240.5</cy>
+            <s>0</s>
+          </intrinsics>
+          <!-- These need to match the intrinsics above or
+            Ignition will default to different default values -->
+          <projection>
+            <p_fx>554.25469</p_fx>
+            <p_fy>554.25469</p_fy>
+            <p_cx>320.5</p_cx>
+            <p_cy>240.5</p_cy>
+            <tx>0</tx>
+            <ty>0</ty>
+          </projection>
+        </lens>
+        <noise>
+          <type>gaussian</type>
+          <mean>0</mean>
+          <stddev>0.00</stddev>
+        </noise>
+        <depth_camera>
+          <clip>
+            <near>0.25</near>
+            <far>5</far>
+          </clip>
+        </depth_camera>
+        <optical_frame_id>wrist_mounted_camera_color_optical_frame</optical_frame_id>
+      </camera>
+      <ignition_frame_id>wrist_mounted_camera_color_frame</ignition_frame_id>
+      <always_on>1</always_on>
+      <update_rate>6</update_rate>
+      <visualize>false</visualize>
+      <topic>wrist_mounted_camera</topic>
+      <enable_metrics>false</enable_metrics>
+    </sensor>
+  </gazebo>
+  <joint name="ur_to_robotiq_joint" type="fixed">
+    <!-- The parent link must be read from the robot model it is attached to. -->
+    <parent link="realsense_camera_adapter_tool0"/>
+    <child link="ur_to_robotiq_link"/>
+    <origin rpy="0 0 0" xyz="0 0 0"/>
+  </joint>
+  <link name="ur_to_robotiq_link">
+    <visual>
+      <origin rpy="0 0 0" xyz="0 0 0"/>
+      <geometry>
+        <mesh filename="package://robotiq_description/meshes/visual/2f_85/ur_to_robotiq_adapter.dae"/>
+      </geometry>
+    </visual>
+    <collision>
+      <origin rpy="0 0 0" xyz="0 0 0"/>
+      <geometry>
+        <mesh filename="package://robotiq_description/meshes/collision/2f_85/ur_to_robotiq_adapter.stl"/>
+      </geometry>
+    </collision>
+    <inertial>
+      <mass value="0.01"/>
+      <origin xyz="0 0 0"/>
+      <inertia ixx="0.000044" ixy="0.0" ixz="0.0" iyy="0.000027" iyz="0.0" izz="0.000027"/>
+    </inertial>
+  </link>
+  <joint name="gripper_side_joint" type="fixed">
+    <parent link="ur_to_robotiq_link"/>
+    <child link="gripper_mount_link"/>
+    <!-- <origin xyz="0 0 0.011" rpy="0 ${-pi/2} ${pi/2}"/> -->
+    <origin rpy="0 0 0" xyz="0 0 0.011"/>
+  </joint>
+  <link name="gripper_mount_link"/>
+  <!-- Add robotiq 2f 85 gripper model -->
+  <link name="robotiq_85_base_link">
+    <visual>
+      <geometry>
+        <mesh filename="package://robotiq_description/meshes/visual/2f_85/robotiq_base.dae"/>
+      </geometry>
+    </visual>
+    <collision>
+      <geometry>
+        <mesh filename="package://robotiq_description/meshes/collision/2f_85/robotiq_base.stl"/>
+      </geometry>
+    </collision>
+    <inertial>
+      <origin rpy="0 0 0" xyz="0.0 2.274e-05 0.03232288"/>
+      <mass value="6.6320197e-01"/>
+      <inertia ixx="5.1617816e-04" ixy="2.936e-8" ixz="0.0" iyy="5.8802208e-04" iyz="-3.2296e-7" izz="3.9462776e-04"/>
+    </inertial>
+  </link>
+  <link name="robotiq_85_left_knuckle_link">
+    <visual>
+      <geometry>
+        <mesh filename="package://robotiq_description/meshes/visual/2f_85/left_knuckle.dae"/>
+      </geometry>
+    </visual>
+    <collision>
+      <geometry>
+        <mesh filename="package://robotiq_description/meshes/collision/2f_85/left_knuckle.stl"/>
+      </geometry>
+    </collision>
+    <inertial>
+      <origin rpy="0 0 0" xyz="0.01213197 0.0002 -0.00058647"/>
+      <mass value="1.384773208e-02"/>
+      <inertia ixx="3.5232e-7" ixy="0.0" ixz="1.1744e-7" iyy="2.31944e-6" iyz="0" izz="2.23136e-6"/>
+    </inertial>
+  </link>
+  <link name="robotiq_85_right_knuckle_link">
+    <visual>
+      <geometry>
+        <mesh filename="package://robotiq_description/meshes/visual/2f_85/right_knuckle.dae"/>
+      </geometry>
+    </visual>
+    <collision>
+      <geometry>
+        <mesh filename="package://robotiq_description/meshes/collision/2f_85/right_knuckle.stl"/>
+      </geometry>
+    </collision>
+    <inertial>
+      <origin rpy="0 0 0" xyz="-0.01213197 0.0002 -0.00058647"/>
+      <mass value="1.384773208e-02"/>
+      <inertia ixx="3.5232e-7" ixy="0.0" ixz="-1.1744e-7" iyy="2.31944e-6" iyz="0.0" izz="2.23136e-6"/>
+    </inertial>
+  </link>
+  <link name="robotiq_85_left_finger_link">
+    <visual>
+      <geometry>
+        <mesh filename="package://robotiq_description/meshes/visual/2f_85/left_finger.dae"/>
+      </geometry>
+    </visual>
+    <collision>
+      <geometry>
+        <mesh filename="package://robotiq_description/meshes/collision/2f_85/left_finger.stl"/>
+      </geometry>
+    </collision>
+    <inertial>
+      <origin rpy="0 0 0" xyz="0.00346899 -0.00079447 0.01867121"/>
+      <mass value="4.260376752e-02"/>
+      <inertia ixx="1.385792000000000e-05" ixy="0.0" ixz="-2.17264e-06" iyy="1.183208e-05" iyz="0.0" izz="5.19672e-06"/>
+    </inertial>
+  </link>
+  <link name="robotiq_85_right_finger_link">
+    <visual>
+      <geometry>
+        <mesh filename="package://robotiq_description/meshes/visual/2f_85/right_finger.dae"/>
+      </geometry>
+    </visual>
+    <collision>
+      <geometry>
+        <mesh filename="package://robotiq_description/meshes/collision/2f_85/right_finger.stl"/>
+      </geometry>
+    </collision>
+    <inertial>
+      <origin rpy="0 0 0" xyz="-0.00346899 -5.53e-06 0.01867121"/>
+      <mass value="4.260376752000000e-02"/>
+      <inertia ixx="1.385792e-05" ixy="0.0" ixz="2.17264e-06" iyy="1.183208e-05" iyz="0.0" izz="5.19672e-06"/>
+    </inertial>
+  </link>
+  <link name="robotiq_85_left_inner_knuckle_link">
+    <visual>
+      <geometry>
+        <mesh filename="package://robotiq_description/meshes/visual/2f_85/left_inner_knuckle.dae"/>
+      </geometry>
+    </visual>
+    <collision>
+      <geometry>
+        <mesh filename="package://robotiq_description/meshes/collision/2f_85/left_inner_knuckle.stl"/>
+      </geometry>
+    </collision>
+    <inertial>
+      <origin rpy="0 0 0" xyz="0.01897699 0.00015001 0.02247101"/>
+      <mass value="2.969376448e-02"/>
+      <inertia ixx="9.57136e-06" ixy="0.0" ixz="-3.93424e-06" iyy="8.69056e-06" iyz="0.0" izz="8.19144e-06"/>
+    </inertial>
+  </link>
+  <link name="robotiq_85_right_inner_knuckle_link">
+    <visual>
+      <geometry>
+        <mesh filename="package://robotiq_description/meshes/visual/2f_85/right_inner_knuckle.dae"/>
+      </geometry>
+    </visual>
+    <collision>
+      <geometry>
+        <mesh filename="package://robotiq_description/meshes/collision/2f_85/right_inner_knuckle.stl"/>
+      </geometry>
+    </collision>
+    <inertial>
+      <origin rpy="0 0 0" xyz="-0.01926824 5.001e-05 0.02222178"/>
+      <mass value="2.969376448e-02"/>
+      <inertia ixx="9.42456e-06" ixy="0.0" ixz="3.9636e-06" iyy="8.69056e-06" iyz="0.0" izz="8.33824e-06"/>
+    </inertial>
+  </link>
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
Commit message: add VFC example to mujoco config

File: src/picknik_ur_mujoco_config/description/picknik_ur.xacro (robot description, xacro)
@@ -783,10 +783,4 @@
     <dynamics damping="0" friction="0"/>
   </joint>
-  <link name="ft_frame"/>
-  <joint name="wrist_3_link-ft_frame" type="fixed">
-    <parent link="wrist_3_link"/>
-    <child link="ft_frame"/>
-    <origin rpy="3.141592653589793 0 0" xyz="0 0 0"/>
-  </joint>
   <!-- ROS-Industrial 'base' frame - base_link to UR 'Base' Coordinates transform -->
   <link name="base"/>

Commit message: update table position

File: src/picknik_ur_mujoco_config/description/picknik_ur.xacro (robot description, xacro)
@@ -867,11 +867,11 @@
       <origin rpy="0 0 0" xyz="0 0 0"/>
       <geometry>
-        <mesh filename="package://picknik_accessories/descriptions/furniture/generic_table/wood_block.dae" scale="0.125 0.125 0.00625"/>
-      </geometry>
-    </visual>
-    <collision>
-      <origin rpy="0 0 0" xyz="0 0 0"/>
-      <geometry>
-        <mesh filename="package://picknik_accessories/descriptions/furniture/generic_table/wood_block.dae" scale="0.125 0.125 0.00625"/>
+        <mesh filename="package://picknik_accessories/descriptions/furniture/generic_table/wood_block.dae" scale="0.125 0.125 0.05"/>
+      </geometry>
+    </visual>
+    <collision>
+      <origin rpy="0 0 0" xyz="0 0 0"/>
+      <geometry>
+        <mesh filename="package://picknik_accessories/descriptions/furniture/generic_table/wood_block.dae" scale="0.125 0.125 0.05"/>
       </geometry>
     </collision>
@@ -880,5 +880,5 @@
     <parent link="world"/>
     <child link="table"/>
-    <origin rpy="0 0 0" xyz="1 0 0.5"/>
+    <origin rpy="0 0 0" xyz="1 0 0.45"/>
   </joint>
   <ros2_control name="ur_mujoco_control" type="system">

Commit message: add VFC example to mujoco config (#319)

File: src/picknik_ur_mujoco_config/description/picknik_ur.xacro (robot description, xacro)
@@ -783,10 +783,4 @@
     <dynamics damping="0" friction="0"/>
   </joint>
-  <link name="ft_frame"/>
-  <joint name="wrist_3_link-ft_frame" type="fixed">
-    <parent link="wrist_3_link"/>
-    <child link="ft_frame"/>
-    <origin rpy="3.141592653589793 0 0" xyz="0 0 0"/>
-  </joint>
   <!-- ROS-Industrial 'base' frame - base_link to UR 'Base' Coordinates transform -->
   <link name="base"/>
@@ -873,11 +867,11 @@
       <origin rpy="0 0 0" xyz="0 0 0"/>
       <geometry>
-        <mesh filename="package://picknik_accessories/descriptions/furniture/generic_table/wood_block.dae" scale="0.125 0.125 0.00625"/>
-      </geometry>
-    </visual>
-    <collision>
-      <origin rpy="0 0 0" xyz="0 0 0"/>
-      <geometry>
-        <mesh filename="package://picknik_accessories/descriptions/furniture/generic_table/wood_block.dae" scale="0.125 0.125 0.00625"/>
+        <mesh filename="package://picknik_accessories/descriptions/furniture/generic_table/wood_block.dae" scale="0.125 0.125 0.05"/>
+      </geometry>
+    </visual>
+    <collision>
+      <origin rpy="0 0 0" xyz="0 0 0"/>
+      <geometry>
+        <mesh filename="package://picknik_accessories/descriptions/furniture/generic_table/wood_block.dae" scale="0.125 0.125 0.05"/>
       </geometry>
     </collision>
@@ -886,5 +880,5 @@
     <parent link="world"/>
     <child link="table"/>
-    <origin rpy="0 0 0" xyz="1 0 0.5"/>
+    <origin rpy="0 0 0" xyz="1 0 0.45"/>
   </joint>
   <ros2_control name="ur_mujoco_control" type="system">
