Commit message: updates to mujoco config

File: src/picknik_ur_mujoco_config/description/picknik_ur.xacro (robot description, xacro)
@@ -783,4 +783,10 @@
     <dynamics damping="0" friction="0"/>
   </joint>
+  <link name="ft_frame"/>
+  <joint name="wrist_3_link-ft_frame" type="fixed">
+    <parent link="wrist_3_link"/>
+    <child link="ft_frame"/>
+    <origin rpy="3.141592653589793 0 0" xyz="0 0 0"/>
+  </joint>
   <!-- ROS-Industrial 'base' frame - base_link to UR 'Base' Coordinates transform -->
   <link name="base"/>
@@ -867,11 +873,11 @@
       <origin rpy="0 0 0" xyz="0 0 0"/>
       <geometry>
-        <mesh filename="package://picknik_accessories/descriptions/furniture/generic_table/wood_block.dae" scale="0.125 0.125 0.05"/>
-      </geometry>
-    </visual>
-    <collision>
-      <origin rpy="0 0 0" xyz="0 0 0"/>
-      <geometry>
-        <mesh filename="package://picknik_accessories/descriptions/furniture/generic_table/wood_block.dae" scale="0.125 0.125 0.05"/>
+        <mesh filename="package://picknik_accessories/descriptions/furniture/generic_table/wood_block.dae" scale="0.125 0.125 0.00625"/>
+      </geometry>
+    </visual>
+    <collision>
+      <origin rpy="0 0 0" xyz="0 0 0"/>
+      <geometry>
+        <mesh filename="package://picknik_accessories/descriptions/furniture/generic_table/wood_block.dae" scale="0.125 0.125 0.00625"/>
       </geometry>
     </collision>
@@ -880,5 +886,5 @@
     <parent link="world"/>
     <child link="table"/>
-    <origin rpy="0 0 0" xyz="1 0 0.45"/>
+    <origin rpy="0 0 0" xyz="1 0 0.5"/>
   </joint>
   <ros2_control name="ur_mujoco_control" type="system">

Commit message: rotate scene 90 deg, add adapter to linear rail

File: src/picknik_ur_mujoco_config/description/picknik_ur.xacro (robot description, xacro)
@@ -531,5 +531,5 @@
     <parent link="world"/>
     <child link="linear_rail"/>
-    <origin rpy="0 0 0" xyz="0.0 0 0.6"/>
+    <origin rpy="0 0 1.5707" xyz="0.0 0 0.6"/>
   </joint>
   <!--
@@ -584,5 +584,12 @@
   <!-- Placeholder for ros2_control transmission which don't yet exist -->
   <!-- links -  main serial chain -->
-  <link name="base_link"/>
+  <link name="base_link">
+    <visual>
+      <origin rpy="0 0 0" xyz="0.0 0.0 -0.2"/>
+      <geometry>
+        <box size="0.16 0.2 0.4"/>
+      </geometry>
+    </visual>
+  </link>
   <link name="base_link_inertia">
     <visual>
@@ -720,5 +727,5 @@
   <!-- base_joint fixes base_link to the environment -->
   <joint name="base_joint" type="fixed">
-    <origin rpy="0 0 0" xyz="0 -0.4 0.0"/>
+    <origin rpy="0 0 0" xyz="-0.06 -0.4 0.0"/>
     <parent link="ur_linear_rail_base"/>
     <child link="base_link"/>
@@ -870,4 +877,40 @@
       </geometry>
     </visual>
+    <visual>
+      <origin rpy="0 0 0" xyz="0.4 0.4 -0.25"/>
+      <geometry>
+        <box size="0.04 0.04 0.5"/>
+      </geometry>
+      <material name="grey">
+        <color rgba="0.1 0.1 0.1 1.0"/>
+      </material>
+    </visual>
+    <visual>
+      <origin rpy="0 0 0" xyz="0.4 -0.4 -0.25"/>
+      <geometry>
+        <box size="0.04 0.04 0.5"/>
+      </geometry>
+      <material name="grey">
+        <color rgba="0.1 0.1 0.1 1.0"/>
+      </material>
+    </visual>
+    <visual>
+      <origin rpy="0 0 0" xyz="-0.4 -0.4 -0.25"/>
+      <geometry>
+        <box size="0.04 0.04 0.5"/>
+      </geometry>
+      <material name="grey">
+        <color rgba="0.1 0.1 0.1 1.0"/>
+      </material>
+    </visual>
+    <visual>
+      <origin rpy="0 0 0" xyz="-0.4 0.4 -0.25"/>
+      <geometry>
+        <box size="0.04 0.04 0.5"/>
+      </geometry>
+      <material name="grey">
+        <color rgba="0.1 0.1 0.1 1.0"/>
+      </material>
+    </visual>
     <collision>
       <origin rpy="0 0 0" xyz="0 0 0"/>
@@ -880,5 +923,5 @@
     <parent link="world"/>
     <child link="table"/>
-    <origin rpy="0 0 0" xyz="1 0 0.45"/>
+    <origin rpy="0 0 0" xyz="0 1 0.45"/>
   </joint>
   <ros2_control name="ur_mujoco_control" type="system">

Commit message: updates

File: src/picknik_ur_mujoco_config/description/picknik_ur.xacro (robot description, xacro)
@@ -878,5 +878,5 @@
   <link name="table">
     <visual>
-      <origin rpy="0 0 0" xyz="0 0 0"/>
+      <origin rpy="0 0 0" xyz="0 0 0.025"/>
       <geometry>
         <mesh filename="package://picknik_accessories/descriptions/furniture/generic_table/wood_block.dae" scale="0.125 0.125 0.00625"/>
@@ -884,7 +884,7 @@
     </visual>
     <visual>
-      <origin rpy="0 0 0" xyz="0.4 0.4 -0.25"/>
-      <geometry>
-        <box size="0.04 0.04 0.5"/>
+      <origin rpy="0 0 0" xyz="0.4 0.4 -0.2"/>
+      <geometry>
+        <box size="0.04 0.04 0.45"/>
       </geometry>
       <material name="grey">
@@ -893,7 +893,7 @@
     </visual>
     <visual>
-      <origin rpy="0 0 0" xyz="0.4 -0.4 -0.25"/>
-      <geometry>
-        <box size="0.04 0.04 0.5"/>
+      <origin rpy="0 0 0" xyz="0.4 -0.4 -0.2"/>
+      <geometry>
+        <box size="0.04 0.04 0.45"/>
       </geometry>
       <material name="grey">
@@ -902,7 +902,7 @@
     </visual>
     <visual>
-      <origin rpy="0 0 0" xyz="-0.4 -0.4 -0.25"/>
-      <geometry>
-        <box size="0.04 0.04 0.5"/>
+      <origin rpy="0 0 0" xyz="-0.4 -0.4 -0.2"/>
+      <geometry>
+        <box size="0.04 0.04 0.45"/>
       </geometry>
       <material name="grey">
@@ -911,7 +911,7 @@
     </visual>
     <visual>
-      <origin rpy="0 0 0" xyz="-0.4 0.4 -0.25"/>
-      <geometry>
-        <box size="0.04 0.04 0.5"/>
+      <origin rpy="0 0 0" xyz="-0.4 0.4 -0.2"/>
+      <geometry>
+        <box size="0.04 0.04 0.45"/>
       </geometry>
       <material name="grey">

Commit message: Mujoco 6.0 (#343)
* updates to mujoco config


Co-authored-by: Sebastian Jahr <sebastian.jahr@picknik.ai>
Co-authored-by: Mario Prats <mario.prats@picknik.ai>

File: src/picknik_ur_mujoco_config/description/picknik_ur.xacro (robot description, xacro)
@@ -531,5 +531,5 @@
     <parent link="world"/>
     <child link="linear_rail"/>
-    <origin rpy="0 0 0" xyz="0.0 0 0.6"/>
+    <origin rpy="0 0 1.5707" xyz="0.0 0 0.6"/>
   </joint>
   <!--
@@ -584,5 +584,12 @@
   <!-- Placeholder for ros2_control transmission which don't yet exist -->
   <!-- links -  main serial chain -->
-  <link name="base_link"/>
+  <link name="base_link">
+    <visual>
+      <origin rpy="0 0 0" xyz="0.0 0.0 -0.2"/>
+      <geometry>
+        <box size="0.16 0.2 0.4"/>
+      </geometry>
+    </visual>
+  </link>
   <link name="base_link_inertia">
     <visual>
@@ -720,5 +727,5 @@
   <!-- base_joint fixes base_link to the environment -->
   <joint name="base_joint" type="fixed">
-    <origin rpy="0 0 0" xyz="0 -0.4 0.0"/>
+    <origin rpy="0 0 0" xyz="-0.06 -0.4 0.0"/>
     <parent link="ur_linear_rail_base"/>
     <child link="base_link"/>
@@ -782,4 +789,10 @@
     <limit effort="28.0" lower="-6.283185307179586" upper="6.283185307179586" velocity="1.0471975511965976"/>
     <dynamics damping="0" friction="0"/>
+  </joint>
+  <link name="ft_frame"/>
+  <joint name="wrist_3_link-ft_frame" type="fixed">
+    <parent link="wrist_3_link"/>
+    <child link="ft_frame"/>
+    <origin rpy="3.141592653589793 0 0" xyz="0 0 0"/>
   </joint>
   <!-- ROS-Industrial 'base' frame - base_link to UR 'Base' Coordinates transform -->
@@ -865,13 +878,49 @@
   <link name="table">
     <visual>
-      <origin rpy="0 0 0" xyz="0 0 0"/>
-      <geometry>
-        <mesh filename="package://picknik_accessories/descriptions/furniture/generic_table/wood_block.dae" scale="0.125 0.125 0.05"/>
-      </geometry>
-    </visual>
-    <collision>
-      <origin rpy="0 0 0" xyz="0 0 0"/>
-      <geometry>
-        <mesh filename="package://picknik_accessories/descriptions/furniture/generic_table/wood_block.dae" scale="0.125 0.125 0.05"/>
+      <origin rpy="0 0 0" xyz="0 0 0.025"/>
+      <geometry>
+        <mesh filename="package://picknik_accessories/descriptions/furniture/generic_table/wood_block.dae" scale="0.125 0.125 0.00625"/>
+      </geometry>
+    </visual>
+    <visual>
+      <origin rpy="0 0 0" xyz="0.4 0.4 -0.2"/>
+      <geometry>
+        <box size="0.04 0.04 0.45"/>
+      </geometry>
+      <material name="grey">
+        <color rgba="0.1 0.1 0.1 1.0"/>
+      </material>
+    </visual>
+    <visual>
+      <origin rpy="0 0 0" xyz="0.4 -0.4 -0.2"/>
+      <geometry>
+        <box size="0.04 0.04 0.45"/>
+      </geometry>
+      <material name="grey">
+        <color rgba="0.1 0.1 0.1 1.0"/>
+      </material>
+    </visual>
+    <visual>
+      <origin rpy="0 0 0" xyz="-0.4 -0.4 -0.2"/>
+      <geometry>
+        <box size="0.04 0.04 0.45"/>
+      </geometry>
+      <material name="grey">
+        <color rgba="0.1 0.1 0.1 1.0"/>
+      </material>
+    </visual>
+    <visual>
+      <origin rpy="0 0 0" xyz="-0.4 0.4 -0.2"/>
+      <geometry>
+        <box size="0.04 0.04 0.45"/>
+      </geometry>
+      <material name="grey">
+        <color rgba="0.1 0.1 0.1 1.0"/>
+      </material>
+    </visual>
+    <collision>
+      <origin rpy="0 0 0" xyz="0 0 0"/>
+      <geometry>
+        <mesh filename="package://picknik_accessories/descriptions/furniture/generic_table/wood_block.dae" scale="0.125 0.125 0.00625"/>
       </geometry>
     </collision>
@@ -880,5 +929,5 @@
     <parent link="world"/>
     <child link="table"/>
-    <origin rpy="0 0 0" xyz="1 0 0.45"/>
+    <origin rpy="0 0 0" xyz="0 1 0.45"/>
   </joint>
   <ros2_control name="ur_mujoco_control" type="system">

Commit message: replace rail stl by boxes and tweak model

File: src/picknik_ur_mujoco_config/description/picknik_ur.xacro (robot description, xacro)
@@ -513,7 +513,7 @@
   <link name="linear_rail">
     <visual>
-      <origin rpy="0 0 0" xyz="0 0 0.05"/>
-      <geometry>
-        <mesh filename="package://picknik_ur_mujoco_config/description/assets/rail.stl"/>
+      <origin rpy="0 0 0" xyz="0 0 0"/>
+      <geometry>
+        <box size="5.0 0.6 0.30"/>
       </geometry>
       <material name="grey">
@@ -521,9 +521,48 @@
       </material>
     </visual>
-    <collision>
-      <origin rpy="0 0 0" xyz="0 0 0.05"/>
-      <geometry>
-        <mesh filename="package://picknik_ur_mujoco_config/description/assets/rail.stl"/>
-      </geometry>
+    <visual>
+      <origin rpy="0 0 0" xyz="0 0.14 0.125"/>
+      <geometry>
+        <box size="5.0 0.2 0.5"/>
+      </geometry>
+      <material name="grey">
+        <color rgba="0.1 0.1 0.1 1.0"/>
+      </material>
+    </visual>
+    <visual>
+      <origin rpy="0 0 0" xyz="0 -0.22 0.125"/>
+      <geometry>
+        <box size="5.0 0.12 0.5"/>
+      </geometry>
+      <material name="grey">
+        <color rgba="0.1 0.1 0.1 1.0"/>
+      </material>
+    </visual>
+    <collision>
+      <origin rpy="0 0 0" xyz="0 0 0"/>
+      <geometry>
+        <box size="5.0 0.6 0.3"/>
+      </geometry>
+      <material name="grey">
+        <color rgba="0.1 0.1 0.1 1.0"/>
+      </material>
+    </collision>
+    <collision>
+      <origin rpy="0 0 0" xyz="0 0.14 0.125"/>
+      <geometry>
+        <box size="5.0 0.2 0.5"/>
+      </geometry>
+      <material name="grey">
+        <color rgba="0.1 0.1 0.1 1.0"/>
+      </material>
+    </collision>
+    <collision>
+      <origin rpy="0 0 0" xyz="0 -0.22 0.125"/>
+      <geometry>
+        <box size="5.0 0.12 0.5"/>
+      </geometry>
+      <material name="grey">
+        <color rgba="0.1 0.1 0.1 1.0"/>
+      </material>
     </collision>
   </link>
@@ -531,5 +570,5 @@
     <parent link="world"/>
     <child link="linear_rail"/>
-    <origin rpy="0 0 1.5707" xyz="0.0 0 0.6"/>
+    <origin rpy="0 0 0" xyz="0.0 0 0.0"/>
   </joint>
   <!--
@@ -727,5 +766,5 @@
   <!-- base_joint fixes base_link to the environment -->
   <joint name="base_joint" type="fixed">
-    <origin rpy="0 0 0" xyz="-0.06 -0.4 0.0"/>
+    <origin rpy="0 0 1.5707" xyz="0.4 -0.06 0.6"/>
     <parent link="ur_linear_rail_base"/>
     <child link="base_link"/>
@@ -868,9 +907,9 @@
   </joint>
   <joint name="linear_rail_joint" type="prismatic">
-    <axis xyz="0 1 0"/>
+    <axis xyz="-1 0 0"/>
     <parent link="linear_rail"/>
     <child link="ur_linear_rail_base"/>
     <origin rpy="0 0 0" xyz="0 0 0"/>
-    <limit acceleration="10.0" effort="1000.0" lower="-5.0" upper="5.0" velocity="0.175"/>
+    <limit acceleration="10.0" effort="1000.0" lower="-2.1" upper="2.9" velocity="0.175"/>
     <dynamics damping="20.0" friction="500.0"/>
   </joint>

Commit message: revert changes to picknik_ur.xacro

File: src/picknik_ur_mujoco_config/description/picknik_ur.xacro (robot description, xacro)
@@ -919,40 +919,4 @@
       </material>
     </visual>
-    <visual>
-      <origin rpy="0 0 0" xyz="0.4 0.4 -0.25"/>
-      <geometry>
-        <box size="0.04 0.04 0.5"/>
-      </geometry>
-      <material name="grey">
-        <color rgba="0.1 0.1 0.1 1.0"/>
-      </material>
-    </visual>
-    <visual>
-      <origin rpy="0 0 0" xyz="0.4 -0.4 -0.25"/>
-      <geometry>
-        <box size="0.04 0.04 0.5"/>
-      </geometry>
-      <material name="grey">
-        <color rgba="0.1 0.1 0.1 1.0"/>
-      </material>
-    </visual>
-    <visual>
-      <origin rpy="0 0 0" xyz="-0.4 -0.4 -0.25"/>
-      <geometry>
-        <box size="0.04 0.04 0.5"/>
-      </geometry>
-      <material name="grey">
-        <color rgba="0.1 0.1 0.1 1.0"/>
-      </material>
-    </visual>
-    <visual>
-      <origin rpy="0 0 0" xyz="-0.4 0.4 -0.25"/>
-      <geometry>
-        <box size="0.04 0.04 0.5"/>
-      </geometry>
-      <material name="grey">
-        <color rgba="0.1 0.1 0.1 1.0"/>
-      </material>
-    </visual>
     <collision>
       <origin rpy="0 0 0" xyz="0 0 0"/>

Commit message: fixed scene camera

File: src/picknik_ur_mujoco_config/description/picknik_ur.xacro (robot description, xacro)
@@ -531,5 +531,5 @@
     <parent link="world"/>
     <child link="linear_rail"/>
-    <origin rpy="0 0 1.5707" xyz="0.0 0 0.6"/>
+    <origin rpy="0 0 1.5707" xyz="0.0 -1 1"/>
   </joint>
   <!--

Commit message: Remove some assets to try to improve camera performance

File: src/picknik_ur_mujoco_config/description/picknik_ur.xacro (robot description, xacro)
@@ -876,5 +876,5 @@
   </joint>
   <!-- Table -->
-  <link name="table">
+  <!-- <link name="table">
     <visual>
       <origin rpy="0 0 0" xyz="0 0 0.025"/>
@@ -930,5 +930,5 @@
     <child link="table"/>
     <origin rpy="0 0 0" xyz="0 1 0.45"/>
-  </joint>
+  </joint> -->
   <ros2_control name="ur_mujoco_control" type="system">
     <hardware>
