Commit message: Update multi arm and gazebo srdfs to use chains for gripper groups.

File: src/picknik_ur_gazebo_config/config/moveit/picknik_ur_gazebo.srdf.xacro (robot description, xacro)
@@ -16,15 +16,7 @@
   </group>
   <group name="gripper">
-    <link name="$(arg gripper_name)_base_link" />
-    <link name="$(arg gripper_name)_left_inner_knuckle_link" />
-    <link name="$(arg gripper_name)_left_finger_tip_link" />
-    <link name="$(arg gripper_name)_left_knuckle_link" />
-    <link name="$(arg gripper_name)_left_finger_link" />
-    <link name="$(arg gripper_name)_right_inner_knuckle_link" />
-    <link name="$(arg gripper_name)_right_finger_tip_link" />
-    <link name="$(arg gripper_name)_right_knuckle_link" />
-    <link name="$(arg gripper_name)_right_finger_link" />
-    <link name="grasp_link" />
-    <joint name="$(arg gripper_name)_left_knuckle_joint" />
+    <chain base_link="robotiq_85_base_link" tip_link="$(arg gripper_name)_left_finger_link"/>
+    <chain base_link="robotiq_85_base_link" tip_link="$(arg gripper_name)_right_finger_link"/>
+    <chain base_link="robotiq_85_base_link" tip_link="grasp_link"/>
   </group>
   <!--GROUP STATES: Purpose: Define a named state for a particular group, in terms of joint values. This is useful to define states like 'folded arms'-->
